File: batteryBalancer/Blaine/batteryBalancer.sch (EAGLE design)
At the start: 30 parts

Commit message: Fancied up the schematic, nets still need to be named
Parts:
- removed BATTERY_A, BATTERY_B, MOTOR_POWER: 39-30-06, con-molex-mini-fit:39-30-06
- removed U$1, U$3: LM5050-1, lio:LM5050-1
- removed U$10, U$11, U$12, U$9: CMX60D20, CMX60D20:CMX60D20
- removed U$13, U$14: 01220083Z, 01220083Z:01220083Z
- removed U$15: ADC128D818, ADC128D818:ADC128D818
- removed U$16: 5530843_MATE, 5530843-6 - backplane:5530843_MATE
- removed U$17, U$5: ACS722, ACS722:ACS722
- removed U$2, U$4: IXFX64N60P3, IXFX64N60P3:IXFX64N60P3
- removed U$6, U$7, U$8: LTST-S270GKT, LTST-S270GKT:LTST-S270GKT
- added ADC: ADC128D818, ADC128D818:ADC128D818
- added BALANCED_STATUS, PORT_STATUS, STBD_STATUS: LTST-S270GKT, LTST-S270GKT:LTST-S270GKT
- added BATTERY_PORT, BATTERY_STBD, MOTOR_POWER2: 39-30-06, con-molex-mini-fit:39-30-06
- added EDGE_CONNECTOR: 5530843, 5530843-6:5530843
- added OFF: (no value), wirepad:2,54/1,1
- added PORT_CS, STBD_CS: ACS722, ACS722:ACS722
- added PORT_FC, STBD_FC: LM5050-1, lio:LM5050-1
- added PORT_FET, STBD_FET: IXFX64N60P3, IXFX64N60P3:IXFX64N60P3
- added PORT_FUSE, STBD_FUSE: 01220083Z, 01220083Z:01220083Z
- added RELAY2, RELAY3, RELAY4, RLAY1: CMX60D20, CMX60D20:CMX60D20
- R1, R2, R3: value (none) -> 700
Connections:
- removed net N$18: U$15.SDA, U$16.SDA_SENSOR
- removed net N$21: U$14.P$2, U$17.IP+1, U$17.IP+2, U$7.ANODE
- new net 3.3V: ADC.V+, EDGE_CONNECTOR.3.3V_1, EDGE_CONNECTOR.3.3V_2, EDGE_CONNECTOR.3.3V_3, PORT_CS.VCC, R6.1, R7.1, STBD_CS.VCC
- new net LOGIC_GND: ADC.GND, EDGE_CONNECTOR.GND_1, EDGE_CONNECTOR.GND_2, EDGE_CONNECTOR.GND_3, PORT_CS.BW_SEL, PORT_CS.GND, R4.2, R5.2, RELAY2.CONTROL-, RELAY3.CONTROL-, RELAY4.CONTROL-, RLAY1.CONTROL-, STBD_CS.BW_SEL, STBD_CS.GND
- new net N$22: MOTOR_POWER2.1, MOTOR_POWER2.2, MOTOR_POWER2.3, RELAY3.LOAD-, RELAY4.LOAD-
- net GND: now also BALANCED_STATUS.C, BATTERY_BALANCED.4, BATTERY_BALANCED.5, BATTERY_BALANCED.6, BATTERY_PORT.4, BATTERY_PORT.5, BATTERY_PORT.6, BATTERY_STBD.4, BATTERY_STBD.5, BATTERY_STBD.6, MOTOR_POWER1.4, MOTOR_POWER1.5, MOTOR_POWER1.6, MOTOR_POWER2.4, MOTOR_POWER2.5, MOTOR_POWER2.6, PORT_FC.GND, STBD_FC.GND; no longer BATTERY_A.1, BATTERY_A.2, BATTERY_A.3, BATTERY_B.1, BATTERY_B.2, BATTERY_B.3, BATTERY_BALANCED.1, BATTERY_BALANCED.2, BATTERY_BALANCED.3, MOTOR_POWER.1, MOTOR_POWER.2, MOTOR_POWER.3, MOTOR_POWER1.1, MOTOR_POWER1.2, MOTOR_POWER1.3, U$1.GND, U$3.GND, U$8.CATHODE
- net N$1: now also BALANCED_STATUS.A; no longer U$8.ANODE
- net N$10: now also PORT_STATUS.C, R1.2; no longer MOTOR_POWER.4, MOTOR_POWER.5, MOTOR_POWER.6, U$10.LOAD-, U$9.LOAD-
- net N$11: now also ADC.A0; no longer U$15.A0
- net N$12: now also EDGE_CONNECTOR.KILL_SWITCH, RELAY2.CONTROL+, RELAY3.CONTROL+, RELAY4.CONTROL+, RLAY1.CONTROL+; no longer MOTOR_POWER1.4, MOTOR_POWER1.5, MOTOR_POWER1.6, U$11.LOAD-, U$12.LOAD-
- net N$13: now also ADC.A1; no longer U$15.A1
- net N$14: now also PORT_CS.IP-1, PORT_CS.IP-2, PORT_FC.IN, PORT_FET.SOURCE; no longer U$1.IN, U$17.IP-1, U$17.IP-2, U$4.SOURCE
- net N$15: now also OFF.P, PORT_FC.OFF, STBD_FC.OFF; no longer R1.2, U$7.CATHODE
- net N$16: now also STBD_CS.IP-1, STBD_CS.IP-2, STBD_FC.IN, STBD_FET.SOURCE; no longer U$2.SOURCE, U$3.IN, U$5.IP-1, U$5.IP-2
- net N$17: now also ADC.SCL, EDGE_CONNECTOR.SCL_SENSOR; no longer U$15.SCL, U$16.SCL_SENSOR
- net N$19: now also BATTERY_PORT.1, BATTERY_PORT.2, BATTERY_PORT.3, PORT_FUSE.P$1; no longer R6.1, R7.1, U$15.V+, U$16.3.3V_2, U$17.VCC, U$5.VCC
- net N$2: now also STBD_FC.GATE, STBD_FET.GATE; no longer U$2.GATE, U$3.GATE
- net N$20: now also STBD_CS.IP+1, STBD_CS.IP+2, STBD_FUSE.P$2, STBD_STATUS.A; no longer U$13.P$2, U$5.IP+1, U$5.IP+2, U$6.ANODE
- net N$24: now also ADC.IN0, PORT_CS.VIOUT; no longer U$15.IN0, U$17.VIOUT
- net N$25: now also ADC.IN1, STBD_CS.VIOUT; no longer U$15.IN1, U$5.VIOUT
- net N$3: now also BATTERY_BALANCED.1, BATTERY_BALANCED.2, BATTERY_BALANCED.3, C1.2, PORT_FC.OUT, PORT_FC.VS, PORT_FET.DRAIN, R3.2, RELAY2.LOAD+, RELAY3.LOAD+, RELAY4.LOAD+, RLAY1.LOAD+, STBD_FC.OUT, STBD_FC.VS, STBD_FET.DRAIN; no longer BATTERY_A.4, BATTERY_A.5, BATTERY_A.6, U$14.P$1
- net N$4: now also BATTERY_STBD.1, BATTERY_STBD.2, BATTERY_STBD.3, STBD_FUSE.P$1; no longer BATTERY_B.4, BATTERY_B.5, BATTERY_B.6, U$13.P$1
- net N$5: now also MOTOR_POWER1.1, MOTOR_POWER1.2, MOTOR_POWER1.3, RELAY2.LOAD-, RLAY1.LOAD-; no longer BATTERY_BALANCED.4, BATTERY_BALANCED.5, BATTERY_BALANCED.6, C1.2, R3.2, U$1.OUT, U$1.VS, U$10.LOAD+, U$11.LOAD+, U$12.LOAD+, U$2.DRAIN, U$3.OUT, U$3.VS, U$4.DRAIN, U$9.LOAD+
- net N$6: now also PORT_FC.GATE, PORT_FET.GATE; no longer U$1.GATE, U$4.GATE
- net N$7: now also PORT_CS.IP+1, PORT_CS.IP+2, PORT_FUSE.P$2, PORT_STATUS.A; no longer R4.2, R5.2, U$10.CONTROL-, U$11.CONTROL-, U$12.CONTROL-, U$15.GND, U$16.GND3, U$17.BW_SEL, U$17.GND, U$5.BW_SEL, U$5.GND, U$9.CONTROL-
- net N$8: now also STBD_STATUS.C; no longer U$6.CATHODE
- net N$9: now also ADC.SDA, EDGE_CONNECTOR.SDA_SENSOR; no longer U$10.CONTROL+, U$11.CONTROL+, U$12.CONTROL+, U$16.KILL_SWITCH, U$9.CONTROL+
Other:
- note added: "Spot for power shutoff if we want it later"
- note added: "These resistors are for addressing, remove for different addresses"
- moved on the sheet: BATTERY_BALANCED, C1, MOTOR_POWER1, R1, R2, R3, R4, R5, R6, R7
