File: batteryBalancer/Blaine/batteryBalancer.sch (EAGLE design)
At the start: 31 parts

Commit message: Added net names
Connections:
- net N$1 renamed BALANCED_INDICATOR
- net N$10 renamed PORT_INDICATOR
- net N$11 renamed ADC_A0
- net N$12 renamed KILL_SWITCH
- net N$13 renamed ADC_A1
- net N$14 renamed PORT_UNBALANCED
- net N$15 renamed OFF
- net N$16 renamed STBD_UNBALANCED
- net N$17 renamed SCL
- net N$19 renamed PORT_POWER
- net N$2 renamed STBD_GATE
- net N$20 renamed STBD_FUSED
- net N$22 renamed MOTOR_POWER2
- net N$24 renamed PORT_CURRENT
- net N$25 renamed STBD_CURRENT
- net N$3 renamed BALANCED_POWER
- net N$4 renamed STBD_POWER
- net N$5 renamed MOTOR_POWER1
- net N$6 renamed PORT_GATE
- net N$7 renamed PORT_FUSED
- net N$8 renamed STBD_INDICATOR
- net N$9 renamed SDA
Changed lines of the file:
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@@
 </segment>
 </net>
-<net name="N$2" class="0">
+<net name="STBD_GATE" class="0">
 <segment>
 <pinref part="STBD_FC" gate="G$1" pin="GATE"/>
@@
 </segment>
 </net>
-<net name="N$6" class="0">
+<net name="PORT_GATE" class="0">
 <segment>
 <pinref part="PORT_FC" gate="G$1" pin="GATE"/>
@@
 </segment>
 </net>
-<net name="N$8" class="0">
+<net name="STBD_INDICATOR" class="0">
 <segment>
 <pinref part="R2" gate="G$1" pin="2"/>
@@
 </segment>
 </net>
-<net name="N$1" class="0">
+<net name="BALANCED_INDICATOR" class="0">
 <segment>
 <pinref part="R3" gate="G$1" pin="1"/>
@@
 </segment>
 </net>
-<net name="N$14" class="0">
+<net name="PORT_UNBALANCED" class="0">
 <segment>
 <pinref part="PORT_FC" gate="G$1" pin="IN"/>
@@
 </segment>
 </net>
-<net name="N$16" class="0">
+<net name="STBD_UNBALANCED" class="0">
 <segment>
 <wire x1="124.46" y1="205.74" x2="129.54" y2="205.74" width="0.1524" layer="91"/>
@@
 </segment>
 </net>
-<net name="N$17" class="0">
+<net name="SCL" class="0">
 <segment>
 <pinref part="ADC" gate="G$1" pin="SCL"/>
@@
 </segment>
 </net>
-<net name="N$11" class="0">
+<net name="ADC_A0" class="0">
 <segment>
 <pinref part="R4" gate="G$1" pin="1"/>
@@
 </segment>
 </net>
-<net name="N$13" class="0">
+<net name="ADC_A1" class="0">
 <segment>
 <pinref part="ADC" gate="G$1" pin="A1"/>
@@
 </segment>
 </net>
-<net name="N$20" class="0">
+<net name="STBD_FUSED" class="0">
 <segment>
 <pinref part="STBD_CS" gate="G$1" pin="IP+1"/>
@@
 </segment>
 </net>
-<net name="N$24" class="0">
+<net name="PORT_CURRENT" class="0">
 <segment>
 <pinref part="PORT_CS" gate="G$1" pin="VIOUT"/>
@@
 </segment>
 </net>
-<net name="N$25" class="0">
+<net name="STBD_CURRENT" class="0">
 <segment>
 <pinref part="STBD_CS" gate="G$1" pin="VIOUT"/>
@@
 </segment>
 </net>
-<net name="N$4" class="0">
+<net name="STBD_POWER" class="0">
 <segment>
 <pinref part="BATTERY_STBD" gate="G$1" pin="3"/>
@@
 </segment>
 </net>
-<net name="N$19" class="0">
+<net name="PORT_POWER" class="0">
 <segment>
 <pinref part="PORT_FUSE" gate="G$1" pin="P$1"/>
@@
 </segment>
 </net>
-<net name="N$3" class="0">
+<net name="BALANCED_POWER" class="0">
 <segment>
 <pinref part="BATTERY_BALANCED" gate="G$1" pin="3"/>
@@
 </segment>
 </net>
-<net name="N$5" class="0">
+<net name="MOTOR_POWER1" class="0">
 <segment>
 <pinref part="RELAY2" gate="G$1" pin="LOAD-"/>
@@
 </segment>
 </net>
-<net name="N$22" class="0">
+<net name="MOTOR_POWER2" class="0">
 <segment>
 <pinref part="RELAY3" gate="G$1" pin="LOAD-"/>
@@
 </segment>
 </net>
-<net name="N$7" class="0">
+<net name="PORT_FUSED" class="0">
 <segment>
 <pinref part="PORT_FUSE" gate="G$1" pin="P$2"/>
@@
 </segment>
 </net>
-<net name="N$9" class="0">
+<net name="SDA" class="0">
 <segment>
 <pinref part="EDGE_CONNECTOR" gate="G$1" pin="SDA_SENSOR"/>
@@
 </segment>
 </net>
-<net name="N$12" class="0">
+<net name="KILL_SWITCH" class="0">
 <segment>
 <pinref part="EDGE_CONNECTOR" gate="G$1" pin="KILL_SWITCH"/>
@@
 </segment>
 </net>
-<net name="N$10" class="0">
+<net name="PORT_INDICATOR" class="0">
 <segment>
 <pinref part="R1" gate="G$1" pin="2"/>
@@
 </segment>
 </net>
-<net name="N$15" class="0">
+<net name="OFF" class="0">
 <segment>
 <pinref part="PORT_FC" gate="G$1" pin="OFF"/>
