File: Converter Board/Converter Board.brd (EAGLE design)
At the start: 101.6 x 101.6 mm, 5 parts, among them P1 39-30-06?, P2 39-30-06?

Commit message: Revising converter board
Parts:
- moved U$2 248.7 mm to (22.2, 61.9)
- moved U$1 182.0 mm to (22.2, 27.0)
- moved P2 172.7 mm to (9.53, 55.6)
- moved U$3 65.7 mm to (15.9, 0.00)
Other:
- board text removed: "The Underwater Robotics Team Riptide -- Board Template"
Changed lines of the file:
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@@
 <text x="15.875" y="17.4625" size="1.778" layer="21">The Ohio State Univerity
 Center for Automotive Research</text>
-<text x="15.875" y="25.4" size="1.778" layer="49">The Underwater Robotics Team
-Riptide -- Board Template</text>
 </plain>
 <attributes>
@@
 </autorouter>
 <elements>
-<element name="U$3" library="5530843-6" package="5530843-6-BOARDFINGERS" value="5530843" x="-23.8125" y="-52.3875"/>
-<element name="P2" library="con-molex-mini-fit" package="39-30-?06?" value="39-30-06?" x="-41.275" y="-109.5375"/>
-<element name="U$1" library="3.3V Converter" package="3.3VCONV" value="3.3VCONV" x="-84.1375" y="-120.65"/>
-<element name="U$2" library="12VCONV" package="12VCONV" value="12VCONV" x="-79.375" y="-165.1"/>
+<element name="U$3" library="5530843-6" package="5530843-6-BOARDFINGERS" value="5530843" x="15.875" y="0"/>
+<element name="P2" library="con-molex-mini-fit" package="39-30-?06?" value="39-30-06?" x="9.525" y="55.5625"/>
+<element name="U$1" library="3.3V Converter" package="3.3VCONV" value="3.3VCONV" x="22.225" y="26.9875"/>
+<element name="U$2" library="12VCONV" package="12VCONV" value="12VCONV" x="22.225" y="61.9125"/>
 <element name="P1" library="con-molex-mini-fit" package="39-30-?06?" value="39-30-06?" x="-69.85" y="-188.9125"/>
 </elements>
@@
 <contactref element="U$3" pad="3.3VP3"/>
 <contactref element="U$1" pad="14"/>
-<wire x1="-22.987" y1="-49.2125" x2="-81.5975" y2="-116.332" width="0" layer="19" extent="1-1"/>
-<wire x1="-20.447" y1="-49.2125" x2="-22.987" y2="-49.2125" width="0" layer="19" extent="1-1"/>
-<wire x1="-17.907" y1="-49.2125" x2="-20.447" y2="-49.2125" width="0" layer="19" extent="1-1"/>
+<wire x1="16.7005" y1="3.175" x2="24.765" y2="31.3055" width="0" layer="19" extent="1-1"/>
+<wire x1="19.2405" y1="3.175" x2="16.7005" y2="3.175" width="0" layer="19" extent="1-1"/>
+<wire x1="21.7805" y1="3.175" x2="19.2405" y2="3.175" width="0" layer="19" extent="1-1"/>
 </signal>
 <signal name="N$6">
@@
 <contactref element="U$3" pad="GND3"/>
 <contactref element="U$1" pad="16"/>
-<wire x1="-15.367" y1="-49.2125" x2="-81.5975" y2="-111.252" width="0" layer="19" extent="1-1"/>
-<wire x1="-12.827" y1="-49.2125" x2="-15.367" y2="-49.2125" width="0" layer="19" extent="1-1"/>
-<wire x1="-10.287" y1="-49.2125" x2="-12.827" y2="-49.2125" width="0" layer="19" extent="1-1"/>
+<wire x1="24.3205" y1="3.175" x2="24.765" y2="36.3855" width="0" layer="19" extent="1-1"/>
+<wire x1="26.8605" y1="3.175" x2="24.3205" y2="3.175" width="0" layer="19" extent="1-1"/>
+<wire x1="29.4005" y1="3.175" x2="26.8605" y2="3.175" width="0" layer="19" extent="1-1"/>
 </signal>
 <signal name="N$1">
@@
 <contactref element="P2" pad="5"/>
 <contactref element="U$2" pad="1,+VIN"/>
-<wire x1="-81.5975" y1="-96.012" x2="-75.819" y2="-139.065" width="0" layer="19" extent="1-1"/>
-<wire x1="-81.5975" y1="-93.472" x2="-81.5975" y2="-96.012" width="0" layer="19" extent="1-1"/>
-<wire x1="-45.466" y1="-104.0257" x2="-81.5975" y2="-96.012" width="0" layer="19" extent="1-1"/>
-<wire x1="-41.275" y1="-104.0257" x2="-45.466" y2="-104.0257" width="0" layer="19" extent="1-1"/>
-<wire x1="-37.084" y1="-104.0257" x2="-41.275" y2="-104.0257" width="0" layer="19" extent="1-1"/>
+<wire x1="24.765" y1="51.6255" x2="25.781" y2="87.9475" width="0" layer="19" extent="1-1"/>
+<wire x1="24.765" y1="54.1655" x2="24.765" y2="51.6255" width="0" layer="19" extent="1-1"/>
+<wire x1="5.334" y1="61.0743" x2="24.765" y2="51.6255" width="0" layer="19" extent="1-1"/>
+<wire x1="9.525" y1="61.0743" x2="5.334" y2="61.0743" width="0" layer="19" extent="1-1"/>
+<wire x1="13.716" y1="61.0743" x2="9.525" y2="61.0743" width="0" layer="19" extent="1-1"/>
 </signal>
 <signal name="N$2">
@@
 <contactref element="P2" pad="2"/>
 <contactref element="U$2" pad="3,-VIN"/>
-<wire x1="-45.466" y1="-109.5375" x2="-75.819" y2="-154.305" width="0" layer="19" extent="1-1"/>
-<wire x1="-41.275" y1="-109.5375" x2="-45.466" y2="-109.5375" width="0" layer="19" extent="1-1"/>
-<wire x1="-37.084" y1="-109.5375" x2="-41.275" y2="-109.5375" width="0" layer="19" extent="1-1"/>
-<wire x1="-65.0875" y1="-96.012" x2="-45.466" y2="-109.5375" width="0" layer="19" extent="1-1"/>
-<wire x1="-65.0875" y1="-93.472" x2="-65.0875" y2="-96.012" width="0" layer="19" extent="1-1"/>
+<wire x1="5.334" y1="55.5625" x2="25.781" y2="72.7075" width="0" layer="19" extent="1-1"/>
+<wire x1="9.525" y1="55.5625" x2="5.334" y2="55.5625" width="0" layer="19" extent="1-1"/>
+<wire x1="13.716" y1="55.5625" x2="9.525" y2="55.5625" width="0" layer="19" extent="1-1"/>
+<wire x1="41.275" y1="51.6255" x2="5.334" y2="55.5625" width="0" layer="19" extent="1-1"/>
+<wire x1="41.275" y1="54.1655" x2="41.275" y2="51.6255" width="0" layer="19" extent="1-1"/>
 </signal>
 <signal name="N$9">
@@
 <wire x1="-69.85" y1="-188.9125" x2="-65.659" y2="-188.9125" width="0" layer="19" extent="1-1"/>
 <wire x1="-74.041" y1="-188.9125" x2="-69.85" y2="-188.9125" width="0" layer="19" extent="1-1"/>
-<wire x1="-25.019" y1="-139.065" x2="-65.659" y2="-188.9125" width="0" layer="19" extent="1-1"/>
+<wire x1="76.581" y1="87.9475" x2="-65.659" y2="-188.9125" width="0" layer="19" extent="1-1"/>
 </signal>
 <signal name="N$10">
@@
 <wire x1="-65.659" y1="-183.4007" x2="-69.85" y2="-183.4007" width="0" layer="19" extent="1-1"/>
 <wire x1="-74.041" y1="-183.4007" x2="-69.85" y2="-183.4007" width="0" layer="19" extent="1-1"/>
-<wire x1="-25.019" y1="-154.305" x2="-65.659" y2="-183.4007" width="0" layer="19" extent="1-1"/>
+<wire x1="76.581" y1="72.7075" x2="-65.659" y2="-183.4007" width="0" layer="19" extent="1-1"/>
 </signal>
 </signals>
