File: Converter Board/Converter Board.sch (EAGLE design)
At the start: 5 parts, among them P1 39-30-06, P2 39-30-06

Commit message: Revising converter board
Connections:
- removed net N$9: P1.1, P1.2, P1.3, U$2.4,-VOUT
- new net N$10: P1.1, P1.2, P1.3
Other:
- moved on the sheet: P1, P2
