File: Converter Board/ConverterBoard.brd (EAGLE design)
At the start: 101.6 x 101.6 mm, 5 parts, among them P1 39-30-06?, P2 39-30-06?

Commit message: Revised 12 V and 3.3 V Converters Finished the majority of the converter board
Parts:
- U$1: value 3.3VCONV -> 12VCONV; device 3.3V Converter:3.3VCONV -> 12VCONV:12VCONV
- U$2: value 12VCONV -> 3.3VCONV; device 12VCONV:12VCONV -> 3.3V Converter:3.3VCONV
- moved P1 240.4 mm to (15.9, 35.7), turned to 270 degrees
- moved P2 78.7 mm to (85.7, 35.7), turned to 90 degrees
- moved U$2 63.6 mm to (66.8, 16.5), turned to 90 degrees
- moved U$1 22.3 mm to (21.8, 49.3)
Connections:
- removed net N$1: P2.4, P2.5, P2.6, U$1.22, U$1.23, U$2.1,+VIN
- removed net N$10: P1.4, P1.5, P1.6, U$2.8,+VOUT
- removed net N$2: P2.1, P2.2, P2.3, U$1.2, U$1.3, U$2.3,-VIN
- removed net N$5: U$1.14, U$3.3.3VP1, U$3.3.3VP2, U$3.3.3VP3
- removed net N$6: U$1.16, U$3.GND1, U$3.GND2, U$3.GND3
- removed net N$9: P1.1, P1.2, P1.3, U$2.4,-VOUT
- new net 12V+: P2.1, P2.2, P2.3, U$1.8,+VOUT
- new net 12V-: P2.4, P2.5, P2.6, U$1.4,-VOUT
- new net 3.3V: U$2.14, U$3.3.3VP1, U$3.3.3VP2, U$3.3.3VP3, U$3.3.3V_4, U$3.3.3V_5, U$3.3.3V_6
- new net 3.3VGROUND: U$2.16, U$3.GND1, U$3.GND2, U$3.GND3, U$3.GND_4, U$3.GND_5, U$3.GND_6
- new net BALANCEDRAW+: P1.1, P1.2, P1.3, U$1.1,+VIN, U$1.2,ON/OFF, U$2.22, U$2.23
- new net BALANCEDRAW-: P1.4, P1.5, P1.6, U$1.3,-VIN, U$2.2, U$2.3
Routing:
- net 3.3V: track 0.00 -> 48.8 mm, vias 0 -> 1
- net 3.3VGROUND: track 0.00 -> 35.1 mm, vias 0 -> 1
- net BALANCEDRAW+: track 0.00 -> 8.38 mm
- added copper zone on layer 1, net 12V+
- added copper zone on layer 16, net 12V-
- added copper zone on layer 1, net 3.3V
- added copper zone on layer 16, net 3.3V
- added copper zone on layer 1, net 3.3VGROUND
- added copper zone on layer 16, net 3.3VGROUND
- added copper zone on layer 1, net BALANCEDRAW+
- added copper zone on layer 16, net BALANCEDRAW-
Other:
- board text added: "The Underwater Robotics Team Riptide -- Board Template"

Commit message: Added LEDs and resistors to converter board
Parts:
- added 12VLED, 3.3VLED, BALANCEDRAWLED: LTST-S270GKT, LTST-S270GKT:LTST-S270GKT
- added 12VR, 3.3VR, BALANCEDRAWR: 330, resistor:0204/7
Connections:
- new net 12VLED: 12VLED.ANODE, 12VR.1
- new net 3.3VLED: 3.3VLED.ANODE, 3.3VR.1
- new net BALANCEDRAWLED: BALANCEDRAWLED.ANODE, BALANCEDRAWR.2
- net 12V+: now also 12VR.2
- net 12V-: now also 12VLED.CATHODE
- net 3.3V: now also 3.3VR.2
- net 3.3VGROUND: now also 3.3VLED.CATHODE
- net BALANCEDRAW+: now also BALANCEDRAWR.1
- net BALANCEDRAW-: now also BALANCEDRAWLED.CATHODE
Changed lines of the file:
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@@
 <layer number="97" name="Info" color="7" fill="1" visible="no" active="no"/>
 <layer number="98" name="Guide" color="6" fill="1" visible="no" active="no"/>
+<layer number="99" name="SpiceOrder" color="5" fill="1" visible="no" active="no"/>
 </layers>
 <board>
@@
 <element name="U$1" library="12VCONV" package="12VCONV" value="12VCONV" x="21.844" y="49.276"/>
 <element name="U$2" library="3.3V Converter" package="3.3VCONV" value="3.3VCONV" x="66.802" y="16.51" rot="R90"/>
+<element name="3.3VLED" library="LTST-S270GKT" package="LTST-S270GKT" value="LTST-S270GKT" x="28.194" y="90.424"/>
+<element name="12VLED" library="LTST-S270GKT" package="LTST-S270GKT" value="LTST-S270GKT" x="80.772" y="89.408"/>
+<element name="BALANCEDRAWLED" library="LTST-S270GKT" package="LTST-S270GKT" value="LTST-S270GKT" x="16.51" y="89.662"/>
+<element name="3.3VR" library="resistor" library_urn="urn:adsk.eagle:library:348" package="0204/7" package3d_urn="urn:adsk.eagle:package:25945/1" value="330" x="35.56" y="85.344"/>
+<element name="BALANCEDRAWR" library="resistor" library_urn="urn:adsk.eagle:library:348" package="0204/7" package3d_urn="urn:adsk.eagle:package:25945/1" value="330" x="45.466" y="62.484"/>
+<element name="12VR" library="resistor" library_urn="urn:adsk.eagle:library:348" package="0204/7" package3d_urn="urn:adsk.eagle:package:25945/1" value="330" x="72.136" y="84.074"/>
 </elements>
 <signals>
@@
 <vertex x="47.752" y="101.6"/>
 </polygon>
+<contactref element="BALANCEDRAWR" pad="1"/>
 </signal>
 <signal name="BALANCEDRAW-">
@@
 <vertex x="47.752" y="101.6"/>
 </polygon>
+<contactref element="BALANCEDRAWLED" pad="CATHODE"/>
+<wire x1="25.4" y1="60.071" x2="15.51" y2="89.662" width="0" layer="19" extent="1-1"/>
 </signal>
 <signal name="12V-">
@@
 <vertex x="49.784" y="101.6"/>
 </polygon>
+<contactref element="12VLED" pad="CATHODE"/>
+<wire x1="76.2" y1="75.311" x2="79.772" y2="89.408" width="0" layer="19" extent="1-1"/>
 </signal>
 <signal name="3.3V">
@@
 <wire x1="25.908" y1="14.732" x2="18.542" y2="7.366" width="2.54" layer="1"/>
 <via x="19.304" y="6.858" extent="1-16" drill="0.55"/>
+<contactref element="3.3VR" pad="2"/>
+<wire x1="62.23" y1="19.05" x2="39.37" y2="85.344" width="0" layer="19" extent="1-1"/>
 </signal>
 <signal name="3.3VGROUND">
@@
 <wire x1="33.274" y1="12.446" x2="27.432" y2="6.604" width="2.54" layer="16"/>
 <via x="26.924" y="6.858" extent="1-16" drill="0.55"/>
+<contactref element="3.3VLED" pad="CATHODE"/>
+<wire x1="57.404" y1="19.05" x2="27.194" y2="90.424" width="0" layer="19" extent="1-1"/>
 </signal>
 <signal name="12V+">
@@
 <vertex x="49.784" y="101.6"/>
 </polygon>
+<contactref element="12VR" pad="2"/>
+</signal>
+<signal name="3.3VLED">
+<contactref element="3.3VR" pad="1"/>
+<contactref element="3.3VLED" pad="ANODE"/>
+<wire x1="31.75" y1="85.344" x2="29.194" y2="90.424" width="0" layer="19" extent="1-1"/>
+</signal>
+<signal name="BALANCEDRAWLED">
+<contactref element="BALANCEDRAWR" pad="2"/>
+<contactref element="BALANCEDRAWLED" pad="ANODE"/>
+<wire x1="17.51" y1="89.662" x2="49.276" y2="62.484" width="0" layer="19" extent="1-1"/>
+</signal>
+<signal name="12VLED">
+<contactref element="12VR" pad="1"/>
+<contactref element="12VLED" pad="ANODE"/>
+<wire x1="68.326" y1="84.074" x2="81.772" y2="89.408" width="0" layer="19" extent="1-1"/>
 </signal>
 </signals>
@@
 which will not be processed correctly with this version.
 </note>
+<note version="8.2" severity="warning">
+Since Version 8.2, EAGLE supports online libraries. The ids
+of those online libraries will not be understood (or retained)
+with this version.
+</note>
+<note version="8.3" severity="warning">
+Since Version 8.3, EAGLE supports URNs for individual library
+assets (packages, symbols, and devices). The URNs of those assets
+will not be understood (or retained) with this version.
+</note>
+<note version="8.3" severity="warning">
+Since Version 8.3, EAGLE supports the association of 3D packages
+with devices in libraries, schematics, and board files. Those 3D
+packages will not be understood (or retained) with this version.
+</note>
 </compatibility>

Commit message: Jennifer's edits on the converter board
Parts:
- moved BALANCEDRAWR 44.4 mm to (11.2, 90.7)
- moved 3.3VLED 30.3 mm to (57.7, 97.5)
- moved 12VR 20.4 mm to (91.4, 90.7)
- moved 3.3VR 20.0 mm to (54.9, 90.7), turned to 180 degrees
- moved 12VLED 10.6 mm to (86.6, 98.3)
- moved BALANCEDRAWLED 8.27 mm to (14.0, 97.5)
Routing:
- net 3.3VGROUND: track 35.1 -> 121.3 mm, vias 1 -> 2
- net 3.3V: track 48.8 -> 129.0 mm
- net BALANCEDRAWLED: track 0.00 -> 6.86 mm
- net 3.3VLED: track 0.00 -> 6.86 mm
- net BALANCEDRAW-: track 0.00 -> 3.12 mm, vias 0 -> 1
- removed copper zone on layer 1, net 12V+
- removed copper zone on layer 16, net 12V-
Changed lines of the file:
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@@
 <?xml version="1.0" encoding="utf-8"?>
 <!DOCTYPE eagle SYSTEM "eagle.dtd">
-<eagle version="8.3.1">
+<eagle version="8.4.0">
 <drawing>
 <settings>
@@
 <param name="dpMaxLengthDifference" value="10mm"/>
 <param name="dpGapFactor" value="2.5"/>
-<param name="checkGrid" value="0"/>
-<param name="checkAngle" value="0"/>
 <param name="checkFont" value="1"/>
 <param name="checkRestrict" value="1"/>
+<param name="checkStop" value="0"/>
 <param name="useDiameter" value="13"/>
 <param name="maxErrors" value="50"/>
@@
 <element name="U$1" library="12VCONV" package="12VCONV" value="12VCONV" x="21.844" y="49.276"/>
 <element name="U$2" library="3.3V Converter" package="3.3VCONV" value="3.3VCONV" x="66.802" y="16.51" rot="R90"/>
-<element name="3.3VLED" library="LTST-S270GKT" package="LTST-S270GKT" value="LTST-S270GKT" x="28.194" y="90.424"/>
-<element name="12VLED" library="LTST-S270GKT" package="LTST-S270GKT" value="LTST-S270GKT" x="80.772" y="89.408"/>
-<element name="BALANCEDRAWLED" library="LTST-S270GKT" package="LTST-S270GKT" value="LTST-S270GKT" x="16.51" y="89.662"/>
-<element name="3.3VR" library="resistor" library_urn="urn:adsk.eagle:library:348" package="0204/7" package3d_urn="urn:adsk.eagle:package:25945/1" value="330" x="35.56" y="85.344"/>
-<element name="BALANCEDRAWR" library="resistor" library_urn="urn:adsk.eagle:library:348" package="0204/7" package3d_urn="urn:adsk.eagle:package:25945/1" value="330" x="45.466" y="62.484"/>
-<element name="12VR" library="resistor" library_urn="urn:adsk.eagle:library:348" package="0204/7" package3d_urn="urn:adsk.eagle:package:25945/1" value="330" x="72.136" y="84.074"/>
+<element name="3.3VLED" library="LTST-S270GKT" package="LTST-S270GKT" value="LTST-S270GKT" x="57.658" y="97.536"/>
+<element name="12VLED" library="LTST-S270GKT" package="LTST-S270GKT" value="LTST-S270GKT" x="86.614" y="98.298"/>
+<element name="BALANCEDRAWLED" library="LTST-S270GKT" package="LTST-S270GKT" value="LTST-S270GKT" x="13.97" y="97.536"/>
+<element name="3.3VR" library="resistor" library_urn="urn:adsk.eagle:library:348" package="0204/7" package3d_urn="urn:adsk.eagle:package:25945/1" value="330" x="54.864" y="90.678" rot="R180"/>
+<element name="BALANCEDRAWR" library="resistor" library_urn="urn:adsk.eagle:library:348" package="0204/7" package3d_urn="urn:adsk.eagle:package:25945/1" value="330" x="11.176" y="90.678"/>
+<element name="12VR" library="resistor" library_urn="urn:adsk.eagle:library:348" package="0204/7" package3d_urn="urn:adsk.eagle:package:25945/1" value="330" x="91.44" y="90.678"/>
 </elements>
 <signals>
@@
 </polygon>
 <contactref element="BALANCEDRAWLED" pad="CATHODE"/>
-<wire x1="25.4" y1="60.071" x2="15.51" y2="89.662" width="0" layer="19" extent="1-1"/>
+<via x="10.414" y="96.012" extent="1-16" drill="0.35"/>
+<wire x1="10.414" y1="96.012" x2="11.192" y2="96.012" width="0.1524" layer="1"/>
+<wire x1="11.192" y1="96.012" x2="12.97" y2="97.536" width="0.1524" layer="1"/>
 </signal>
 <signal name="12V-">
@@
 <contactref element="P2" pad="5"/>
 <contactref element="U$1" pad="4,-VOUT"/>
-<polygon width="0.2032" layer="16">
-<vertex x="101.6" y="101.6"/>
-<vertex x="101.6" y="26.67"/>
-<vertex x="98.298" y="23.368"/>
-<vertex x="76.2" y="23.368"/>
-<vertex x="52.578" y="23.368"/>
-<vertex x="49.784" y="26.162"/>
-<vertex x="49.784" y="101.6"/>
-</polygon>
 <contactref element="12VLED" pad="CATHODE"/>
-<wire x1="76.2" y1="75.311" x2="79.772" y2="89.408" width="0" layer="19" extent="1-1"/>
+<wire x1="76.2" y1="75.311" x2="85.614" y2="98.298" width="0" layer="19" extent="1-1"/>
+<wire x1="80.2132" y1="39.8785" x2="76.2" y2="75.311" width="0" layer="19" extent="1-1"/>
+<wire x1="80.2132" y1="35.6875" x2="80.2132" y2="39.8785" width="0" layer="19" extent="1-1"/>
+<wire x1="80.2132" y1="31.4965" x2="80.2132" y2="35.6875" width="0" layer="19" extent="1-1"/>
 </signal>
 <signal name="3.3V">
@@
 <vertex x="17.018" y="8.382"/>
 </polygon>
-<wire x1="62.484" y1="19.05" x2="62.23" y2="19.05" width="2.54" layer="1"/>
+<wire x1="62.23" y1="19.05" x2="62.484" y2="19.05" width="2.54" layer="1"/>
 <wire x1="62.23" y1="19.05" x2="57.912" y2="14.732" width="2.54" layer="1"/>
 <wire x1="57.912" y1="14.732" x2="25.908" y2="14.732" width="2.54" layer="1"/>
@@
 <via x="19.304" y="6.858" extent="1-16" drill="0.55"/>
 <contactref element="3.3VR" pad="2"/>
-<wire x1="62.23" y1="19.05" x2="39.37" y2="85.344" width="0" layer="19" extent="1-1"/>
+<wire x1="62.484" y1="19.05" x2="59.436" y2="19.05" width="0.1524" layer="1"/>
+<wire x1="59.436" y1="19.05" x2="48.514" y2="29.972" width="0.1524" layer="1"/>
+<wire x1="48.514" y1="29.972" x2="48.514" y2="88.138" width="0.1524" layer="1"/>
+<wire x1="48.514" y1="88.138" x2="51.054" y2="90.678" width="0.1524" layer="1"/>
 </signal>
 <signal name="3.3VGROUND">
@@
 <vertex x="29.21" y="8.382"/>
 </polygon>
-<wire x1="57.404" y1="19.05" x2="50.8" y2="12.446" width="2.54" layer="16"/>
+<wire x1="50.8" y1="12.446" x2="57.404" y2="19.05" width="2.54" layer="16"/>
 <wire x1="50.8" y1="12.446" x2="33.274" y2="12.446" width="2.54" layer="16"/>
 <wire x1="33.274" y1="12.446" x2="27.432" y2="6.604" width="2.54" layer="16"/>
 <via x="26.924" y="6.858" extent="1-16" drill="0.55"/>
 <contactref element="3.3VLED" pad="CATHODE"/>
-<wire x1="57.404" y1="19.05" x2="27.194" y2="90.424" width="0" layer="19" extent="1-1"/>
+<wire x1="57.404" y1="19.05" x2="48.514" y2="27.94" width="0.1524" layer="16"/>
+<via x="54.356" y="96.266" extent="1-16" drill="0.35"/>
+<wire x1="48.514" y1="90.424" x2="54.356" y2="96.266" width="0.1524" layer="16"/>
+<wire x1="48.514" y1="27.94" x2="48.514" y2="90.424" width="0.1524" layer="16"/>
+<wire x1="54.356" y1="96.266" x2="55.626" y2="97.536" width="0.1524" layer="1"/>
+<wire x1="55.626" y1="97.536" x2="56.658" y2="97.536" width="0.1524" layer="1"/>
 </signal>
 <signal name="12V+">
@@
 <contactref element="P2" pad="2"/>
 <contactref element="U$1" pad="8,+VOUT"/>
-<polygon width="0.2032" layer="1">
-<vertex x="101.6" y="101.6"/>
-<vertex x="101.6" y="25.4"/>
-<vertex x="99.568" y="23.368"/>
-<vertex x="52.578" y="23.368"/>
-<vertex x="49.784" y="26.162"/>
-<vertex x="49.784" y="101.6"/>
-</polygon>
 <contactref element="12VR" pad="2"/>
+<wire x1="76.2" y1="60.071" x2="95.25" y2="90.678" width="0" layer="19" extent="1-1"/>
+<wire x1="85.725" y1="39.8785" x2="76.2" y2="60.071" width="0" layer="19" extent="1-1"/>
+<wire x1="85.725" y1="35.6875" x2="85.725" y2="39.8785" width="0" layer="19" extent="1-1"/>
+<wire x1="85.725" y1="31.4965" x2="85.725" y2="35.6875" width="0" layer="19" extent="1-1"/>
 </signal>
 <signal name="3.3VLED">
 <contactref element="3.3VR" pad="1"/>
 <contactref element="3.3VLED" pad="ANODE"/>
-<wire x1="31.75" y1="85.344" x2="29.194" y2="90.424" width="0" layer="19" extent="1-1"/>
+<wire x1="58.658" y1="97.536" x2="58.658" y2="90.694" width="0.1524" layer="1"/>
+<wire x1="58.658" y1="90.694" x2="58.674" y2="90.678" width="0.1524" layer="1"/>
 </signal>
 <signal name="BALANCEDRAWLED">
 <contactref element="BALANCEDRAWR" pad="2"/>
 <contactref element="BALANCEDRAWLED" pad="ANODE"/>
-<wire x1="17.51" y1="89.662" x2="49.276" y2="62.484" width="0" layer="19" extent="1-1"/>
+<wire x1="14.986" y1="90.678" x2="14.986" y2="97.52" width="0.1524" layer="1"/>
+<wire x1="14.986" y1="97.52" x2="14.97" y2="97.536" width="0.1524" layer="1"/>
 </signal>
 <signal name="12VLED">
 <contactref element="12VR" pad="1"/>
 <contactref element="12VLED" pad="ANODE"/>
-<wire x1="68.326" y1="84.074" x2="81.772" y2="89.408" width="0" layer="19" extent="1-1"/>
+<wire x1="87.63" y1="90.678" x2="87.614" y2="98.298" width="0" layer="19" extent="1-1"/>
 </signal>
 </signals>
