File: Converter Board/ConverterBoardRev2.brd (EAGLE design)
At the start: 101.6 x 101.6 mm, 18 parts

Commit message: Additions to Rev2, added sensors to schematic
Parts:
- added U$4, U$5: CURRENTSENS, CurrentSensor:CURRENTSENS
- added U$6: HUMIDITYSENSOR, HumiditySensor:HUMIDITYSENSOR
- added U$7: TEMPSENS, TemperatureSensor:TEMPSENS
- moved U$2 6.61 mm to (57.1, 18.0)
- renumbered 3.3VGROUNDTP to 3.3V-TP, 3.3VTP to 3.3V+TP
Connections:
- net N$5 renamed 3.3VLED
- removed net 3.3V: 3.3VLED.CATHODE, U$2.14, U$3.3.3VP1, U$3.3.3VP2, U$3.3.3VP3, U$3.3.3V_4, U$3.3.3V_5, U$3.3.3V_6
- removed net 3.3VGROUND: 3.3VR.2, U$2.16, U$3.GND1, U$3.GND2, U$3.GND3
- removed net N$2: 12V+TP.TP, 12VOUT.4, 12VOUT.5, 12VOUT.6, 12VOUT1.4, 12VOUT1.5, 12VOUT1.6, 12VR.1, U$1.8,+VOUT
- removed net N$3: 12V-TP.TP, 12VLED.CATHODE, 12VOUT.1, 12VOUT.2, 12VOUT.3, 12VOUT1.1, 12VOUT1.2, 12VOUT1.3, U$1.4,-VOUT
- new net 12V+: 12V+TP.TP, 12VOUT.4, 12VOUT.5, 12VOUT.6, 12VOUT1.4, 12VOUT1.5, 12VOUT1.6, 12VR.1, U$1.8,+VOUT, U$4.8,VCC
- new net 12V-: 12V-TP.TP, 12VLED.CATHODE, 12VOUT.1, 12VOUT.2, 12VOUT.3, 12VOUT1.1, 12VOUT1.2, 12VOUT1.3, U$1.4,-VOUT, U$4.5,GND
- new net 3.3V+: 3.3V+TP.TP, 3.3VLED.CATHODE, U$2.14, U$3.3.3VP1, U$3.3.3VP2, U$3.3.3VP3, U$3.3.3V_4, U$3.3.3V_5, U$3.3.3V_6, U$4.1,IP+, U$4.2,IP+, U$5.1,IP+, U$5.2,IP+, U$5.8,VCC, U$6.+VE, U$7.1,VDD
- new net 3.3V-: 3.3V-TP.TP, 3.3VR.2, U$2.16, U$3.GND1, U$3.GND2, U$3.GND3, U$4.3,IP-, U$4.4,IP-, U$5.3,IP-, U$5.4,IP-, U$5.5,GND, U$6.-VE, U$7.3,GND
- net BALANCED-: now also U$2.1
Routing:
- added copper zone on layer 1, net 3.3V+
- added copper zone on layer 16, net 3.3V+
- added copper zone on layer 1, net 3.3V-
- added copper zone on layer 16, net 3.3V-
- removed copper zone on layer 1, net 3.3V
- removed copper zone on layer 16, net 3.3V
- removed copper zone on layer 1, net 3.3VGROUND
- removed copper zone on layer 16, net 3.3VGROUND
