File: Converter Board/ConverterBoardRev2 (3).brd (EAGLE design)
At the start: 101.6 x 101.3 mm, 32 parts

Commit message: General cleanup (salutes) of the converter and copro eagle files
Parts:
- removed 12VOUT, 12VOUT1: 39-30-06?, con-molex-mini-fit:39-30-?06?
- removed U$4, U$5: CURRENTSENS, CurrentSensor:CURRENTSENS
- removed U$7: TEMPSENS, TemperatureSensor:TEMPSENS
- added 12VCUR, 3V3CUR: CURRENTSENS, CurrentSensor:CURRENTSENS
- added DIAMOND: 43045-08, con-molex-micro-fit:43045-08
- added NUC, PNUEMATICS: 39-30-02?, con-molex-mini-fit:39-30-?02?
- added TEMPSENSE: 2SC458, transistor:TO92-ECB
- moved U$8 21.5 mm to (74.7, 20.8)
- moved U$6 20.1 mm to (70.9, 28.2)
- moved R1 15.3 mm to (62.2, 20.6)
- moved R3 14.0 mm to (65.0, 20.6)
- moved R6 10.7 mm to (71.6, 38.6), turned to 90 degrees
- moved 12VR 8.52 mm to (83.6, 91.2), turned to 0 degrees
- moved R7 8.27 mm to (86.4, 47.0)
- moved 3.3VR 7.97 mm to (53.1, 90.7), turned to 180 degrees
- moved BALANCEDR 7.64 mm to (11.2, 90.9), turned to 180 degrees
- moved R8 7.54 mm to (92.7, 43.2), turned to 0 degrees
- moved R5 5.93 mm to (68.6, 38.6), turned to 90 degrees
- moved R4 1.27 mm to (58.2, 20.6)
- moved R2 1.14 mm to (55.6, 20.6)
Connections:
- removed net 12V+: 12VOUT.4, 12VOUT.5, 12VOUT.6, 12VOUT1.4, 12VOUT1.5, 12VOUT1.6, 12VR.1, U$1.8,+VOUT, U$4.8,VCC
- removed net 12V-: 12V-TP.TP, 12VLED.CATHODE, 12VOUT.1, 12VOUT.2, 12VOUT.3, 12VOUT1.1, 12VOUT1.2, 12VOUT1.3, R8.2, U$1.4,-VOUT, U$4.5,GND
- removed net N$4: U$3.GND_4, U$3.GND_5, U$3.GND_6
- removed net N$5: R7.1
- removed net NTC: U$2.11, U$2.9
- new net 12VGND: 12V-TP.TP, 12VLED.CATHODE, DIAMOND.5, DIAMOND.6, DIAMOND.7, DIAMOND.8, NUC.2, PNUEMATICS.2, R8.2, U$1.4,-VOUT
- new net 12VMON: 12VCUR.3,IP-, 12VCUR.4,IP-, 12VR.1, DIAMOND.1, DIAMOND.2, DIAMOND.3, DIAMOND.4, NUC.1, PNUEMATICS.1, R7.1
- new net 12VUNMON: 12VCUR.1,IP+, 12VCUR.2,IP+, U$1.8,+VOUT
- new net 3.3VBKPLN: 3V3CUR.3,IP-, 3V3CUR.4,IP-, U$3.3.3VP1, U$3.3.3VP2, U$3.3.3VP3, U$3.3.3V_4, U$3.3.3V_5, U$3.3.3V_6
- net 12IDATA: now also 12VCUR.7,VIOUT; no longer U$4.7,VIOUT
- net 3.3IDATA: now also 3V3CUR.7,VIOUT; no longer U$5.7,VIOUT
- net 3.3V+: now also 12VCUR.8,VCC, 3V3CUR.1,IP+, 3V3CUR.2,IP+, 3V3CUR.8,VCC, TEMPSENSE.E, U$8.VREF; no longer R5.2, U$3.3.3VP1, U$3.3.3VP2, U$3.3.3VP3, U$3.3.3V_4, U$3.3.3V_5, U$3.3.3V_6, U$4.1,IP+, U$4.2,IP+, U$5.1,IP+, U$5.2,IP+, U$5.8,VCC, U$7.1,VDD
- net 3.3V-: now also 12VCUR.5,GND, 3V3CUR.5,GND, R5.2, TEMPSENSE.B, U$3.GND_4, U$3.GND_5, U$3.GND_6; no longer U$4.3,IP-, U$4.4,IP-, U$5.3,IP-, U$5.4,IP-, U$5.5,GND, U$7.3,GND
- net HUMIDITYDATA: now also U$8.IN1; no longer U$8.IN2
- net TEMPDATA: now also TEMPSENSE.C, U$8.IN2; no longer U$7.2,OUT, U$8.IN3
Routing:
- net 3.3V+: track 83.8 -> 17.3 mm, vias 1 -> 0
- net 12VMON: track 0.00 -> 60.7 mm
- net TEMPDATA: track 27.6 -> 67.8 mm
- net 3.3VBKPLN: track 0.00 -> 32.2 mm, vias 0 -> 1
- net 3.3IDATA: track 35.7 -> 67.7 mm, vias 0 -> 2
- net 3.3V-: track 102.7 -> 71.6 mm, vias 4 -> 6
- net A1: track 3.81 -> 27.2 mm
- net 3.3VDATA: track 32.6 -> 15.5 mm
- net A0: track 4.06 -> 19.2 mm
- net 12VUNMON: track 0.00 -> 15.0 mm
- net 12VGND: track 0.00 -> 12.9 mm, vias 0 -> 1
- net SDA: track 27.9 -> 16.7 mm
- net 12VDATA: track 21.2 -> 31.6 mm, vias 0 -> 1
- net SCL: track 25.5 -> 17.5 mm
- net NTC: track 5.08 -> 0.00 mm
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- added copper zone on layer 16, net 12VGND
- added copper zone on layer 1, net 12VMON
- added copper zone on layer 1, net 12VUNMON
- added copper zone on layer 1, net 3.3VBKPLN
- added copper zone on layer 16, net 3.3VBKPLN
- removed copper zone on layer 1, net 12V+
- removed copper zone on layer 16, net 12V-
- removed copper zone on layer 16, net 3.3V+
Other:
- board text added: "A0"
- board text added: "A1"
- board text added: "The Ohio State Univerity Center for Automotive Research The Underwater Robotics Team Converter Board -- Rev. 2.0"
- board text removed: "3.3 V GROUND"
- board text removed: "3.3 V OUT"
- board text removed: "The Ohio State Univerity Center for Automotive Research"
- board text removed: "The Underwater Robotics Team Riptide -- Converter Board"
