File: Converter Board/ConverterBoardRev2 (3).sch (EAGLE design)
At the start: 32 parts

Commit message: General cleanup (salutes) of the converter and copro eagle files
Parts:
- removed 12VOUT, 12VOUT1: 39-30-06, con-molex-mini-fit:39-30-06
- removed U$4: CURRENTSENS, CurrentSensor:CURRENTSENS
- removed U$7: TEMPSENS, TemperatureSensor:TEMPSENS
- added 12VCUR: CURRENTSENS, CurrentSensor:CURRENTSENS
- added DIAMOND: 43045-08, con-molex-micro-fit:43045-08
- added NUC, PNUEMATICS: 39-30-02, con-molex-mini-fit:39-30-02
- added TEMPSENSE: 2SC458, transistor:2SC458
- renumbered U$5 to 3V3CUR
Connections:
- removed net 12V+: 12VOUT.4, 12VOUT.5, 12VOUT.6, 12VOUT1.4, 12VOUT1.5, 12VOUT1.6, 12VR.1, U$1.8,+VOUT, U$4.8,VCC
- removed net 12V-: 12V-TP.TP, 12VLED.C, 12VOUT.1, 12VOUT.2, 12VOUT.3, 12VOUT1.1, 12VOUT1.2, 12VOUT1.3, R8.2, U$1.4,-VOUT, U$4.5,GND
- removed net N$4: U$3.GND_4, U$3.GND_5, U$3.GND_6
- removed net N$5: R7.1
- removed net NTC: U$2.11,NTC, U$2.9,NTC
- new net 12VGND: 12V-TP.TP, 12VLED.C, DIAMOND.5, DIAMOND.6, DIAMOND.7, DIAMOND.8, NUC.2, PNUEMATICS.2, R8.2, U$1.4,-VOUT
- new net 12VMON: 12VCUR.3,IP-, 12VCUR.4,IP-, 12VR.1, DIAMOND.1, DIAMOND.2, DIAMOND.3, DIAMOND.4, NUC.1, PNUEMATICS.1, R7.1
- new net 12VUNMON: 12VCUR.1,IP+, 12VCUR.2,IP+, U$1.8,+VOUT
- new net 3.3VBKPLN: 3V3CUR.3,IP-, 3V3CUR.4,IP-, U$3.3.3V_1, U$3.3.3V_2, U$3.3.3V_3, U$3.3.3V_4, U$3.3.3V_5, U$3.3.3V_6
- net 12IDATA: now also 12VCUR.7,VIOUT; no longer U$4.7,VIOUT
- net 3.3V+: now also 12VCUR.8,VCC, TEMPSENSE.E, U$8.VREF; no longer R5.2, U$3.3.3V_1, U$3.3.3V_2, U$3.3.3V_3, U$3.3.3V_4, U$3.3.3V_5, U$3.3.3V_6, U$4.1,IP+, U$4.2,IP+, U$7.1,VDD
- net 3.3V-: now also 12VCUR.5,GND, R5.2, TEMPSENSE.B, U$3.GND_4, U$3.GND_5, U$3.GND_6; no longer 3V3CUR.3,IP-, 3V3CUR.4,IP-, U$4.3,IP-, U$4.4,IP-, U$7.3,GND
- net HUMIDITYDATA: now also U$8.IN1; no longer U$8.IN2
- net TEMPDATA: now also TEMPSENSE.C, U$8.IN2; no longer U$7.2,OUT, U$8.IN3
Other:
- note added: "Please don't judge me, it made the board package easier."
