File: Converter Board/ConverterBoard.sch (EAGLE design)
At the start: 17 parts

Commit message: Adjustments to the converter board
Parts:
- BALANCEDRAWR: value 330 -> 700
Changed lines of the file:
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@@
 <part name="BALANCEDRAWLED" library="LTST-S270GKT" deviceset="LTST-S270GKT" device=""/>
 <part name="3.3VR" library="resistor" library_urn="urn:adsk.eagle:library:348" deviceset="R-US_" device="0204/7" package3d_urn="urn:adsk.eagle:package:25945/1" value="330"/>
-<part name="BALANCEDRAWR" library="resistor" library_urn="urn:adsk.eagle:library:348" deviceset="R-US_" device="0204/7" package3d_urn="urn:adsk.eagle:package:25945/1" value="330"/>
+<part name="BALANCEDRAWR" library="resistor" library_urn="urn:adsk.eagle:library:348" deviceset="R-US_" device="0204/7" package3d_urn="urn:adsk.eagle:package:25945/1" value="700"/>
 <part name="12VR" library="resistor" library_urn="urn:adsk.eagle:library:348" deviceset="R-US_" device="0204/7" package3d_urn="urn:adsk.eagle:package:25945/1" value="330"/>
 <part name="3.3VTP" library="testpad" library_urn="urn:adsk.eagle:library:385" deviceset="PTR1" device="B1,27" package3d_urn="urn:adsk.eagle:package:27944/1"/>

Commit message: Fixed 3.3V converter Added extra connector Updated board with new parts
Parts:
- added 12VOUT1: 39-30-06, con-molex-mini-fit:39-30-06
Connections:
- net 12V+: now also 12VOUT1.1, 12VOUT1.2, 12VOUT1.3
- net 12V-: now also 12VOUT1.4, 12VOUT1.5, 12VOUT1.6
Changed lines of the file:
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@@
 <part name="12VOUT" library="con-molex-mini-fit" deviceset="39-30-?06?" device=""/>
 <part name="U$1" library="12VCONV" deviceset="12VCONV" device=""/>
-<part name="U$2" library="3.3V Converter" deviceset="3.3VCONV" device=""/>
 <part name="3.3VLED" library="LTST-S270GKT" deviceset="LTST-S270GKT" device=""/>
 <part name="12VLED" library="LTST-S270GKT" deviceset="LTST-S270GKT" device=""/>
@@
 <part name="BALANCEDRAW-TP" library="testpad" library_urn="urn:adsk.eagle:library:385" deviceset="PTR1" device="B1,27" package3d_urn="urn:adsk.eagle:package:27944/1"/>
 <part name="3.3VGROUNDTP" library="testpad" library_urn="urn:adsk.eagle:library:385" deviceset="PTR1" device="B1,27" package3d_urn="urn:adsk.eagle:package:27944/1"/>
+<part name="U$2" library="3.3V Converter" deviceset="3.3VCONV" device=""/>
+<part name="12VOUT1" library="con-molex-mini-fit" deviceset="39-30-?06?" device=""/>
 </parts>
 <sheets>
@@
 <instance part="12VOUT" gate="G$1" x="139.7" y="78.74"/>
 <instance part="U$1" gate="G$1" x="0" y="58.42"/>
-<instance part="U$2" gate="G$1" x="0" y="7.62"/>
 <instance part="3.3VLED" gate="G$1" x="-20.32" y="-2.54"/>
 <instance part="12VLED" gate="G$1" x="121.92" y="88.9"/>
@@
 <instance part="BALANCEDRAW-TP" gate="G$1" x="-20.32" y="71.12"/>
 <instance part="3.3VGROUNDTP" gate="G$1" x="10.16" y="-10.16" rot="R270"/>
+<instance part="U$2" gate="G$1" x="7.62" y="7.62"/>
+<instance part="12VOUT1" gate="G$1" x="139.7" y="48.26"/>
 </instances>
 <busses>
@@
 <junction x="-5.08" y="68.58"/>
 <wire x1="-5.08" y1="68.58" x2="-15.24" y2="68.58" width="0.1524" layer="91"/>
-<wire x1="-5.08" y1="35.56" x2="-5.08" y2="33.02" width="0.1524" layer="91"/>
-<wire x1="-5.08" y1="35.56" x2="-12.7" y2="35.56" width="0.1524" layer="91"/>
+<wire x1="-2.54" y1="35.56" x2="-15.24" y2="35.56" width="0.1524" layer="91"/>
 <wire x1="-15.24" y1="35.56" x2="-38.1" y2="35.56" width="0.1524" layer="91"/>
 <wire x1="-38.1" y1="35.56" x2="-38.1" y2="48.26" width="0.1524" layer="91"/>
@@
 <wire x1="-38.1" y1="48.26" x2="-53.34" y2="48.26" width="0.1524" layer="91"/>
 <junction x="-53.34" y="48.26"/>
-<pinref part="U$2" gate="G$1" pin="22,+VIN"/>
-<pinref part="U$2" gate="G$1" pin="23,+VIN"/>
-<junction x="-5.08" y="35.56"/>
 <pinref part="BALANCEDRAWR" gate="G$1" pin="1"/>
 <wire x1="-53.34" y1="55.88" x2="-53.34" y2="63.5" width="0.1524" layer="91"/>
@@
 <wire x1="-15.24" y1="68.58" x2="-15.24" y2="50.8" width="0.1524" layer="91"/>
 <wire x1="-15.24" y1="50.8" x2="-15.24" y2="35.56" width="0.1524" layer="91"/>
-<wire x1="-15.24" y1="35.56" x2="-12.7" y2="35.56" width="0.1524" layer="91"/>
 <pinref part="BALANCEDRAW+TP" gate="G$1" pin="TP"/>
 <junction x="-15.24" y="50.8"/>
+<wire x1="-2.54" y1="35.56" x2="-2.54" y2="45.72" width="0.1524" layer="91"/>
+<pinref part="U$2" gate="G$1" pin="23,+VIN"/>
+<wire x1="-2.54" y1="45.72" x2="33.02" y2="45.72" width="0.1524" layer="91"/>
+<wire x1="33.02" y1="45.72" x2="33.02" y2="35.56" width="0.1524" layer="91"/>
+<pinref part="U$2" gate="G$1" pin="22,+VIN"/>
+<wire x1="33.02" y1="33.02" x2="33.02" y2="35.56" width="0.1524" layer="91"/>
+<junction x="33.02" y="35.56"/>
+<junction x="-15.24" y="35.56"/>
 </segment>
 </net>
 <net name="BALANCEDRAW-" class="0">
 <segment>
-<wire x1="25.4" y1="33.02" x2="25.4" y2="35.56" width="0.1524" layer="91"/>
-<wire x1="25.4" y1="35.56" x2="27.94" y2="35.56" width="0.1524" layer="91"/>
-<wire x1="27.94" y1="35.56" x2="27.94" y2="43.18" width="0.1524" layer="91"/>
 <pinref part="BALANCEDRAWIN" gate="G$1" pin="6"/>
 <pinref part="BALANCEDRAWIN" gate="G$1" pin="5"/>
@@
 <wire x1="-53.34" y1="43.18" x2="-40.64" y2="43.18" width="0.1524" layer="91"/>
 <wire x1="-40.64" y1="43.18" x2="-20.32" y2="43.18" width="0.1524" layer="91"/>
-<wire x1="-20.32" y1="43.18" x2="27.94" y2="43.18" width="0.1524" layer="91"/>
 <wire x1="-5.08" y1="88.9" x2="-20.32" y2="88.9" width="0.1524" layer="91"/>
 <wire x1="-20.32" y1="88.9" x2="-20.32" y2="73.66" width="0.1524" layer="91"/>
-<junction x="-20.32" y="43.18"/>
 <pinref part="U$1" gate="G$1" pin="3,-VIN"/>
-<pinref part="U$2" gate="G$1" pin="2,-VIN"/>
-<junction x="25.4" y="35.56"/>
-<pinref part="U$2" gate="G$1" pin="3,-VIN"/>
 <pinref part="BALANCEDRAWLED" gate="G$1" pin="C"/>
 <wire x1="-20.32" y1="73.66" x2="-20.32" y2="43.18" width="0.1524" layer="91"/>
@@
 <pinref part="BALANCEDRAW-TP" gate="G$1" pin="TP"/>
 <junction x="-20.32" y="73.66"/>
+<wire x1="-20.32" y1="43.18" x2="0" y2="43.18" width="0.1524" layer="91"/>
+<wire x1="0" y1="43.18" x2="0" y2="35.56" width="0.1524" layer="91"/>
+<junction x="-20.32" y="43.18"/>
+<pinref part="U$2" gate="G$1" pin="2,-VIN"/>
+<wire x1="0" y1="35.56" x2="2.54" y2="35.56" width="0.1524" layer="91"/>
+<pinref part="U$2" gate="G$1" pin="3,-VIN"/>
+<wire x1="2.54" y1="33.02" x2="2.54" y2="35.56" width="0.1524" layer="91"/>
+<junction x="2.54" y="35.56"/>
 </segment>
 </net>
@@
 <wire x1="121.92" y1="76.2" x2="99.06" y2="76.2" width="0.1524" layer="91"/>
 <junction x="121.92" y="76.2"/>
+<wire x1="132.08" y1="68.58" x2="129.54" y2="68.58" width="0.1524" layer="91"/>
+<junction x="132.08" y="68.58"/>
+<pinref part="12VOUT1" gate="G$1" pin="4"/>
+<wire x1="147.32" y1="45.72" x2="147.32" y2="48.26" width="0.1524" layer="91"/>
+<pinref part="12VOUT1" gate="G$1" pin="6"/>
+<pinref part="12VOUT1" gate="G$1" pin="5"/>
+<wire x1="132.08" y1="45.72" x2="132.08" y2="38.1" width="0.1524" layer="91"/>
+<wire x1="132.08" y1="38.1" x2="147.32" y2="38.1" width="0.1524" layer="91"/>
+<wire x1="147.32" y1="38.1" x2="147.32" y2="45.72" width="0.1524" layer="91"/>
+<junction x="147.32" y="45.72"/>
+<wire x1="129.54" y1="68.58" x2="129.54" y2="45.72" width="0.1524" layer="91"/>
+<wire x1="129.54" y1="45.72" x2="132.08" y2="45.72" width="0.1524" layer="91"/>
+<junction x="132.08" y="45.72"/>
 </segment>
 </net>
 <net name="3.3V" class="0">
 <segment>
-<pinref part="U$2" gate="G$1" pin="14,+VOUT"/>
-<wire x1="-5.08" y1="12.7" x2="-5.08" y2="5.08" width="0.1524" layer="91"/>
 <pinref part="3.3VR" gate="G$1" pin="2"/>
 <wire x1="-10.16" y1="5.08" x2="-5.08" y2="5.08" width="0.1524" layer="91"/>
@@
 <wire x1="-5.08" y1="2.54" x2="-5.08" y2="-15.24" width="0.1524" layer="91"/>
 <junction x="-5.08" y="2.54"/>
+<pinref part="U$2" gate="G$1" pin="14,+VOUT"/>
+<wire x1="-5.08" y1="5.08" x2="33.02" y2="5.08" width="0.1524" layer="91"/>
+<wire x1="33.02" y1="5.08" x2="33.02" y2="12.7" width="0.1524" layer="91"/>
 </segment>
 </net>
@@
 <wire x1="30.48" y1="-15.24" x2="25.4" y2="-15.24" width="0.1524" layer="91"/>
 <wire x1="25.4" y1="-15.24" x2="20.32" y2="-15.24" width="0.1524" layer="91"/>
-<wire x1="-5.08" y1="15.24" x2="-7.62" y2="15.24" width="0.1524" layer="91"/>
-<wire x1="-7.62" y1="15.24" x2="-7.62" y2="-7.62" width="0.1524" layer="91"/>
+<wire x1="-7.62" y1="2.54" x2="-7.62" y2="-7.62" width="0.1524" layer="91"/>
 <wire x1="-7.62" y1="-7.62" x2="-7.62" y2="-10.16" width="0.1524" layer="91"/>
 <wire x1="-7.62" y1="-10.16" x2="12.7" y2="-10.16" width="0.1524" layer="91"/>
@@
 <junction x="25.4" y="-15.24"/>
 <junction x="30.48" y="-15.24"/>
-<pinref part="U$2" gate="G$1" pin="16,-VOUT"/>
 <pinref part="3.3VLED" gate="G$1" pin="C"/>
 <wire x1="-20.32" y1="-7.62" x2="-7.62" y2="-7.62" width="0.1524" layer="91"/>
@@
 <pinref part="3.3VGROUNDTP" gate="G$1" pin="TP"/>
 <junction x="12.7" y="-10.16"/>
+<wire x1="-7.62" y1="2.54" x2="35.56" y2="2.54" width="0.1524" layer="91"/>
+<wire x1="35.56" y1="2.54" x2="35.56" y2="15.24" width="0.1524" layer="91"/>
+<pinref part="U$2" gate="G$1" pin="16,-VOUT"/>
+<wire x1="35.56" y1="15.24" x2="33.02" y2="15.24" width="0.1524" layer="91"/>
 </segment>
 </net>
@@
 <junction x="132.08" y="78.74"/>
 <wire x1="93.98" y1="81.28" x2="132.08" y2="81.28" width="0.1524" layer="91"/>
-</segment>
-</net>
+<wire x1="147.32" y1="88.9" x2="149.86" y2="88.9" width="0.1524" layer="91"/>
+<junction x="147.32" y="88.9"/>
+<pinref part="12VOUT1" gate="G$1" pin="2"/>
+<junction x="147.32" y="50.8"/>
+<wire x1="147.32" y1="58.42" x2="147.32" y2="50.8" width="0.1524" layer="91"/>
+<wire x1="132.08" y1="58.42" x2="147.32" y2="58.42" width="0.1524" layer="91"/>
+<pinref part="12VOUT1" gate="G$1" pin="1"/>
+<wire x1="132.08" y1="50.8" x2="132.08" y2="58.42" width="0.1524" layer="91"/>
+<junction x="132.08" y="50.8"/>
+<pinref part="12VOUT1" gate="G$1" pin="3"/>
+<wire x1="132.08" y1="48.26" x2="132.08" y2="50.8" width="0.1524" layer="91"/>
+<junction x="132.08" y="48.26"/>
+<wire x1="149.86" y1="88.9" x2="149.86" y2="58.42" width="0.1524" layer="91"/>
+<wire x1="149.86" y1="58.42" x2="147.32" y2="58.42" width="0.1524" layer="91"/>
+<junction x="147.32" y="58.42"/>
+</segment>
+</net>
