File: coProcessor/old/co_processor.sch (EAGLE design)
At the start: 75 parts

Commit message: some progress on the copro eagle schematic, optoisolator needs fixed
Other:
- moved on the sheet: PWM_IN0
Changed lines of the file:
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@@
 <?xml version="1.0" encoding="utf-8"?>
 <!DOCTYPE eagle SYSTEM "eagle.dtd">
-<eagle version="8.2.2">
+<eagle version="8.3.1">
 <drawing>
 <settings>
 <setting alwaysvectorfont="no"/>
+<setting keepoldvectorfont="yes"/>
 <setting verticaltext="up"/>
 </settings>
@@
 <instance part="OSC2_C" gate="G$1" x="406.4" y="254" rot="R180"/>
 <instance part="OPI_PWM0" gate="A" x="508" y="312.42" rot="R90"/>
-<instance part="PWM_IN0" gate="G$1" x="505.46" y="294.64" rot="R90"/>
+<instance part="PWM_IN0" gate="G$1" x="505.46" y="289.56" rot="R90"/>
 <instance part="GND_ESC1" gate="1" x="518.16" y="307.34"/>
 <instance part="SUPPLY10" gate="GND" x="510.54" y="297.18"/>
@@
 <instance part="BIAS_R9" gate="G$1" x="891.54" y="322.58" rot="R270"/>
 <instance part="GND_ESC10" gate="1" x="891.54" y="312.42"/>
-<instance part="SUPPLY22" gate="GND" x="883.92" y="302.26"/>
+<instance part="SUPPLY22" gate="GND" x="886.46" y="302.26"/>
 <instance part="BIAS_R0" gate="G$1" x="518.16" y="317.5" rot="R270"/>
 </instances>
@@
 <pinref part="SUPPLY22" gate="GND" pin="GND"/>
 <pinref part="OPI_PWM9" gate="A" pin="C"/>
-<wire x1="883.92" y1="304.8" x2="883.92" y2="307.34" width="0.1524" layer="91"/>
+<wire x1="886.46" y1="304.8" x2="883.92" y2="307.34" width="0.1524" layer="91"/>
 </segment>
 </net>
@@
 <segment>
 <pinref part="PWM_IN0" gate="G$1" pin="1"/>
-<wire x1="505.46" y1="289.56" x2="505.46" y2="287.02" width="0.1524" layer="91"/>
+<wire x1="505.46" y1="284.48" x2="505.46" y2="287.02" width="0.1524" layer="91"/>
 </segment>
 </net>
@@
 <pinref part="PWM_IN0" gate="G$1" pin="2"/>
 <pinref part="OPI_PWM0" gate="A" pin="A"/>
-<wire x1="505.46" y1="299.72" x2="505.46" y2="302.26" width="0.1524" layer="91"/>
+<wire x1="505.46" y1="294.64" x2="505.46" y2="302.26" width="0.1524" layer="91"/>
 </segment>
 </net>
@@
 <compatibility>
 <note version="8.2" severity="warning">
-Since Version 8.2, Eagle supports online libraries. The ids
+Since Version 8.2, EAGLE supports online libraries. The ids
 of those online libraries will not be understood (or retained)
 with this version.
