File: coProcessor/old/co_processor.brd (EAGLE design)
At the start: 101.6 x 101.6 mm, 75 parts

Commit message: The current official coprocessor board is now saved under the filename "copro - copy". I will change that. More importantly, the board is tentatively finished, atleast enough for others to check it, which i highly suggest.
Connections:
- new net 3.3V: C10.1, C11.1, C12.1, C13.1, C14.1, C15.1, C9.1, DEPTH_SENSOR.P$1, JTAG.1, JTAG.2, MICROSD.VCC, R1.2, R2.2, STM32F405.13, STM32F405.19, STM32F405.32, STM32F405.48, STM32F405.64, SWITCHES.1, SWITCHES.2, U$4.1, U$4.11, U$4.3, U$4.5, U$4.7, U$4.9, U$7.2
- net +3V3: no longer C10.1, C11.1, C12.1, C13.1, C14.1, C15.1, C9.1, DEPTH_SENSOR.P$1, JTAG.1, JTAG.2, MICROSD.VCC, R1.2, R2.2, STM32F405.13, STM32F405.19, STM32F405.32, STM32F405.48, STM32F405.64, SWITCHES.1, SWITCHES.2, U$4.1, U$4.11, U$4.3, U$4.5, U$4.7, U$4.9, U$7.2
Routing:
- net +3V3: track 424.5 -> 29.8 mm, vias 6 -> 0
- net 3.3V: track 0.00 -> 387.3 mm, vias 0 -> 6
