File: coProcessor/rev1noah/copro.brd (EAGLE design)
At the start: 101.6 x 101.6 mm, 97 parts, among them IC1 STM32F405RGT6, J1 USB_MINI-B_SMT, J2 79107-08, J3 693061010911, J4 30320-6002HB, T1 2N2222, T10 2N2222, T2 2N2222, T3 2N2222, T4 2N2222, T5 2N2222, T6 2N2222, T7 2N2222, T8 2N2222, T9 2N2222, U1 LM2597N-5.0, U2 SN65HVD232QD

Commit message: Slight progress on last commit, just so everything is up to date
Parts:
- added C5: 100pF, SparkFun-Capacitors:0603
- added CANH_R, CANL_R: LTST-S270GKT, LTST-S270GKT:0603
- added R45: 60, SparkFun-Resistors:0603
- added R46, R47: 330, SparkFun-Resistors:0603
- renumbered U2 to CAN_TRANSCEIVER
Connections:
- net N$5 renamed RXD
- removed net N$12: CAN_TRANSCEIVER.6, U$1.CAN_L
- new net CANH: C5.2, CAN_TRANSCEIVER.7, R45.1, R46.2, U$1.CAN_H
- new net CANL: C5.1, CAN_TRANSCEIVER.6, R45.2, R47.2, U$1.CAN_L
- new net N$34: CANH_R.2, R46.1
- net GND: now also CANH_R.1, CANL_R.1
- net N$8: now also CANL_R.2, R47.1; no longer CAN_TRANSCEIVER.7, U$1.CAN_H
Changed lines of the file:
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@@
 <attribute name="PRICE" value="1.62 USD" x="-127" y="-65.0875" size="1.778" layer="27" display="off"/>
 </element>
-<element name="U2" library="SN65HVD232QD" package="SOIC127P600X175-8N" value="SN65HVD232QD" x="-152.4" y="-80.9625">
+<element name="CAN_TRANSCEIVER" library="SN65HVD232QD" package="SOIC127P600X175-8N" value="SN65HVD232QD" x="-152.4" y="-80.9625">
 <attribute name="AVAILABILITY" value="Good" x="-152.4" y="-80.9625" size="1.778" layer="27" display="off"/>
 <attribute name="DESCRIPTION" value=" Automotive Catalog 3.3-V CAN Transceiver 8-SOIC -40 to 125 " x="-152.4" y="-80.9625" size="1.778" layer="27" display="off"/>
@@
 </element>
 <element name="J2" library="con-molex-milli-grid" package="79107-08" value="79107-08" x="-147.6375" y="-95.25"/>
+<element name="R45" library="SparkFun-Resistors" package="0603" value="60" x="-155.575" y="-106.3625">
+<attribute name="PROD_ID" value="RES-07856" x="-155.575" y="-106.3625" size="1.778" layer="27" display="off"/>
+</element>
+<element name="C5" library="SparkFun-Capacitors" package="0603" value="100pF" x="-155.575" y="-111.125">
+<attribute name="PROD_ID" value="CAP-08390" x="-155.575" y="-111.125" size="1.778" layer="27" display="off"/>
+</element>
+<element name="R46" library="SparkFun-Resistors" package="0603" value="330" x="-155.575" y="-115.8875">
+<attribute name="PROD_ID" value="RES-07856" x="-155.575" y="-115.8875" size="1.778" layer="27" display="off"/>
+</element>
+<element name="R47" library="SparkFun-Resistors" package="0603" value="330" x="-155.575" y="-120.65">
+<attribute name="PROD_ID" value="RES-07856" x="-155.575" y="-120.65" size="1.778" layer="27" display="off"/>
+</element>
+<element name="CANL_R" library="LTST-S270GKT" package="0603" value="LTST-S270GKT" x="-155.575" y="-125.4125">
+<attribute name="AVAILABILITY" value="Good" x="-155.575" y="-125.4125" size="1.778" layer="27" display="off"/>
+<attribute name="DESCRIPTION" value=" Green 1.6 x 0.6 x 1.15 mm 130° Water Clear 12 mcd 2.1 V Molded SMT LED " x="-155.575" y="-125.4125" size="1.778" layer="27" display="off"/>
+<attribute name="MF" value="Lite-On" x="-155.575" y="-125.4125" size="1.778" layer="27" display="off"/>
+<attribute name="MP" value="LTST-S270GKT" x="-155.575" y="-125.4125" size="1.778" layer="27" display="off"/>
+<attribute name="PACKAGE" value="0603 Lite-On" x="-155.575" y="-125.4125" size="1.778" layer="27" display="off"/>
+<attribute name="PRICE" value="0.08 USD" x="-155.575" y="-125.4125" size="1.778" layer="27" display="off"/>
+</element>
+<element name="CANH_R" library="LTST-S270GKT" package="0603" value="LTST-S270GKT" x="-155.575" y="-131.7625">
+<attribute name="AVAILABILITY" value="Good" x="-155.575" y="-131.7625" size="1.778" layer="27" display="off"/>
+<attribute name="DESCRIPTION" value=" Green 1.6 x 0.6 x 1.15 mm 130° Water Clear 12 mcd 2.1 V Molded SMT LED " x="-155.575" y="-131.7625" size="1.778" layer="27" display="off"/>
+<attribute name="MF" value="Lite-On" x="-155.575" y="-131.7625" size="1.778" layer="27" display="off"/>
+<attribute name="MP" value="LTST-S270GKT" x="-155.575" y="-131.7625" size="1.778" layer="27" display="off"/>
+<attribute name="PACKAGE" value="0603 Lite-On" x="-155.575" y="-131.7625" size="1.778" layer="27" display="off"/>
+<attribute name="PRICE" value="0.08 USD" x="-155.575" y="-131.7625" size="1.778" layer="27" display="off"/>
+</element>
 </elements>
 <signals>
@@
 <contactref element="HEARTBEAT1" pad="1"/>
 <contactref element="U1" pad="6"/>
-<contactref element="U2" pad="2"/>
+<contactref element="CAN_TRANSCEIVER" pad="2"/>
+<contactref element="CANL_R" pad="1"/>
+<contactref element="CANH_R" pad="1"/>
 <wire x1="230.925" y1="-11.1125" x2="246.38" y2="-0.3175" width="0" layer="19" extent="1-1"/>
 <wire x1="230.925" y1="-17.4625" x2="230.925" y2="-11.1125" width="0" layer="19" extent="1-1"/>
@@
 <wire x1="-127" y1="-62.5475" x2="-127" y2="26.25" width="0" layer="19" extent="1-1"/>
 <wire x1="-154.8638" y1="-80.3275" x2="-127" y2="-62.5475" width="0" layer="19" extent="1-1"/>
+<wire x1="-156.425" y1="-125.4125" x2="-154.8638" y2="-80.3275" width="0" layer="19" extent="1-1"/>
+<wire x1="-156.425" y1="-131.7625" x2="-156.425" y2="-125.4125" width="0" layer="19" extent="1-1"/>
 <wire x1="314.0075" y1="108.9025" x2="246.38" y2="-0.3175" width="0" layer="19" extent="1-1"/>
 <wire x1="314.0075" y1="170.815" x2="314.0075" y2="108.9025" width="0" layer="19" extent="1-1"/>
@@
 <contactref element="J4" pad="1"/>
 <contactref element="J4" pad="2"/>
-<contactref element="U2" pad="3"/>
+<contactref element="CAN_TRANSCEIVER" pad="3"/>
 <contactref element="J2" pad="7"/>
 <contactref element="J2" pad="1"/>
@@
 <signal name="TXD">
 <contactref element="IC1" pad="45"/>
-<contactref element="U2" pad="1"/>
+<contactref element="CAN_TRANSCEIVER" pad="1"/>
 <wire x1="54.9625" y1="53.05" x2="-154.8638" y2="-79.0575" width="0" layer="19" extent="1-1"/>
 </signal>
-<signal name="N$5">
+<signal name="RXD">
 <contactref element="IC1" pad="44"/>
-<contactref element="U2" pad="4"/>
+<contactref element="CAN_TRANSCEIVER" pad="4"/>
 <wire x1="54.9625" y1="52.55" x2="-154.8638" y2="-82.8675" width="0" layer="19" extent="1-1"/>
-</signal>
-<signal name="N$8">
-<contactref element="U$1" pad="CAN_H"/>
-<contactref element="U2" pad="7"/>
-<wire x1="67.5005" y1="3.175" x2="-149.9362" y2="-80.3275" width="0" layer="19" extent="1-1"/>
-</signal>
-<signal name="N$12">
-<contactref element="U$1" pad="CAN_L"/>
-<contactref element="U2" pad="6"/>
-<wire x1="70.0405" y1="3.175" x2="-149.9362" y2="-81.5975" width="0" layer="19" extent="1-1"/>
 </signal>
 <signal name="N$20">
@@
 <wire x1="43.4625" y1="49.55" x2="-144.6375" y2="-96.25" width="0" layer="19" extent="1-1"/>
 </signal>
+<signal name="CANH">
+<contactref element="R45" pad="1"/>
+<contactref element="C5" pad="2"/>
+<contactref element="CAN_TRANSCEIVER" pad="7"/>
+<contactref element="U$1" pad="CAN_H"/>
+<contactref element="R46" pad="2"/>
+<wire x1="-156.425" y1="-106.3625" x2="-149.9362" y2="-80.3275" width="0" layer="19" extent="1-1"/>
+<wire x1="-154.725" y1="-111.125" x2="-156.425" y2="-106.3625" width="0" layer="19" extent="1-1"/>
+<wire x1="-154.725" y1="-115.8875" x2="-154.725" y2="-111.125" width="0" layer="19" extent="1-1"/>
+<wire x1="67.5005" y1="3.175" x2="-149.9362" y2="-80.3275" width="0" layer="19" extent="1-1"/>
+</signal>
+<signal name="N$8">
+<contactref element="R47" pad="1"/>
+<contactref element="CANL_R" pad="2"/>
+<wire x1="-156.425" y1="-120.65" x2="-154.725" y2="-125.4125" width="0" layer="19" extent="1-1"/>
+</signal>
+<signal name="N$34">
+<contactref element="R46" pad="1"/>
+<contactref element="CANH_R" pad="2"/>
+<wire x1="-156.425" y1="-115.8875" x2="-154.725" y2="-131.7625" width="0" layer="19" extent="1-1"/>
+</signal>
+<signal name="CANL">
+<contactref element="R45" pad="2"/>
+<contactref element="C5" pad="1"/>
+<contactref element="CAN_TRANSCEIVER" pad="6"/>
+<contactref element="U$1" pad="CAN_L"/>
+<contactref element="R47" pad="2"/>
+<wire x1="-154.725" y1="-106.3625" x2="-149.9362" y2="-81.5975" width="0" layer="19" extent="1-1"/>
+<wire x1="-156.425" y1="-111.125" x2="-154.725" y2="-106.3625" width="0" layer="19" extent="1-1"/>
+<wire x1="-154.725" y1="-120.65" x2="-156.425" y2="-111.125" width="0" layer="19" extent="1-1"/>
+<wire x1="70.0405" y1="3.175" x2="-149.9362" y2="-81.5975" width="0" layer="19" extent="1-1"/>
+</signal>
 </signals>

Commit message: The current official coprocessor board is now saved under the filename "copro - copy". I will change that. More importantly, the board is tentatively finished, atleast enough for others to check it, which i highly suggest.
Parts:
- removed 455-1750-1-ND: (no value), SparkFun-Connectors:1X03
- removed C1: 4.7uF, SparkFun-Capacitors:0603
- removed C12, C2, C4, C6, C9: 100nF, SparkFun-Capacitors:0603
- removed C14: 1uF, SparkFun-Capacitors:0603
- removed C3, C8: 2.2uF, SparkFun-Capacitors:0603
- removed J3: 693061010911, 693061010911:693061010911
- removed R10, R14, R18, R22, R26, R30, R34, R38, R4, R6: 1k, SparkFun-Resistors:0603
- removed R12, R13, R16, R17, R2, R20, R21, R24, R25, R28, R29, R3, R32, R33, R36, R37, R40, R8, R9: 10k, SparkFun-Resistors:0603
- removed R41, R42: 2.2k, SparkFun-Resistors:0603
- removed R45: 60, SparkFun-Resistors:0603
- removed U1: LM2597N-5.0, LM2597N-5.0:DIP254P762X508-8
- added 455-1750-1-ND10: (no value), SparkFun-Connectors:1X03
- added C10: 1nF, SparkFun-Capacitors:0603
- added C7: .1 uF, SparkFun-Capacitors:0603
- added CAP1, CAP2, CAP3, CAP4, VDDACAP1: 100nF, SparkFun-Capacitors:0603
- added CAP5, CAP6: 2.2uF, SparkFun-Capacitors:0603
- added CAP7: 4.7uF, SparkFun-Capacitors:0603
- added J5: 5008730806, 5008730806:5008730806
- added OSCILLATOR: (no value), crystal:HC49/S
- added R12C, RI2C: 4.7k, SparkFun-Resistors:0603
- added RO10A, RO1A, RO2A, RO3A, RO4A, RO5A, RO6A, RO7A, RO8A, RO9A: 1k, SparkFun-Resistors:0603
- added RO10B, RO10C, RO1B, RO1C, RO2B, RO2C, RO3B, RO3C, RO4B, RO4C, RO5B, RO5C, RO6B, RO6C, RO7B, RO7C, RO8B, RO8C, RO9B, RO9C: 10k, SparkFun-Resistors:0603
- added VDDACAP2: 1uF, SparkFun-Capacitors:0603
- added VOLTAGE_REG: TL780_VREG, TL780_VREG:D2PAK-3
- C5: value 100pF -> 1nF
- CAN_TRANSCEIVER: value SN65HVD232QD -> MCP2551-I/P; device SN65HVD232QD:SOIC127P600X175-8N -> MCP2551-I_P:DIP254P762X432-8
- R1: value 10k -> 330
- T1, T10, T2, T3, T4, T5, T6, T7, T8, T9: value 2N2222 -> (none); device transistor:TO18 -> transistor:TO126V
- moved OI7 350.2 mm to (85.7, 31.8), turned to 270 degrees
- moved 455-1750-1-ND6 314.5 mm to (100.0, 47.6), turned to 270 degrees
- moved R27 312.2 mm to (81.0, 34.9)
- moved OI8 310.0 mm to (85.7, 25.4), turned to 270 degrees
- moved T7 293.2 mm to (98.4, 60.3), turned to 270 degrees
- moved R31 280.7 mm to (81.0, 22.2)
- moved 455-1750-1-ND7 277.5 mm to (100.0, 39.7), turned to 270 degrees
- moved OI9 275.2 mm to (85.7, 19.1), turned to 270 degrees
- moved C5 258.5 mm to (33.4, 65.2), turned to 180 degrees
- moved T8 250.7 mm to (98.4, 68.3), turned to 270 degrees
- moved CANL_R 249.1 mm to (44.0, 23.6)
- moved OI10 248.1 mm to (85.7, 12.7), turned to 270 degrees
- moved R35 246.8 mm to (81.0, 28.6)
- moved 455-1750-1-ND8 246.7 mm to (100.0, 31.8), turned to 270 degrees
- moved CANH_R 242.1 mm to (37.3, 14.5), turned to 270 degrees
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Connections:
- net N$20 renamed 2
- net N$25 renamed 4
- net N$27 renamed 6
- net N$32 renamed 8
- removed net +3V3: C1.1, C12.1, C14.2, C2.1, C4.1, C6.2, C9.1, CAN_TRANSCEIVER.3, DEPTH_SENSOR.P$1, IC1.13, IC1.19, IC1.32, IC1.48, IC1.64, J1.VBUS, J2.1, J2.3, J2.5, J2.7, J3.4, J4.1, J4.2, POWERJACK.1.1, POWERJACK.1.2, R41.2, R42.2
- removed net GNDA: 455-1750-1-ND1.3, 455-1750-1-ND2.3, 455-1750-1-ND3.3, 455-1750-1-ND4.3, 455-1750-1-ND5.3, 455-1750-1-ND6.3, 455-1750-1-ND7.3, 455-1750-1-ND8.3, 455-1750-1-ND9.3, OI10.4, OI2.4, OI3.4, OI4.4, OI5.4, OI6.4, OI7.4, OI8.4, OI9.4, SWITCH1.1, T10.1, T2.1, T3.1, T4.1, T5.1, T6.1, T7.1, T8.1, T9.1
- removed net N$21: J3.3, J3.6, J3.Z1, J3.Z2
- removed net N$3: C3.1, C8.1, IC1.31, IC1.47
- removed net PB8: DEPTH_SENSOR.P$2, IC1.61, R41.1
- new net N$12: CAN_TRANSCEIVER.5, R1.1
- new net N$5: CAN_TRANSCEIVER.2, R1.2
- new net OSC1: C5.1, IC1.6, OSCILLATOR.1
- new net OSC2: C10.1, IC1.5, OSCILLATOR.2
- new net P$2: DEPTH_SENSOR.P$2, IC1.61, RI2C.1
- new net VCAP_2TO1: CAP5.1, CAP6.1, IC1.31, IC1.47
- net 3.3V: now also C7.1, CAN_TRANSCEIVER.3, CAP1.1, CAP2.1, CAP3.1, CAP4.1, CAP7.1, DEPTH_SENSOR.P$1, IC1.13, IC1.19, IC1.32, IC1.48, IC1.64, J1.VBUS, J2.1, J2.3, J2.5, J2.7, J4.1, J4.2, J5.4, POWERJACK.1.1, POWERJACK.1.2, R12C.2, RI2C.2, VDDACAP1.2, VDDACAP2.2
- net CANH: now also CAN_TRANSCEIVER.6; no longer C5.2, CAN_TRANSCEIVER.7, R45.1
- net CANL: now also CAN_TRANSCEIVER.7; no longer C5.1, CAN_TRANSCEIVER.6, R45.2
- net CLK: now also J5.5; no longer J3.5
- net CMD: now also J5.2; no longer J3.2
- net DATO: now also J5.7; no longer J3.7
- net GND: now also C10.2, C5.2, C7.2, CAP1.2, CAP2.2, CAP3.2, CAP4.2, CAP5.2, CAP6.2, CAP7.2, J5.6, J5.S3, J5.S4, VDDACAP1.1, VDDACAP2.1, VOLTAGE_REG.2; no longer C1.2, C12.2, C14.1, C2.2, C3.2, C4.2, C6.1, C8.2, C9.2, CAN_TRANSCEIVER.2, U1.6
- net GNDBAT: now also 455-1750-1-ND1.3, 455-1750-1-ND10.3, 455-1750-1-ND2.3, 455-1750-1-ND3.3, 455-1750-1-ND4.3, 455-1750-1-ND5.3, 455-1750-1-ND6.3, 455-1750-1-ND7.3, 455-1750-1-ND8.3, 455-1750-1-ND9.3, OI10.4, OI2.4, OI3.4, OI4.4, OI5.4, OI6.4, OI7.4, OI8.4, OI9.4, SWITCH1.1, T10.1, T2.1, T3.1, T4.1, T5.1, T6.1, T7.1, T8.1, T9.1; no longer 455-1750-1-ND.3
- net N$1: now also RO2A.2, RO2B.1; no longer R1.1, R6.2
- net N$10: now also RO1B.2, RO1C.2; no longer R2.2, R3.2
- net N$15: now also RO2B.2, RO2C.2; no longer R1.2, R8.2
- net N$16: now also RO3A.2, RO3B.1; no longer R10.2, R9.1
- net N$17: now also RO3A.1, T3.3; no longer R10.1, T3.2
- net N$18: now also 455-1750-1-ND10.1, RO10C.1, RO1C.1, RO2C.1, RO3C.1, RO4C.1, RO5C.1, RO6C.1, RO7C.1, RO8C.1, RO9C.1, T1.2, T10.2, T2.2, T3.2, T4.2, T5.2, T6.2, T7.2, T8.2, T9.2, VOLTAGE_REG.3; no longer 455-1750-1-ND.1, R12.1, R16.1, R2.1, R20.1, R24.1, R28.1, R32.1, R36.1, R40.1, R8.1, T1.3, T10.3, T2.3, T3.3, T4.3, T5.3, T6.3, T7.3, T8.3, T9.3, U1.8
- net N$2: now also RO1A.1, T1.3; no longer R4.1, T1.2
- net N$22: now also RO3B.2, RO3C.2; no longer R12.2, R9.2
- net N$23: now also RO4A.2, RO4B.1; no longer R13.1, R14.2
- net N$24: now also RO4A.1, T4.3; no longer R14.1, T4.2
- net N$29: now also RO4B.2, RO4C.2; no longer R13.2, R16.2
- net N$30: now also RO5A.2, RO5B.1; no longer R17.1, R18.2
- net N$31: now also RO5A.1, T5.3; no longer R18.1, T5.2
- net N$36: now also RO5B.2, RO5C.2; no longer R17.2, R20.2
- net N$37: now also RO6A.2, RO6B.1; no longer R21.1, R22.2
- net N$38: now also RO6A.1, T6.3; no longer R22.1, T6.2
- net N$43: now also RO6B.2, RO6C.2; no longer R21.2, R24.2
- net N$44: now also RO7A.2, RO7B.1; no longer R25.1, R26.2
- net N$45: now also RO7A.1, T7.3; no longer R26.1, T7.2
- net N$50: now also RO7B.2, RO7C.2; no longer R25.2, R28.2
- net N$51: now also RO8A.2, RO8B.1; no longer R29.1, R30.2
- net N$52: now also RO8A.1, T8.3; no longer R30.1, T8.2
- net N$57: now also RO8B.2, RO8C.2; no longer R29.2, R32.2
- net N$58: now also RO9A.2, RO9B.1; no longer R33.1, R34.2
- net N$59: now also RO9A.1, T9.3; no longer R34.1, T9.2
- net N$6: now also RO1A.2, RO1B.1; no longer R3.1, R4.2
- net N$64: now also RO9B.2, RO9C.2; no longer R33.2, R36.2
- net N$65: now also RO10A.2, RO10B.1; no longer R37.1, R38.2
- net N$66: now also RO10A.1, T10.3; no longer R38.1, T10.2
- net N$7: now also VOLTAGE_REG.1; no longer U1.7
- net N$71: now also RO10B.2, RO10C.2; no longer R37.2, R40.2
- net N$9: now also RO2A.1, T2.3; no longer R6.1, T2.2
- net PS$3: now also R12C.1; no longer R42.1
Routing:
- net GND: track 0.00 -> 404.6 mm, vias 0 -> 20
- net 3.3V: track 5.08 -> 326.4 mm, vias 0 -> 12
- net 8: track 0.00 -> 142.4 mm
- net D+: track 0.00 -> 132.6 mm, vias 0 -> 2
- net DATO: track 0.00 -> 123.2 mm, vias 0 -> 2
- net D-: track 0.00 -> 108.4 mm, vias 0 -> 2
- net PS$3: track 0.00 -> 96.0 mm, vias 0 -> 2
- net JTAG9: track 0.00 -> 91.0 mm, vias 0 -> 4
- net JTAG13: track 0.00 -> 79.7 mm, vias 0 -> 2
- net JTAG5: track 0.00 -> 71.9 mm, vias 0 -> 2
- net JTAG3: track 0.00 -> 71.5 mm
- net PA15: track 0.00 -> 68.2 mm
- net JTAG15: track 0.00 -> 67.6 mm, vias 0 -> 2
- net P$2: track 0.00 -> 57.5 mm, vias 0 -> 1
- net CLK: track 0.00 -> 52.6 mm, vias 0 -> 2
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Other:
- board text removed: "The Ohio State Univerity Center for Automotive Research"
- board text removed: "The Underwater Robotics Team Riptide -- Board Template"
