File: coProcessor/rev1noah/Coprocessor_Board.brd (EAGLE design)
At the start: 101.6 x 101.6 mm, 98 parts, among them IC1 STM32F405RGT6, J1 USB_MINI-B_SMT, J4 30320-6002HB, J5 5008730806, P1 39-30-08?, Q1 L78M05CV

Commit message: Fixing USB lines, we RF now boyz
Parts:
- added D+PULL, D-PULL: 1.5k, resistor:0204/7
- added D+SERIES, D-SERIES: 22Ohm, resistor:0204/7
- RHB1, RHB2: value 330 -> 1k; device SparkFun-Resistors:AXIAL-0.1 -> SparkFun-Resistors:AXIAL-0.3
- moved RHB1 3.22 mm to (42.7, 84.0)
- moved RHB2 2.54 mm to (42.3, 81.2)
- moved HBL1 1.28 mm to (33.2, 84.0)
- moved HBL2 0.27 mm to (31.2, 81.2)
Connections:
- new net D+CON: D+PULL.1, D+SERIES.2, J1.D+
- new net D-CON: D-PULL.1, D-SERIES.2, J1.D-
- net 3.3V: now also D+PULL.2, D-PULL.2
- net USB_OTG_HS_DM: now also D-SERIES.1; no longer J1.D-
- net USB_OTG_HS_DP: now also D+SERIES.1; no longer J1.D+
Routing:
- net SCL_BKPLN: track 146.1 -> 96.0 mm
- net SDA_BKPLN: track 140.4 -> 94.6 mm
- net USB_OTG_HS_DM: track 54.1 -> 18.0 mm
- net D-CON: track 0.00 -> 29.4 mm
- net USB_OTG_HS_DP: track 52.7 -> 27.7 mm
- net D+CON: track 0.00 -> 18.3 mm
- net 3.3V: track 298.0 -> 315.5 mm
- net HEARTBEAT_1: track 19.8 -> 13.3 mm
- net HEARTBEAT_2: track 15.3 -> 10.5 mm
- net GND: track 112.3 -> 110.9 mm

Commit message: Trace clean up
Parts:
- D+SERIES, D-SERIES: value 22Ohm -> 22Ω
- moved C8 2.28 mm to (33.3, 44.9)
- moved C9 2.18 mm to (40.6, 45.0)
- moved OSCILLATOR 2.12 mm to (37.0, 41.1)
Routing:
- net KILLSWITCH: track 71.0 -> 109.1 mm, vias 4 -> 2
- net SURGESTBDHI: track 42.2 -> 48.5 mm
- net SURGESTBDLOW: track 34.2 -> 39.0 mm
- net RCC_OSC_IN: track 25.6 -> 22.6 mm
- net SURGEPORTHI: track 26.8 -> 29.1 mm
- net RCC_OSC_OUT: track 22.3 -> 20.5 mm
- net SURGEPORTLOW: track 22.7 -> 23.8 mm
- net SW_FWD: track 27.9 -> 26.9 mm
- net SW_AFT: track 21.0 -> 20.1 mm
- net GND: track 110.9 -> 110.3 mm

Commit message: Future proofing
Parts:
- added USB_ID: 0Ω, resistor:0204/7
Connections:
- new net OTG_ID: IC1.33, USB_ID.1
- new net OTG_ID_CON: J1.ID, USB_ID.2
Routing:
- net OTG_ID_CON: track 0.00 -> 41.1 mm, vias 0 -> 1
- net OTG_ID: track 0.00 -> 4.89 mm
Changed lines of the file:
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@@
 <attribute name="VALUE" x="27.20063125" y="82.47418125" size="0.9906" layer="27" ratio="10" rot="R270"/>
+</element>
+<element name="USB_ID" library="resistor" library_urn="urn:adsk.eagle:library:348" package="0204/7" package3d_urn="urn:adsk.eagle:package:25945/1" value="0Ω" x="49.355734375" y="79.070759375" smashed="yes" rot="R90">
+<attribute name="NAME" x="51.7006375" y="79.070503125" size="0.9906" layer="25" ratio="10" rot="R90"/>
+<attribute name="VALUE" x="52.9706875" y="79.222984375" size="0.9906" layer="27" ratio="10" rot="R90"/>
 </element>
 </elements>
@@
 <contactref element="RESET" pad="4"/>
 <contactref element="RESET" pad="3"/>
-<wire x1="11.172003125" y1="59.257859375" x2="9.905009375" y2="57.990865625" width="0.1524" layer="1"/>
-<wire x1="11.172003125" y1="59.257859375" x2="11.172003125" y2="59.6248875" width="0.1524" layer="1"/>
 <via x="45.8000875" y="55.02783125" extent="1-16" drill="0.35"/>
 <wire x1="44.85" y1="59.5375" x2="44.85" y2="55.893259375" width="0.1524" layer="1"/>
@@
 <wire x1="18.9634375" y1="54.77385625" x2="16.737153125" y2="52.547571875" width="0.1524" layer="1"/>
 <wire x1="14.002790625" y1="50.007828125" x2="16.737153125" y2="52.547571875" width="0.1524" layer="1"/>
-<wire x1="9.905009375" y1="57.990865625" x2="9.905009375" y2="56.72099375" width="0.1524" layer="1"/>
-<wire x1="9.905009375" y1="56.72099375" x2="8.042528125" y2="54.8585125" width="0.1524" layer="1"/>
-<wire x1="8.042528125" y1="54.8585125" x2="8.042528125" y2="50.549965625" width="0.1524" layer="1"/>
-<wire x1="8.042528125" y1="50.549965625" x2="7.500390625" y2="50.007828125" width="0.1524" layer="1"/>
-<wire x1="7.500390625" y1="50.007828125" x2="14.002790625" y2="50.007828125" width="0.1524" layer="1"/>
+<wire x1="7.6192375" y1="50.007828125" x2="7.500390625" y2="50.007828125" width="0.1524" layer="1"/>
+<wire x1="7.6192375" y1="50.007828125" x2="14.002790625" y2="50.007828125" width="0.1524" layer="1"/>
+<wire x1="11.172003125" y1="59.6248875" x2="10.861765625" y2="59.6248875" width="0.1524" layer="1"/>
+<wire x1="10.861765625" y1="59.6248875" x2="9.98966875" y2="58.752790625" width="0.1524" layer="1"/>
+<wire x1="9.98966875" y1="58.752790625" x2="9.98966875" y2="52.378259375" width="0.1524" layer="1"/>
+<wire x1="9.98966875" y1="52.378259375" x2="7.6192375" y2="50.007828125" width="0.1524" layer="1"/>
 </signal>
 <signal name="SYS_JTCK-SWCLK">
@@
 <contactref element="J4" pad="3"/>
 <contactref element="IC1" pad="56"/>
-<wire x1="27.74101875" y1="60.953903125" x2="26.412003125" y2="59.6248875" width="0.2032" layer="1"/>
-<wire x1="39.85" y1="65.5375" x2="37.2616625" y2="65.5375" width="0.2032" layer="1"/>
-<wire x1="37.2616625" y1="65.5375" x2="32.678065625" y2="60.953903125" width="0.2032" layer="1"/>
-<wire x1="32.678065625" y1="60.953903125" x2="27.74101875" y2="60.953903125" width="0.2032" layer="1"/>
+<wire x1="39.85" y1="65.5375" x2="37.5156375" y2="65.5375" width="0.1524" layer="1"/>
+<wire x1="37.5156375" y1="65.5375" x2="32.932040625" y2="60.953903125" width="0.1524" layer="1"/>
+<wire x1="32.932040625" y1="60.953903125" x2="27.74101875" y2="60.953903125" width="0.1524" layer="1"/>
+<wire x1="27.74101875" y1="60.953903125" x2="26.412003125" y2="59.6248875" width="0.1524" layer="1"/>
 </signal>
 <signal name="DEPTHSDA">
@@
 <wire x1="27.6832375" y1="86.605721875" x2="27.7675125" y2="86.689996875" width="0.1524" layer="1"/>
 </signal>
+<signal name="OTG_ID">
+<contactref element="IC1" pad="33"/>
+<contactref element="USB_ID" pad="1"/>
+<wire x1="49.35" y1="71.0375" x2="49.35" y2="75.59365625" width="0.1524" layer="1"/>
+<wire x1="49.35" y1="75.59365625" x2="49.355734375" y2="75.260759375" width="0.1524" layer="1"/>
+</signal>
+<signal name="OTG_ID_CON">
+<contactref element="USB_ID" pad="2"/>
+<contactref element="J1" pad="ID"/>
+<wire x1="49.355734375" y1="82.880759375" x2="49.355734375" y2="83.134346875" width="0.1524" layer="16"/>
+<wire x1="49.355734375" y1="83.134346875" x2="46.562009375" y2="85.674096875" width="0.1524" layer="16"/>
+<via x="46.562009375" y="85.674096875" extent="1-16" drill="0.35"/>
+<wire x1="46.562009375" y1="85.674096875" x2="25.035546875" y2="85.674096875" width="0.1524" layer="1"/>
+<wire x1="25.035546875" y1="85.674096875" x2="25.025565625" y2="85.664115625" width="0.1524" layer="1"/>
+<wire x1="10.95908125" y1="85.6783375" x2="9.861409375" y2="85.6783375" width="0.1524" layer="1"/>
+<wire x1="9.861409375" y1="85.6783375" x2="9.59260625" y2="85.947140625" width="0.1524" layer="1"/>
+<wire x1="25.025565625" y1="85.664115625" x2="10.973303125" y2="85.664115625" width="0.1524" layer="1"/>
+<wire x1="10.973303125" y1="85.664115625" x2="10.95908125" y2="85.6783375" width="0.1524" layer="1"/>
+</signal>
 </signals>
