File: coProcessor/rev1noah/Coprocessor_Board.sch (EAGLE design)
At the start: 106 parts, among them IC1 STM32F405RGT6, J1 USB_MINI-B_SMT, J2 79107-08, J4 30320-6002HB, J5 5008730806, Q1 L78M05CV

Commit message: coprocessor board tentatively finished draft2, many things fixed, CAN kicked the can, and parts list added
Parts:
- removed CANH_R, CANL_R: LTST-S270GKT, LTST-S270GKT:LTST-S270GKT
- removed CAN_TRANSCEIVER: MCP2551-I/P, MCP2551-I_P:MCP2551-I/P
- removed CAP1, CAP2, CAP3, CAP4, VDDACAP1: 100nF, SparkFun-Capacitors:0.1UF-0603-100V-10%
- removed CAP5, CAP6: 2.2uF, SparkFun-Capacitors:0.1UF-0603-100V-10%
- removed CAP7: 4.7uF, SparkFun-Capacitors:0.1UF-0603-100V-10%
- removed RHB3, RH_R, RL_R: 330, SparkFun-Resistors:1KOHM-VERT-1/4W-1%
- removed SWITCH1: 39-30-02, con-molex-mini-fit:39-30-02
- removed VDDACAP2: 1uF, SparkFun-Capacitors:0.1UF-0603-100V-10%
- added C1: 4.7 uF, SparkFun-Capacitors:0.1UF-0603-100V-10%
- added C11: 2.2uF, SparkFun-Capacitors:0.1UF-0603-100V-10%
- added C12: 2.2 uF, SparkFun-Capacitors:0.1UF-0603-100V-10%
- added C2, C3, C4: 100 nF, SparkFun-Capacitors:0.1UF-0603-100V-10%
- added C8, C9: 1 nF, SparkFun-Capacitors:22PF-PTH-2.54MM-200V-5%
- C10, C5: value 1nF -> 100 nF
- C7: value .1 uF -> 1 uF
Connections:
- net T1 renamed GATE1
- net T10 renamed GATE10
- net T2 renamed GATE2
- net T3 renamed GATE3
- net T4 renamed GATE4
- net T5 renamed GATE5
- net T6 renamed GATE6
- net T7 renamed GATE7
- net T8 renamed GATE8
- net T9 renamed GATE9
- removed net 18_22V: Q1.IN, SWITCH1.2, U$1.EXTRA23
- removed net CANL: CAN_TRANSCEIVER.CANH, RL_R.1, U$1.CAN_L
- removed net CANRX_BKPLN: CAN_TRANSCEIVER.RXD, IC1.PA11
- removed net CANTX-BKPLN: CAN_TRANSCEIVER.TXD, IC1.PA12
- removed net N$12: CAN_TRANSCEIVER.VREF, RHB3.1
- removed net N$5: CAN_TRANSCEIVER.VSS, RHB3.2
- removed net N$8: CANL_R.A2, RL_R.2
- removed net N$9: CANH_R.A2, RH_R.2
- removed net POWER1O1: RO1B.2, RO1C.2
- removed net POWER1O10: RO10B.2, RO10C.2
- removed net POWER1O2: RO2B.2, RO2C.2
- removed net POWER1O3: RO3B.2, RO3C.2
- removed net POWER1O4: RO4B.2, RO4C.2
- removed net POWER1O5: RO5B.2, RO5C.2
- removed net POWER1O6: RO6B.2, RO6C.2
- removed net POWER1O7: RO7B.2, RO7C.2
- removed net POWER1O8: RO8B.2, RO8C.2
- removed net POWER1O9: RO9B.2, RO9C.2
- removed net VCAP_2_1: CAP5.1, CAP6.1, IC1.VCAP_1, IC1.VCAP_2
- new net 18V: Q1.IN, U$1.EXTRA23
- new net SOURCE1: ESC1.1, RO1C.1, T1.C
- new net SOURCE10: ESC10.1, RO10C.1, T10.C
- new net SOURCE2: ESC2.1, RO2C.1, T2.C
- new net SOURCE3: ESC3.1, RO3C.1, T3.C
- new net SOURCE4: ESC4.1, RO4C.1, T4.C
- new net SOURCE5: ESC5.1, RO5C.1, T5.C
- new net SOURCE6: ESC6.1, RO6C.1, T6.C
- new net SOURCE7: ESC7.1, RO7C.1, T7.C
- new net SOURCE8: ESC8.1, RO8C.1, T8.C
- new net SOURCE9: ESC9.1, RO9C.1, T9.C
- new net VCAP: C11.2, IC1.VCAP_2
- new net VCAP2: C12.1, IC1.VCAP_1
- net 3.3V: now also C1.1, C10.1, C2.1, C3.1, C4.1, C5.1; no longer CAN_TRANSCEIVER.VDD, CAP1.1, CAP2.1, CAP3.1, CAP4.1, CAP7.1, J1.VBUS, VDDACAP1.2, VDDACAP2.2
- net 5V: now also RO10B.2, RO10C.2, RO1B.2, RO1C.2, RO2B.2, RO2C.2, RO3B.2, RO3C.2, RO4B.2, RO4C.2, RO5B.2, RO5C.2, RO6B.2, RO6C.2, RO7B.2, RO7C.2, RO8B.2, RO8C.2, RO9B.2, RO9C.2; no longer ESC1.1, ESC10.1, ESC2.1, ESC3.1, ESC4.1, ESC5.1, ESC6.1, ESC7.1, ESC8.1, ESC9.1, RO10C.1, RO1C.1, RO2C.1, RO3C.1, RO4C.1, RO5C.1, RO6C.1, RO7C.1, RO8C.1, RO9C.1, T1.C, T10.C, T2.C, T3.C, T4.C, T5.C, T6.C, T7.C, T8.C, T9.C
- net CANH: no longer CAN_TRANSCEIVER.CANL, RH_R.1
- net GND: now also C1.2, C11.1, C12.2, C2.2, C3.2, C4.2, C8.1, C9.1; no longer CANH_R.K2, CANL_R.K2, CAP1.2, CAP2.2, CAP3.2, CAP4.2, CAP5.2, CAP6.2, CAP7.2, VDDACAP1.1, VDDACAP2.1
- net GNDBAT: no longer SWITCH1.1
- net RCC_OSC_IN: now also C8.2; no longer C10.1
- net RCC_OSC_OUT: now also C9.2; no longer C5.1
Other:
- moved on the sheet: C10, C5, C7, HEARTBEAT1, HEARTBEAT2, J4, J5, POWERJACK, RHB1, RHB2, S2

Commit message: General clean (salute) up of copro
Parts:
- removed HEARTBEAT1, HEARTBEAT2: LTST-S270GKT, LTST-S270GKT:LTST-S270GKT
- removed J2: 79107-08, con-molex-milli-grid:79107-08
- removed S2: MOMENTARY-SWITCH-SPST-SMD-4.5MM, SparkFun-Switches:MOMENTARY-SWITCH-SPST-SMD-4.5MM
- added HBL1, HBL2: LED, SparkFun-Resistors:1KOHM-VERT-1/4W-1%
- added P1: 39-30-08, con-molex-mini-fit:39-30-08
- added RESET: (no value), switch-omron:10-XX
- renumbered POWERJACK to 3V3_ONLY
Connections:
- removed net N$10: HEARTBEAT1.A2, RHB1.2
- removed net POWER: U$1.3.3V_4, U$1.3.3V_5, U$1.3.3V_6
- new net N$1: HBL1.1, RHB1.2
- net 3.3V: now also P1.1, P1.2, P1.3, P1.4, U$1.3.3V_4, U$1.3.3V_5, U$1.3.3V_6; no longer J2.1, J2.3, J2.5, J2.7
- net DEPTHSCL: now also DEPTH_SENSOR.2; no longer DEPTH_SENSOR.3
- net DEPTHSDA: now also DEPTH_SENSOR.3; no longer DEPTH_SENSOR.2
- net GND: now also HBL1.2, HBL2.2, RESET.S1; no longer HEARTBEAT1.K2, HEARTBEAT2.K2, S2.1
- net JTAG15: now also RESET.P, RESET.P1; no longer S2.2
- net MISSION_START: now also P1.8; no longer J2.2
- net N$14: now also HBL2.1; no longer HEARTBEAT2.A2
- net SDIO_CMD: now also J5.CMD(DI); no longer J5.CD/DAT3(!CS!)
- net SWITCH_3: now also P1.7; no longer J2.4
- net SWITCH_4: now also P1.6; no longer J2.6
- net SWITCH_5: now also P1.5; no longer J2.8
Other:
- moved on the sheet: DEPTH_SENSOR, DS_R1, DS_R2

Commit message: Fixing USB lines, we RF now boyz
Parts:
- added D+PULL, D-PULL: 1.5k, resistor:R-US_0204/7
- added D+SERIES, D-SERIES: 22Ohm, resistor:R-US_0204/7
- RHB1: value 330 -> 1k; device SparkFun-Resistors:1KOHM-VERT-1/4W-1% -> SparkFun-Resistors:1KOHM-HORIZ-1/4W-1%
- RHB2: value 330 -> 1k; device SparkFun-Resistors:1KOHM-VERT-1/4W-1% -> SparkFun-Resistors:1KOHM-HORIZ-1/4W-5%
Connections:
- new net D+CON: D+PULL.1, D+SERIES.2, J1.D+
- new net D-CON: D-PULL.1, D-SERIES.2, J1.D-
- net 3.3V: now also D+PULL.2, D-PULL.2
- net USB_OTG_HS_DM: now also D-SERIES.1; no longer J1.D-
- net USB_OTG_HS_DP: now also D+SERIES.1; no longer J1.D+
Other:
- moved on the sheet: J1

Commit message: Trace clean up
Parts:
- D+SERIES, D-SERIES: value 22Ohm -> 22Ω
Changed lines of the file:
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@@
 <part name="HBL2" library="SparkFun-Resistors" deviceset="1KOHM" device="-VERT-1/4W-1%" value="LED"/>
 <part name="HBL1" library="SparkFun-Resistors" deviceset="1KOHM" device="-VERT-1/4W-1%" value="LED"/>
-<part name="D+SERIES" library="resistor" library_urn="urn:adsk.eagle:library:348" deviceset="R-US_" device="0204/7" package3d_urn="urn:adsk.eagle:package:25945/1" value="22Ohm"/>
-<part name="D-SERIES" library="resistor" library_urn="urn:adsk.eagle:library:348" deviceset="R-US_" device="0204/7" package3d_urn="urn:adsk.eagle:package:25945/1" value="22Ohm"/>
+<part name="D+SERIES" library="resistor" library_urn="urn:adsk.eagle:library:348" deviceset="R-US_" device="0204/7" package3d_urn="urn:adsk.eagle:package:25945/1" value="22Ω"/>
+<part name="D-SERIES" library="resistor" library_urn="urn:adsk.eagle:library:348" deviceset="R-US_" device="0204/7" package3d_urn="urn:adsk.eagle:package:25945/1" value="22Ω"/>
 <part name="D-PULL" library="resistor" library_urn="urn:adsk.eagle:library:348" deviceset="R-US_" device="0204/7" package3d_urn="urn:adsk.eagle:package:25945/1" value="1.5k"/>
 <part name="D+PULL" library="resistor" library_urn="urn:adsk.eagle:library:348" deviceset="R-US_" device="0204/7" package3d_urn="urn:adsk.eagle:package:25945/1" value="1.5k"/>

Commit message: Future proofing
Parts:
- added USB_ID: 0Ω, resistor:R-US_0204/7
Connections:
- new net OTG_ID: IC1.PB12, USB_ID.1
- new net OTG_ID_CON: J1.ID, USB_ID.2
Changed lines of the file:
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@@
 <part name="D+PULL" library="resistor" library_urn="urn:adsk.eagle:library:348" deviceset="R-US_" device="0204/7" package3d_urn="urn:adsk.eagle:package:25945/1" value="1.5k"/>
 <part name="3.3V1" library="supply1" library_urn="urn:adsk.eagle:library:371" deviceset="+3V3" device=""/>
+<part name="USB_ID" library="resistor" library_urn="urn:adsk.eagle:library:348" deviceset="R-US_" device="0204/7" package3d_urn="urn:adsk.eagle:package:25945/1" value="0Ω"/>
 </parts>
 <sheets>
@@
 <instance part="D+PULL" gate="G$1" x="289.56" y="175.26" rot="R90"/>
 <instance part="3.3V1" gate="G$1" x="284.48" y="187.96"/>
+<instance part="USB_ID" gate="G$1" x="243.84" y="160.02"/>
 </instances>
 <busses>
@@
 </segment>
 </net>
+<net name="OTG_ID" class="0">
+<segment>
+<pinref part="IC1" gate="G$1" pin="PB12"/>
+<wire x1="200.66" y1="160.02" x2="238.76" y2="160.02" width="0.1524" layer="91"/>
+<pinref part="USB_ID" gate="G$1" pin="1"/>
+</segment>
+</net>
+<net name="OTG_ID_CON" class="0">
+<segment>
+<pinref part="USB_ID" gate="G$1" pin="2"/>
+<pinref part="J1" gate="G$1" pin="ID"/>
+<wire x1="248.92" y1="160.02" x2="297.18" y2="160.02" width="0.1524" layer="91"/>
+</segment>
+</net>
