File: coProcessor/Coprocessor_Board_Rev2 - Copy.brd (EAGLE design)
At the start: 101.6 x 101.6 mm, 94 parts, among them IC1 STM32F405RGT6, J1 USB_MINI-B_SMT, J4 30320-6002HB, J5 5008730806, Q1 L78M05CV, U1 MAX3051ESA

Commit message: 2 pin connector for can. please check... USB moved No usb id line Different switch connector, custom-made 12 pin package Esc names horizontal LEDs for programming Pushbutton for programming 4 leds , 1 pushbutton
Parts:
- removed CAN_OUT_HEADER: (no value), Wurth_Elektronik_Electromechanic_Board_to_Board_Connectors_rev16a:61300211821
- removed PA4LED, PA5LED, PC4LED, PC5LED: LED, SparkFun-Resistors:AXIAL-0.1
- removed RESET1: (no value), switch-omron:B3F-10XX
- removed RPA4, RPA5, RPC4, RPC5: 1k, SparkFun-Resistors:AXIAL-0.3
- removed U$2: 105314-2112, 105314-2112 nanofit hdr:105314-2112
- added P1: 39-30-08?, con-molex-mini-fit:39-30-?08?
- added USB_ID: 0Ω, resistor:0204/7
- RHB3: value 1.5k -> 7k
- moved RHB3 82.5 mm to (74.5, 12.9), turned to 180 degrees
- moved RHB4 21.8 mm to (56.3, 98.6)
- moved 3.3VSENS 17.2 mm to (46.9, 99.0)
- moved J1 11.2 mm to (7.09, 86.7), turned to 0 degrees
- moved ESC10 9.31 mm to (99.0, 91.8), turned to 270 degrees
- moved ESC2 8.00 mm to (99.0, 27.8), turned to 270 degrees
- moved ESC3 8.00 mm to (99.0, 35.8), turned to 270 degrees
- moved ESC4 8.00 mm to (99.0, 43.8), turned to 270 degrees
- moved ESC5 8.00 mm to (99.0, 51.8), turned to 270 degrees
- moved ESC6 8.00 mm to (99.0, 59.8), turned to 270 degrees
- moved ESC7 8.00 mm to (99.0, 67.8), turned to 270 degrees
- moved ESC8 8.00 mm to (99.0, 75.8), turned to 270 degrees
- moved ESC9 8.00 mm to (99.0, 83.8), turned to 270 degrees
- moved BATVSENS 7.44 mm to (84.9, 99.3)
- moved ESC1 6.78 mm to (99.0, 19.8), turned to 270 degrees
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Connections:
- removed net +3V3: U$2.CK10, U$2.CK11, U$2.CK12, U$2.CK7, U$2.CK8, U$2.CK9
- removed net HEARTBEAT_3: IC1.20, RPA4.P$1
- removed net HEARTBEAT_4: IC1.21, RPA5.P$1
- removed net N$10: PC4LED.P$1, RPC4.P$2
- removed net N$11: PC5LED.P$1, RPC5.P$2
- removed net N$12: IC1.62, RESET1.2
- removed net N$7: PA4LED.P$1, RPA4.P$2
- removed net N$8: PA5LED.P$1, RPA5.P$2
- removed net N$9: RESET1.3, RESET1.4
- removed net PC4: IC1.24, RPC4.P$1
- removed net PC5: IC1.25, RPC5.P$1
- new net OTG_ID: IC1.33, USB_ID.1
- new net OTG_ID_CON: J1.ID, USB_ID.2
- net 18V: now also RHB3.P$2
- net 3.3V: now also P1.1, P1.2, P1.3, P1.4
- net 5V: no longer RHB3.P$1
- net CANH: no longer CAN_OUT_HEADER.2
- net CANL: no longer CAN_OUT_HEADER.1
- net GND: no longer PA4LED.P$2, PA5LED.P$2, PC4LED.P$2, PC5LED.P$2
- net GNDA: now also BATVSENS.P$1; no longer BATVSENS.P$2
- net MISSION_START: now also P1.8; no longer U$2.CK6
- net N$3: now also BATVSENS.P$2, RHB3.P$1; no longer BATVSENS.P$1, RHB3.P$2
- net SWITCH_3: now also P1.7; no longer U$2.CK5
- net SWITCH_4: now also P1.6; no longer U$2.CK4
- net SWITCH_5: now also P1.5; no longer U$2.CK3
Routing:
- net SWITCH_4: track 0.00 -> 51.0 mm
- net SWITCH_3: track 0.00 -> 46.6 mm
- net OTG_ID_CON: track 0.00 -> 41.1 mm, vias 0 -> 1
- net HEARTBEAT_3: track 32.2 -> 0.00 mm, vias 2 -> 0
- net HEARTBEAT_4: track 31.4 -> 0.00 mm, vias 2 -> 0
- net PC4: track 28.0 -> 0.00 mm, vias 2 -> 0
- net SWITCH_5: track 30.9 -> 55.5 mm
- net 3.3V: track 354.3 -> 375.9 mm
- net MISSION_START: track 25.8 -> 45.7 mm
- net PC5: track 18.0 -> 0.00 mm, vias 2 -> 0
- net 18V: track 61.4 -> 45.7 mm
- net D+CON: track 3.38 -> 18.3 mm
- net D-CON: track 19.1 -> 29.4 mm
- net SURGESTBDHI: track 48.7 -> 40.3 mm
- net N$3: track 7.39 -> 0.00 mm
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