File: coProcessor/Coprocessor_Board_Rev2 - Copy.sch (EAGLE design)
At the start: 95 parts, among them IC1 STM32F405RGT6, J1 USB_MINI-B_SMT, J4 30320-6002HB, J5 5008730806, P1 39-30-06, Q1 L78M05CV, U1 MAX3051ESA, X1 5566-12

Commit message: 2 pin connector for can. please check... USB moved No usb id line Different switch connector, custom-made 12 pin package Esc names horizontal LEDs for programming Pushbutton for programming 4 leds , 1 pushbutton
Parts:
- removed CAN_OUT_HEADER: (no value), Wurth_Elektronik_Electromechanic_Board_to_Board_Connectors_rev16a:61300211821
- removed PA4LED, PA5LED, PC4LED, PC5LED: LED, SparkFun-Resistors:1KOHM-VERT-1/4W-1%
- removed RESET1: (no value), switch-omron:10-XX
- removed RPA4, RPA5, RPC4, RPC5: 1k, SparkFun-Resistors:1KOHM-HORIZ-1/4W-1%
- removed X1: 5566-12, con-molex:5566-12
- added USB_ID: 0Ω, resistor:R-US_0204/7
- P1: value 39-30-06 -> 39-30-08; device con-molex-mini-fit:39-30-06 -> con-molex-mini-fit:39-30-08
- RHB3: value 1.5k -> 7k
Connections:
- removed net +3V3: P1.1, P1.2
- removed net HEARTBEAT_3: IC1.PA4, RPA4.1
- removed net HEARTBEAT_4: IC1.PA5, RPA5.1
- removed net N$10: PC4LED.1, RPC4.2
- removed net N$11: PC5LED.1, RPC5.2
- removed net N$12: IC1.PB9, RESET1.S1
- removed net N$7: PA4LED.1, RPA4.2
- removed net N$8: PA5LED.1, RPA5.2
- removed net N$9: RESET1.P, RESET1.P1
- removed net PC4: IC1.PC4, RPC4.1
- removed net PC5: IC1.PC5, RPC5.1
- new net OTG_ID: IC1.PB12, USB_ID.1
- new net OTG_ID_CON: J1.ID, USB_ID.2
- net 18V: now also RHB3.2
- net 3.3V: now also P1.1, P1.2, P1.3, P1.4
- net 5V: no longer RHB3.1
- net CANH: no longer CAN_OUT_HEADER.2
- net CANL: no longer CAN_OUT_HEADER.1
- net GND: no longer PA4LED.2, PA5LED.2, PC4LED.2, PC5LED.2
- net GNDA: now also BATVSENS.1; no longer BATVSENS.2
- net MISSION_START: now also P1.8; no longer P1.6
- net N$3: now also BATVSENS.2, RHB3.1; no longer BATVSENS.1, RHB3.2
- net SWITCH_3: now also P1.7; no longer P1.5
- net SWITCH_4: now also P1.6; no longer P1.4
- net SWITCH_5: now also P1.5; no longer P1.3
Other:
- moved on the sheet: BATVSENS, RHB3
