File: coProcessor/Coprocessor_Board_Rev2.sch (EAGLE design)
At the start: 103 parts, among them IC1 STM32F405RGT6, J1 USB_MINI-B_SMT, J4 30320-6002HB, J5 5008730806, P1 39-30-08, Q1 L78M05CV

Commit message: Rev 2 of Coprocessor Board (No IMU) 1.fixed wires that were flipped. JTAG 5 fixed to pin 50. JTAG 7 fixed to pin 46 2.LEDs for power 3.CAN 4.LEDs for CAN 5.Swapped Through-Hole Resistors with more spaced packages. 6.Simplified the Opto-couplers 7.IMU yet to be added
Parts:
- removed DS_R1, DS_R2: 4.7k, SparkFun-Resistors:1KOHM-VERT-1/4W-1%
- removed ORIN1, ORIN10, ORIN2, ORIN3, ORIN4, ORIN5, ORIN6, ORIN7, ORIN8, ORIN9: 220, SparkFun-Resistors:1KOHM-VERT-1/4W-1%
- removed RO10A, RO1A, RO2A, RO3A, RO4A, RO5A, RO6A, RO7A, RO8A, RO9A: 1k, SparkFun-Resistors:1KOHM-0603-1/10W-1%
- removed RO10B, RO10C, RO1B, RO1C, RO2B, RO2C, RO3B, RO3C, RO4B, RO4C, RO5B, RO5C, RO6B, RO6C, RO7B, RO7C, RO8B, RO8C, RO9B, RO9C: 10k, SparkFun-Resistors:1KOHM-0603-1/10W-1%
- removed T1, T10, T2, T3, T4, T5, T6, T7, T8, T9: (no value), transistor:-NPN-TO126V
- added 3.3VSENS, BATVSENS, CANH_LED, CANL_LED: LED, SparkFun-Resistors:1KOHM-VERT-1/4W-1%
- added CANH_OUT_R, CANL_OUT_R: 60, resistor:R-US_0204/7
- added CANH_R, CANL_R: 330, resistor:R-US_0204/7
- added CAN_SPLIT_C: 4700 pF, SparkFun-Capacitors:22PF-PTH-2.54MM-200V-5%
- added DS_1, DS_2: 4.7k, resistor:R-US_0204/7
- added OR1, OR10, OR2, OR3, OR4, OR5, OR6, OR7, OR8, OR9: 220, resistor:R-US_0204/7
- added RHB3: 7k, SparkFun-Resistors:1KOHM-HORIZ-1/4W-1%
- added RHB4: 1k, SparkFun-Resistors:1KOHM-HORIZ-1/4W-1%
- added RO1, RO10, RO2, RO3, RO4, RO5, RO6, RO7, RO8, RO9: 10k, resistor:R-US_0204/7
- added U1: MCP2561-E/P, Microchip-MCP2561-E_P:MCP2561-E/P
Connections:
- removed net GATE1: RO1A.1, T1.B
- removed net GATE10: RO10A.1, T10.B
- removed net GATE2: RO2A.1, T2.B
- removed net GATE3: RO3A.1, T3.B
- removed net GATE4: RO4A.1, T4.B
- removed net GATE5: RO5A.1, T5.B
- removed net GATE6: RO6A.1, T6.B
- removed net GATE7: RO7A.1, T7.B
- removed net GATE8: RO8A.1, T8.B
- removed net GATE9: RO9A.1, T9.B
- removed net POWER207: OI7.COL, RO7A.2, RO7B.1
- removed net POWER208: OI8.COL, RO8A.2, RO8B.1
- removed net POWER2O1: OI1.COL, RO1A.2, RO1B.1
- removed net POWER2O10: OI10.COL, RO10A.2, RO10B.1
- removed net POWER2O2: OI2.COL, RO2A.2, RO2B.1
- removed net POWER2O3: OI3.COL, RO3A.2, RO3B.1
- removed net POWER2O4: OI4.COL, RO4A.2, RO4B.1
- removed net POWER2O5: OI5.COL, RO5A.2, RO5B.1
- removed net POWER2O6: OI6.COL, RO6A.2, RO6B.1
- removed net POWER2O9: OI9.COL, RO9A.2, RO9B.1
- removed net SOURCE1: ESC1.1, RO1C.1, T1.C
- removed net SOURCE10: ESC10.1, RO10C.1, T10.C
- removed net SOURCE2: ESC2.1, RO2C.1, T2.C
- removed net SOURCE3: ESC3.1, RO3C.1, T3.C
- removed net SOURCE4: ESC4.1, RO4C.1, T4.C
- removed net SOURCE5: ESC5.1, RO5C.1, T5.C
- removed net SOURCE6: ESC6.1, RO6C.1, T6.C
- removed net SOURCE7: ESC7.1, RO7C.1, T7.C
- removed net SOURCE8: ESC8.1, RO8C.1, T8.C
- removed net SOURCE9: ESC9.1, RO9C.1, T9.C
- new net CAN1_RXD: IC1.PA11, U1.RXD
- new net CAN1_TXD: IC1.PA12
- new net CANL: CANL_OUT_R.2, CANL_R.2, U$1.CAN_L, U1.CANL
- new net N$2: 3.3VSENS.1
- new net N$3: BATVSENS.2, RHB3.1
- new net N$4: 3.3VSENS.2, RHB4.1
- new net N$5: CANH_LED.1, CANH_R.1
- new net N$6: CANL_LED.2, CANL_R.1
- new net PWM5V1: ESC1.1, OI1.EMIT, RO1.2
- new net PWM5V10: ESC10.1, OI10.EMIT, RO10.2
- new net PWM5V2: ESC2.1, OI2.EMIT, RO2.2
- new net PWM5V3: ESC3.1, OI3.EMIT, RO3.2
- new net PWM5V4: ESC4.1, OI4.EMIT, RO4.2
- new net PWM5V5: ESC5.1, OI5.EMIT, RO5.2
- new net PWM5V6: ESC6.1, OI6.EMIT, RO6.2
- new net PWM5V7: ESC7.1, OI7.EMIT, RO7.2
- new net PWM5V8: ESC8.1, OI8.EMIT, RO8.2
- new net PWM5V9: ESC9.1, OI9.EMIT, RO9.2
- new net SPLIT: CANH_OUT_R.1, CANL_OUT_R.1, CAN_SPLIT_C.1
- net 18V: now also RHB3.2; no longer Q1.IN
- net 3.3V: now also DS_1.1, DS_2.1, RHB4.2; no longer DS_R1.2, DS_R2.2
- net 5V: now also OI1.COL, OI10.COL, OI2.COL, OI3.COL, OI4.COL, OI5.COL, OI6.COL, OI7.COL, OI8.COL, OI9.COL, U1.VDD; no longer RO10B.2, RO10C.2, RO1B.2, RO1C.2, RO2B.2, RO2C.2, RO3B.2, RO3C.2, RO4B.2, RO4C.2, RO5B.2, RO5C.2, RO6B.2, RO6C.2, RO7B.2, RO7C.2, RO8B.2, RO8C.2, RO9B.2, RO9C.2
- net CANH: now also CANH_OUT_R.2, CANH_R.2, U1.CANH
- net DEPTHSCL: now also DS_2.2; no longer DS_R2.1
- net DEPTHSDA: now also DS_1.2; no longer DS_R1.1
- net GNDBAT: now also BATVSENS.1, CANH_LED.2, CANL_LED.1, CAN_SPLIT_C.2, Q1.IN, RO1.1, RO10.1, RO2.1, RO3.1, RO4.1, RO5.1, RO6.1, RO7.1, RO8.1, RO9.1; no longer OI1.EMIT, OI10.EMIT, OI2.EMIT, OI3.EMIT, OI4.EMIT, OI5.EMIT, OI6.EMIT, OI7.EMIT, OI8.EMIT, OI9.EMIT, T1.E, T10.E, T2.E, T3.E, T4.E, T5.E, T6.E, T7.E, T8.E, T9.E
- net HEAVE_PORT_AFT: now also OR8.2; no longer ORIN8.1
- net HEAVE_PORT_FWD: now also OR7.2; no longer ORIN7.1
- net HEAVE_STBD_AFT: now also OR6.2; no longer ORIN6.1
- net HEAVE_STBD_FWD: now also OR5.2; no longer ORIN5.1
- net PWM1: now also OR1.1; no longer ORIN1.2
- net PWM10: now also OR10.1; no longer ORIN10.2
- net PWM2: now also OR2.1; no longer ORIN2.2
- net PWM3: now also OR3.1; no longer ORIN3.2
- net PWM4: now also OR4.1; no longer ORIN4.2
- net PWM5: now also OR5.1; no longer ORIN5.2
- net PWM6: now also OR6.1; no longer ORIN6.2
- net PWM7: now also OR7.1; no longer ORIN7.2
- net PWM8: now also OR8.1; no longer ORIN8.2
- net PWM9: now also OR9.1; no longer ORIN9.2
- net SURGEPORTHI: now also OR3.2; no longer ORIN3.1
- net SURGEPORTLOW: now also OR4.2; no longer ORIN4.1
- net SURGESTBDHI: now also OR1.2; no longer ORIN1.1
- net SURGESTBDLOW: now also OR2.2; no longer ORIN2.1
- net SW_AFT: now also OR9.2; no longer ORIN9.1
- net SW_FWD: now also OR10.2; no longer ORIN10.1
Other:
- moved on the sheet: ESC1, ESC10, ESC2, ESC3, ESC4, ESC5, ESC6, ESC7, ESC8, ESC9, Q1

Commit message: replaced 5v can tran with correct 3.3v
Parts:
- removed CAN_SPLIT_C: 4700 pF, SparkFun-Capacitors:22PF-PTH-2.54MM-200V-5%
- added CAN_VCC: .1 uF, SparkFun-Capacitors:22PF-PTH-2.54MM-200V-5%
- CANH_OUT_R, CANL_OUT_R: value 60 -> 120
- U1: value MCP2561-E/P -> MAX3051ESA; device Microchip-MCP2561-E_P:MCP2561-E/P -> MAX3051ESA:MAX3051ESA
Connections:
- removed net SPLIT: CANH_OUT_R.1, CANL_OUT_R.1, CAN_SPLIT_C.1
- net 3.3V: now also CAN_VCC.1, U1.VCC
- net 5V: no longer U1.VDD
- net CAN1_TXD: now also U1.TXD
- net CANH: now also CANH_OUT_R.1, CANL_OUT_R.1; no longer CANH_OUT_R.2
- net CANL: now also CANH_OUT_R.2
- net GND: now also CANH_LED.2, CANL_LED.1, CAN_VCC.2, U1.GND, U1.RS
- net GNDBAT: no longer CANH_LED.2, CANL_LED.1, CAN_SPLIT_C.2
Other:
- moved on the sheet: CANH_LED, CANH_OUT_R, CANH_R, CANL_LED, CANL_OUT_R

Commit message: 2 pin connector for can. please check... USB moved No usb id line Different switch connector, custom-made 12 pin package Esc names horizontal LEDs for programming Pushbutton for programming 4 leds , 1 pushbutton
Parts:
- removed P1: 39-30-08, con-molex-mini-fit:39-30-08
- removed USB_ID: 0Ω, resistor:R-US_0204/7
- added CAN_OUT_HEADER: (no value), Wurth_Elektronik_Electromechanic_Board_to_Board_Connectors_rev16a:61300211821
- added PA4LED, PA5LED, PC4LED, PC5LED: LED, SparkFun-Resistors:1KOHM-VERT-1/4W-1%
- added RESET1: (no value), switch-omron:10-XX
- added RPA4, RPA5, RPC4, RPC5: 1k, SparkFun-Resistors:1KOHM-HORIZ-1/4W-1%
- added U$2: 105314-2112, 105314-2112 nanofit hdr:105314-2112
- RHB3: value 7k -> 1.5k
Connections:
- removed net OTG_ID: IC1.PB12, USB_ID.1
- removed net OTG_ID_CON: J1.ID, USB_ID.2
- new net GNDA: BATVSENS.2
- new net HEARTBEAT_3: IC1.PA4, RPA4.1
- new net HEARTBEAT_4: IC1.PA5, RPA5.1
- new net N$10: PC4LED.1, RPC4.2
- new net N$11: PC5LED.1, RPC5.2
- new net N$12: IC1.PB9, RESET1.S1
- new net N$7: PA4LED.1, RPA4.2
- new net N$8: PA5LED.1, RPA5.2
- new net N$9: RESET1.P, RESET1.P1
- new net PC4: IC1.PC4, RPC4.1
- new net PC5: IC1.PC5, RPC5.1
- net 18V: now also Q1.IN; no longer RHB3.2
- net 3.3V: now also U$2.CK10, U$2.CK11, U$2.CK12, U$2.CK7, U$2.CK8, U$2.CK9; no longer P1.1, P1.2, P1.3, P1.4
- net 5V: now also RHB3.1
- net CANH: now also CAN_OUT_HEADER.2
- net CANL: now also CAN_OUT_HEADER.1
- net GND: now also PA4LED.2, PA5LED.2, PC4LED.2, PC5LED.2
- net GNDBAT: no longer BATVSENS.1, Q1.IN
- net MISSION_START: now also U$2.CK6; no longer P1.8
- net N$3: now also BATVSENS.1, RHB3.2; no longer BATVSENS.2, RHB3.1
- net SWITCH_3: now also U$2.CK5; no longer P1.7
- net SWITCH_4: now also U$2.CK4; no longer P1.6
- net SWITCH_5: now also U$2.CK3; no longer P1.5
Other:
- moved on the sheet: BATVSENS, RHB3

Commit message: added gpio pin connector, erc, fixed some air wires
Parts:
- removed CAN_OUT_HEADER: (no value), Wurth_Elektronik_Electromechanic_Board_to_Board_Connectors_rev16a:61300211821
- added GPIO: (no value), SparkFun-Connectors:CONN_03
- added J2: (no value), SparkFun-Connectors:CONN_02
- renumbered RESET1 to DEBUG
Connections:
- removed net N$2: 3.3VSENS.1
- new net PB8: GPIO.3, IC1.PB8
- new net PC13: GPIO.2, IC1.PC13
- new net PC14: GPIO.1, IC1.PC14
- net CANH: now also J2.2; no longer CAN_OUT_HEADER.2
- net CANL: now also J2.1; no longer CAN_OUT_HEADER.1
- net GND: now also 3.3VSENS.1
Changed lines of the file:
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@@
 <part name="GND24" library="supply1" library_urn="urn:adsk.eagle:library:371" deviceset="GND" device=""/>
 <part name="GND25" library="supply1" library_urn="urn:adsk.eagle:library:371" deviceset="GND" device=""/>
-<part name="CAN_OUT_HEADER" library="Wurth_Elektronik_Electromechanic_Board_to_Board_Connectors_rev16a" deviceset="61300211821" device=""/>
 <part name="GND26" library="supply1" library_urn="urn:adsk.eagle:library:371" deviceset="GND" device=""/>
 <part name="RPA4" library="SparkFun-Resistors" deviceset="1KOHM" device="-HORIZ-1/4W-1%" value="1k"/>
@@
 <part name="RPC5" library="SparkFun-Resistors" deviceset="1KOHM" device="-HORIZ-1/4W-1%" value="1k"/>
 <part name="PC5LED" library="SparkFun-Resistors" deviceset="1KOHM" device="-VERT-1/4W-1%" value="LED"/>
-<part name="RESET1" library="switch-omron" library_urn="urn:adsk.eagle:library:377" deviceset="10-XX" device="" package3d_urn="urn:adsk.eagle:package:27496/1"/>
+<part name="DEBUG" library="switch-omron" library_urn="urn:adsk.eagle:library:377" deviceset="10-XX" device="" package3d_urn="urn:adsk.eagle:package:27496/1"/>
 <part name="U$2" library="105314-2112 nanofit hdr" deviceset="105314-2112" device=""/>
+<part name="J2" library="SparkFun-Connectors" deviceset="CONN_02" device=""/>
+<part name="GPIO" library="SparkFun-Connectors" deviceset="CONN_03" device=""/>
 </parts>
 <sheets>
@@
 <instance part="GND24" gate="1" x="477.52" y="48.26"/>
 <instance part="GND25" gate="1" x="497.84" y="50.8"/>
-<instance part="CAN_OUT_HEADER" gate="G$1" x="520.7" y="86.36" rot="R270"/>
 <instance part="GND26" gate="1" x="251.46" y="292.1"/>
 <instance part="RPA4" gate="G$1" x="243.84" y="259.08" rot="R90"/>
@@
 <instance part="RPC5" gate="G$1" x="223.52" y="307.34" rot="R90"/>
 <instance part="PC5LED" gate="G$1" x="223.52" y="320.04" rot="R90"/>
-<instance part="RESET1" gate="1" x="223.52" y="337.82" rot="MR270"/>
+<instance part="DEBUG" gate="1" x="223.52" y="337.82" rot="MR270"/>
 <instance part="U$2" gate="G$1" x="-66.04" y="66.04"/>
+<instance part="J2" gate="G$1" x="515.62" y="76.2" rot="R90"/>
+<instance part="GPIO" gate="J$1" x="165.1" y="71.12" rot="R90"/>
 </instances>
 <busses>
@@
 <pinref part="PC5LED" gate="G$1" pin="2"/>
 <wire x1="223.52" y1="325.12" x2="223.52" y2="330.2" width="0.1524" layer="91"/>
+</segment>
+<segment>
+<pinref part="3.3VSENS" gate="G$1" pin="1"/>
+<wire x1="388.62" y1="73.66" x2="396.24" y2="73.66" width="0.1524" layer="91"/>
+<pinref part="GND21" gate="1" pin="GND"/>
 </segment>
 </net>
@@
 <segment>
 <pinref part="IC1" gate="G$1" pin="PC7"/>
-<wire x1="187.96" y1="160.02" x2="187.96" y2="170.18" width="0.1524" layer="91"/>
-<wire x1="187.96" y1="170.18" x2="231.14" y2="170.18" width="0.1524" layer="91"/>
-<wire x1="231.14" y1="170.18" x2="233.68" y2="172.72" width="0.1524" layer="91"/>
+<wire x1="187.96" y1="160.02" x2="187.96" y2="172.72" width="0.1524" layer="91"/>
 <pinref part="RHB2" gate="G$1" pin="1"/>
 <wire x1="248.92" y1="172.72" x2="248.92" y2="180.34" width="0.1524" layer="91"/>
-<wire x1="233.68" y1="172.72" x2="248.92" y2="172.72" width="0.1524" layer="91"/>
+<wire x1="187.96" y1="172.72" x2="248.92" y2="172.72" width="0.1524" layer="91"/>
 </segment>
 </net>
@@
 <pinref part="CANH_R" gate="G$1" pin="2"/>
 <wire x1="497.84" y1="78.74" x2="497.84" y2="76.2" width="0.1524" layer="91"/>
-<pinref part="CAN_OUT_HEADER" gate="G$1" pin="2"/>
 <wire x1="513.08" y1="86.36" x2="492.76" y2="86.36" width="0.1524" layer="91"/>
 <wire x1="492.76" y1="86.36" x2="492.76" y2="78.74" width="0.1524" layer="91"/>
+<pinref part="J2" gate="G$1" pin="2"/>
+<wire x1="513.08" y1="86.36" x2="513.08" y2="83.82" width="0.1524" layer="91"/>
 </segment>
 </net>
@@
 <wire x1="289.56" y1="170.18" x2="289.56" y2="162.56" width="0.1524" layer="91"/>
 <junction x="289.56" y="162.56"/>
-</segment>
-</net>
-<net name="N$2" class="0">
-<segment>
-<pinref part="3.3VSENS" gate="G$1" pin="1"/>
-<wire x1="388.62" y1="73.66" x2="396.24" y2="73.66" width="0.1524" layer="91"/>
-<pinref part="GND21" gate="1" pin="GND"/>
 </segment>
 </net>
@@
 <wire x1="477.52" y1="76.2" x2="477.52" y2="88.9" width="0.1524" layer="91"/>
 <wire x1="477.52" y1="88.9" x2="518.16" y2="88.9" width="0.1524" layer="91"/>
-<pinref part="CAN_OUT_HEADER" gate="G$1" pin="1"/>
-<wire x1="518.16" y1="88.9" x2="518.16" y2="86.36" width="0.1524" layer="91"/>
+<pinref part="J2" gate="G$1" pin="1"/>
+<wire x1="515.62" y1="83.82" x2="518.16" y2="83.82" width="0.1524" layer="91"/>
+<wire x1="518.16" y1="83.82" x2="518.16" y2="88.9" width="0.1524" layer="91"/>
 </segment>
 </net>
@@
 <net name="N$9" class="0">
 <segment>
-<pinref part="RESET1" gate="1" pin="P1"/>
-<pinref part="RESET1" gate="1" pin="P"/>
+<pinref part="DEBUG" gate="1" pin="P1"/>
+<pinref part="DEBUG" gate="1" pin="P"/>
 <wire x1="228.6" y1="335.28" x2="228.6" y2="337.82" width="0.1524" layer="91"/>
 </segment>
@@
 <wire x1="137.16" y1="185.42" x2="218.44" y2="185.42" width="0.1524" layer="91"/>
 <wire x1="218.44" y1="185.42" x2="218.44" y2="335.28" width="0.1524" layer="91"/>
-<pinref part="RESET1" gate="1" pin="S1"/>
+<pinref part="DEBUG" gate="1" pin="S1"/>
+</segment>
+</net>
+<net name="PC14" class="0">
+<segment>
+<pinref part="GPIO" gate="J$1" pin="1"/>
+<pinref part="IC1" gate="G$1" pin="PC14"/>
+<wire x1="167.64" y1="78.74" x2="167.64" y2="106.68" width="0.1524" layer="91"/>
+</segment>
+</net>
+<net name="PC13" class="0">
+<segment>
+<pinref part="IC1" gate="G$1" pin="PC13"/>
+<pinref part="GPIO" gate="J$1" pin="2"/>
+<wire x1="165.1" y1="106.68" x2="165.1" y2="78.74" width="0.1524" layer="91"/>
+</segment>
+</net>
+<net name="PB8" class="0">
+<segment>
+<pinref part="IC1" gate="G$1" pin="PB8"/>
+<wire x1="144.78" y1="121.92" x2="144.78" y2="78.74" width="0.1524" layer="91"/>
+<pinref part="GPIO" gate="J$1" pin="3"/>
+<wire x1="144.78" y1="78.74" x2="162.56" y2="78.74" width="0.1524" layer="91"/>
 </segment>
 </net>
@@
 </sheet>
 </sheets>
+<errors>
+</errors>
 </schematic>
 </drawing>
