File: coProcessor/Coprocessor_Board_Rev2.sch (EAGLE design)
At the start: 96 parts, among them IC1 STM32F405RGT6, J1 USB_MINI-B_SMT, J4 30320-6002HB, J5 5008730806, Q1 L78M05CV, U1 MAX3051ESA

Commit message: General cleanup (salutes) of the converter and copro eagle files
Parts:
- removed 18VLED, 3.3VLED: WHITE, SparkFun-LED:LED-WHITE1206
- removed RS: 0, resistor:R-US_0204/7
- added 3.3VSENS, BATVSENS: LED, SparkFun-Resistors:1KOHM-VERT-1/4W-1%
- C10, C2, C3, C4, C5: value .1 uF -> 100 nF
- GPIO: device SparkFun-Connectors:CONN_02 -> SparkFun-Connectors:CONN_03
- PA4LED, PA5LED, PC4LED, PC5LED: value WHITE -> LED; device SparkFun-LED:LED-WHITE1206 -> SparkFun-Resistors:1KOHM-VERT-1/4W-1%
- RHB3: value 1.8k -> 1.5k
- RHB4, RPA4, RPA5, RPC4, RPC5: value 330 -> 1k
- U$2: SPICEPREFIX X -> (none)
Connections:
- removed net N$2: RS.2, U1.RS
- removed net N$9: DEBUG.P, DEBUG.P1
- removed net SWITCH6: IC1.PC14, U$2.CK2
- new net GNDA: BATVSENS.2
- new net PC14: GPIO.1, IC1.PC14
- net GND: now also 3.3VSENS.1, PA4LED.2, PA5LED.2, PC4LED.2, PC5LED.2, U1.RS; no longer 3.3VLED.C, PA4LED.C, PA5LED.C, PC4LED.C, PC5LED.C, RS.1
- net GNDBAT: no longer 18VLED.C
- net N$10: now also PC4LED.1; no longer PC4LED.A
- net N$11: now also PC5LED.1; no longer PC5LED.A
- net N$3: now also BATVSENS.1; no longer 18VLED.A
- net N$4: now also 3.3VSENS.2; no longer 3.3VLED.A
- net N$7: now also PA4LED.1; no longer PA4LED.A
- net N$8: now also PA5LED.1; no longer PA5LED.A
- net PB8: now also GPIO.3; no longer GPIO.2
- net PB9: now also DEBUG.S
- net PC13: now also GPIO.2; no longer GPIO.1
Other:
- moved on the sheet: PA4LED, PA5LED, PC4LED, PC5LED
