File: coProcessor/CoprocessorBoard3.0.brd (EAGLE design)
At the start: 101.6 x 101.6 mm, 87 parts, among them IC1 STM32F405RGT6, J1 5008730806

Commit message: Mega cleanup and initial placement of rev3 parts
Parts:
- removed 5V_LED1: WHITE, SparkFun-LED:LED-0603
- removed 5V_R1: 1k, SparkFun-Resistors:AXIAL-0.3
- removed D+PULL, D-PULL: 1.5k, SparkFun-Resistors:AXIAL-0.3
- removed DEPTH_SENSOR: NANOFIT4PIN, nanofit 4pin:NANOFIT_4PIN
- removed ESC_CONNECTOR_1, ESC_CONNECTOR_3: 455-1750-1-ND, SparkFun-Connectors:1X03
- removed J1: 5008730806, 5008730806:5008730806
- removed OPTOCOUPLER_1, OPTOCOUPLER_3: SFH610, optocoupler:DIL04
- removed O_IN_1, O_IN_3: 220, SparkFun-Resistors:AXIAL-0.3
- removed O_R1, O_R3: 10k, SparkFun-Resistors:AXIAL-0.3
- added 3V_LED: WHITE, SparkFun-LED:LED-0603
- added 3V_R: 1k, SparkFun-Resistors:AXIAL-0.3
- added U$2: NANOFIT_4PIN_STR, nanofit_4pin_str:NANOFIT_4PIN_STR
- CPC1: value 100nF -> 0.1uF
- CPC3: device SparkFun-Capacitors:1206 -> SparkFun-Capacitors:0603
- CPC5, CPC6, CPC7, CPC8: value 1nF -> 0.1uF
- moved ESC_CONNECTOR_10 197.8 mm to (94.0, 83.8), turned to 0 degrees
- moved ESC_CONNECTOR_8 196.7 mm to (94.0, 66.0), turned to 0 degrees
- moved ESC_CONNECTOR_2 196.2 mm to (94.0, 21.6), turned to 0 degrees
- moved ESC_CONNECTOR_7 194.1 mm to (94.0, 57.1), turned to 0 degrees
- moved ESC_CONNECTOR_5 189.5 mm to (94.0, 39.4), turned to 0 degrees
- moved ESC_CONNECTOR_9 189.2 mm to (94.0, 74.9), turned to 0 degrees
- moved ESC_CONNECTOR_6 185.0 mm to (94.0, 48.3), turned to 0 degrees
- moved ESC_CONNECTOR_4 181.0 mm to (94.0, 30.5), turned to 0 degrees
- moved CPC2 179.0 mm to (53.7, 52.4)
- moved CPC1 175.9 mm to (42.3, 47.9), turned to 180 degrees
- moved CPC6 173.6 mm to (55.9, 52.4)
- moved O_R6 172.0 mm to (87.6, 44.5), turned to 270 degrees
- moved O_R5 171.7 mm to (90.2, 35.6), turned to 270 degrees
- moved O_R2 171.5 mm to (90.2, 17.8), turned to 270 degrees
- moved O_R4 170.9 mm to (87.6, 26.7), turned to 270 degrees
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Connections:
- removed net +3.3V: D+PULL.P$2, D-PULL.P$2, DEPTH_SENSOR.CKT_1, J1.4, JTAG_CONNECTOR.1, JTAG_CONNECTOR.2, POWER_JACK.1.1, POWER_JACK.1.2, R_DS_1.P$2, R_DS_2.P$2, SWITCH_CONNECTOR.CK10, SWITCH_CONNECTOR.CK11, SWITCH_CONNECTOR.CK12, SWITCH_CONNECTOR.CK7, SWITCH_CONNECTOR.CK8, SWITCH_CONNECTOR.CK9, U$1.3.3VP1, U$1.3.3VP2, U$1.3.3VP3, U$1.3.3V_4, U$1.3.3V_5, U$1.3.3V_6
- removed net GND1: 5V_LED.C
- removed net GNDA: U$1.EXTRA24, VOLTAGE_REGULATOR.2
- removed net GND_THRUSTER: ESC_CONNECTOR_1.3, ESC_CONNECTOR_10.3, ESC_CONNECTOR_2.3, ESC_CONNECTOR_3.3, ESC_CONNECTOR_4.3, ESC_CONNECTOR_5.3, ESC_CONNECTOR_6.3, ESC_CONNECTOR_7.3, ESC_CONNECTOR_8.3, ESC_CONNECTOR_9.3, O_R1.P$2, O_R10.P$2, O_R2.P$2, O_R3.P$2, O_R4.P$2, O_R5.P$2, O_R6.P$2, O_R7.P$2, O_R8.P$2, O_R9.P$2
- removed net N$1: ESC_CONNECTOR_1.1, OPTOCOUPLER_1.4, O_R1.P$1
- removed net N$20: OPTOCOUPLER_3.1, O_IN_3.P$2
- removed net N$22: OPTOCOUPLER_1.1, O_IN_1.P$2
- removed net N$35: CAP1.1, CAP2.1, IC1.31, IC1.47
- removed net N$5: ESC_CONNECTOR_3.1, OPTOCOUPLER_3.4, O_R3.P$1
- removed net V+: 5V_R1.P$1, CPC1.1, CPC2.1, CPC3.1, CPC5.1, CPC6.1, CPC7.1, CPC8.1, IC1.13, IC1.19, IC1.32, IC1.48, IC1.64
- new net 3V3: 3V_R.P$1, CPC1.1, CPC2.1, CPC3.1, CPC5.1, CPC6.1, CPC7.1, CPC8.1, IC1.13, IC1.19, IC1.32, IC1.48, IC1.64, JTAG_CONNECTOR.1, JTAG_CONNECTOR.2, POWER_JACK.1.1, POWER_JACK.1.2, R_DS_1.P$2, R_DS_2.P$2, SWITCH_CONNECTOR.CK10, SWITCH_CONNECTOR.CK11, SWITCH_CONNECTOR.CK12, SWITCH_CONNECTOR.CK7, SWITCH_CONNECTOR.CK8, SWITCH_CONNECTOR.CK9, U$1.3.3VP1, U$1.3.3VP2, U$1.3.3VP3, U$1.3.3V_4, U$1.3.3V_5, U$1.3.3V_6, U$2.P$1
- new net GNDBAT: 5V_LED.C, ESC_CONNECTOR_10.3, ESC_CONNECTOR_2.3, ESC_CONNECTOR_4.3, ESC_CONNECTOR_5.3, ESC_CONNECTOR_6.3, ESC_CONNECTOR_7.3, ESC_CONNECTOR_8.3, ESC_CONNECTOR_9.3, O_R10.P$2, O_R2.P$2, O_R4.P$2, O_R5.P$2, O_R6.P$2, O_R7.P$2, O_R8.P$2, O_R9.P$2, U$1.EXTRA24, VOLTAGE_REGULATOR.2
- new net KILL_SWITCH: IC1.4, U$1.KILL_SWITCH
- new net VCAP1: CAP1.1, IC1.31
- new net VCAP2: CAP2.1, IC1.47
- net +5V: no longer OPTOCOUPLER_1.3, OPTOCOUPLER_3.3
- net D+CON: no longer D+PULL.P$1
- net D-CON: no longer D-PULL.P$1
- net DEPTHSCL: now also U$2.P$3; no longer DEPTH_SENSOR.CKT_2
- net DEPTHSDA: now also U$2.P$2; no longer DEPTH_SENSOR.CKT_3
- net GND: now also 3V_LED.C, U$2.P$4; no longer 5V_LED1.C, DEPTH_SENSOR.CKT_4, J1.6, J1.S3, J1.S4, OPTOCOUPLER_1.2, OPTOCOUPLER_3.2
- net N$43: now also 3V_LED.A, 3V_R.P$2; no longer 5V_LED1.A, 5V_R1.P$2
- net SDIO_CK: no longer J1.5
- net SDIO_CMD: no longer J1.3
- net SDIO_DO: no longer J1.7
- net SURGEPORTHI: no longer O_IN_3.P$1
- net SURGESTBDHI: no longer O_IN_1.P$1
- net SWITCH_3: now also SWITCH_CONNECTOR.CK5; no longer SWITCH_CONNECTOR.CK3
- net SWITCH_5: now also SWITCH_CONNECTOR.CK3; no longer SWITCH_CONNECTOR.CK5
- net USB_OTG_HS_DM: now also IC1.35
- net USB_OTG_HS_DP: now also IC1.36
Routing:
- net 3V3: track 0.00 -> 265.3 mm, vias 0 -> 3
- net +5V: track 0.00 -> 102.5 mm
- net GND: track 0.00 -> 81.3 mm, vias 0 -> 12
- net SWITCH_5: track 0.00 -> 61.2 mm
- net SWITCH_4: track 0.00 -> 60.3 mm
- net SWITCH_3: track 0.00 -> 59.7 mm
- net MISSION_START: track 0.00 -> 58.7 mm
- net GNDBAT: track 0.00 -> 57.3 mm, vias 0 -> 1
- net +18V: track 0.00 -> 55.3 mm
- net KILL_SWITCH: track 0.00 -> 55.0 mm, vias 0 -> 4
- net SURGESTBDLOW: track 0.00 -> 39.9 mm, vias 0 -> 2
- net SURGEPORTLOW: track 0.00 -> 34.2 mm, vias 0 -> 2
- net HEAVE_STBD_FWD: track 0.00 -> 33.8 mm
- net PB9: track 0.00 -> 28.9 mm
- net SW_FWD: track 0.00 -> 27.9 mm
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- added copper zone on layer 1, net 3V3
- added copper zone on layer 16, net 3V3
- added copper zone on layer 1, net GND
- added copper zone on layer 16, net GND
- added copper zone on layer 16, net GNDBAT
