File: Status Board/Status Board 0.4.brd (EAGLE design)
At the start: 172.7 x 55.9 mm, 47 parts

Commit message: Add files via upload
Parts:
- renumbered RSET_SETS_PEAK_CURRENT to RSET, SV1 to AD0, SV2 to AD1
Other:
- board text added: ":P"
- board text added: ">:-}"
- board text added: "Status Board -- Rev 1.0 Anthony Condo"
- board text added: "The Ohio State University Center For Automotive Research"
- board text added: "^_^"
Changed lines of the file:
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@@
 <rectangle x1="40.64" y1="11.176" x2="47.498" y2="17.78" layer="25"/>
 <rectangle x1="53.594" y1="11.176" x2="60.452" y2="17.78" layer="25"/>
+<text x="73.66" y="42.164" size="0.8128" layer="25">^_^</text>
+<text x="134.874" y="41.91" size="0.8128" layer="25">:P</text>
+<text x="14.478" y="40.894" size="0.8128" layer="25">&gt;:-}</text>
+<text x="1.27" y="55.118" size="2.54" layer="25">The Ohio State University
+Center For Automotive Research</text>
+<text x="56.134" y="55.118" size="2.54" layer="25">Status Board -- Rev 1.0
+Anthony Condo</text>
 </plain>
 <attributes>
@@
 <attribute name="OC_NEWARK" value="unknown" x="98.933" y="42.037" size="1.778" layer="27" display="off"/>
 </element>
-<element name="RSET_SETS_PEAK_CURRENT" library="resistor" library_urn="urn:adsk.eagle:library:348" package="0207/12" package3d_urn="urn:adsk.eagle:package:25938/1" value="" x="89.662" y="11.938"/>
+<element name="RSET" library="resistor" library_urn="urn:adsk.eagle:library:348" package="0207/12" package3d_urn="urn:adsk.eagle:package:25938/1" value="" x="89.662" y="11.938"/>
 <element name="U$2" library="5530843-6" package="5530843-6-BOARDFINGERS" value="5530843" x="122.174" y="71.12" rot="R180"/>
-<element name="MAX6955" library="MAX6955" package="SSOP36" value="MAX6955" x="92.4052" y="24.4348" rot="R270"/>
+<element name="MAX6955" library="MAX6955" package="SSOP36" value="MAX6955" x="92.4052" y="24.4348" smashed="yes" rot="R270">
+<attribute name="NAME" x="93.0402" y="22.7838" size="1.27" layer="25" rot="R90"/>
+<attribute name="VALUE" x="91.7702" y="30.1498" size="1.27" layer="27" rot="R270"/>
+</element>
 <element name="SW1" library="special" library_urn="urn:adsk.eagle:library:367" package="EDG-04" package3d_urn="urn:adsk.eagle:package:26655/2" value="" x="68.1228" y="14.1986"/>
 <element name="HUM0R" library="led" library_urn="urn:adsk.eagle:library:259" package="LED3MM" package3d_urn="urn:adsk.eagle:package:15797/1" value="" x="124.714" y="28.956" smashed="yes">
@@
 <attribute name="NAME" x="72.644" y="21.336" size="0.6096" layer="25" font="vector" ratio="20" rot="R270" align="bottom-center"/>
 </element>
-<element name="LS1" library="Buzzer-AI-1223-TWT-3V-2-R" package="BUZZER-12MM-NS" value="BUZZER-PTH_NO_SILK" x="105.918" y="25.654" rot="R292.5">
+<element name="LS1" library="Buzzer-AI-1223-TWT-3V-2-R" package="BUZZER-12MM-NS" value="BUZZER-PTH_NO_SILK" x="105.918" y="25.654" smashed="yes" rot="R292.5">
 <attribute name="PROD_ID" value="COMP-08253" x="105.918" y="25.654" size="1.778" layer="27" rot="R292.5" display="off"/>
 <attribute name="SF_SKU" value="COM-07950" x="105.918" y="25.654" size="1.778" layer="27" rot="R292.5" display="off"/>
 </element>
-<element name="SV1" library="con-lstb" library_urn="urn:adsk.eagle:library:162" package="MA03-1" package3d_urn="urn:adsk.eagle:package:8339/1" value="" x="78.74" y="20.066" rot="R180">
+<element name="AD0" library="con-lstb" library_urn="urn:adsk.eagle:library:162" package="MA03-1" package3d_urn="urn:adsk.eagle:package:8339/1" value="" x="78.74" y="20.066" smashed="yes" rot="R180">
 <attribute name="MF" value="" x="78.74" y="20.066" size="1.778" layer="27" rot="R180" display="off"/>
 <attribute name="MPN" value="" x="78.74" y="20.066" size="1.778" layer="27" rot="R180" display="off"/>
+<attribute name="NAME" x="82.55" y="18.415" size="1.27" layer="25" ratio="10" rot="R180"/>
 <attribute name="OC_FARNELL" value="unknown" x="78.74" y="20.066" size="1.778" layer="27" rot="R180" display="off"/>
 <attribute name="OC_NEWARK" value="unknown" x="78.74" y="20.066" size="1.778" layer="27" rot="R180" display="off"/>
-</element>
-<element name="SV2" library="con-lstb" library_urn="urn:adsk.eagle:library:162" package="MA03-1" package3d_urn="urn:adsk.eagle:package:8339/1" value="" x="78.74" y="14.224" rot="R180">
+<attribute name="VALUE" x="82.55" y="22.987" size="1.27" layer="27" ratio="10" rot="R180"/>
+</element>
+<element name="AD1" library="con-lstb" library_urn="urn:adsk.eagle:library:162" package="MA03-1" package3d_urn="urn:adsk.eagle:package:8339/1" value="" x="78.74" y="14.224" rot="R180">
 <attribute name="MF" value="" x="78.74" y="14.224" size="1.778" layer="27" rot="R180" display="off"/>
 <attribute name="MPN" value="" x="78.74" y="14.224" size="1.778" layer="27" rot="R180" display="off"/>
@@
 <signals>
 <signal name="GND">
-<contactref element="RSET_SETS_PEAK_CURRENT" pad="2"/>
+<contactref element="RSET" pad="2"/>
 <contactref element="U$2" pad="GND1"/>
 <contactref element="U$2" pad="GND2"/>
@@
 <wire x1="100.838" y1="14.859" x2="107.372196875" y2="21.393196875" width="0.1524" layer="16"/>
 <wire x1="107.372196875" y1="21.393196875" x2="107.372196875" y2="22.14325625" width="0.1524" layer="16"/>
-<contactref element="SV2" pad="1"/>
-<contactref element="SV1" pad="1"/>
+<contactref element="AD1" pad="1"/>
+<contactref element="AD0" pad="1"/>
 <wire x1="91.186" y1="15.494" x2="94.742" y2="11.938" width="0.508" layer="16"/>
 <wire x1="94.742" y1="11.938" x2="96.012" y2="11.938" width="0.508" layer="16"/>
@@
 <wire x1="81.28" y1="20.066" x2="82.1112" y2="19.2348" width="0.1524" layer="1"/>
 <wire x1="82.1112" y1="19.2348" x2="85.6672" y2="19.2348" width="0.1524" layer="1"/>
-<wire x1="113.7285" y1="67.945" x2="113.7285" y2="67.945" width="0" layer="19" extent="1-16"/>
-<wire x1="111.1885" y1="67.945" x2="113.7285" y2="67.945" width="0" layer="19" extent="1-1"/>
-<wire x1="111.1885" y1="67.945" x2="111.1885" y2="67.945" width="0" layer="19" extent="1-16"/>
-<wire x1="108.6485" y1="67.945" x2="111.1885" y2="67.945" width="0" layer="19" extent="1-1"/>
-<wire x1="108.6485" y1="67.945" x2="108.6485" y2="67.945" width="0" layer="19" extent="1-16"/>
-<wire x1="111.125" y1="63.754" x2="111.1885" y2="67.945" width="0" layer="19" extent="1-1"/>
 </signal>
 <signal name="N$20">
@@
 <wire x1="118.872" y1="64.008" x2="119.634" y2="63.246" width="0.508" layer="1"/>
 <wire x1="119.634" y1="63.246" x2="119.634" y2="27.0705375" width="0.508" layer="1"/>
-<contactref element="SV2" pad="3"/>
-<contactref element="SV1" pad="3"/>
+<contactref element="AD1" pad="3"/>
+<contactref element="AD0" pad="3"/>
 <wire x1="99.06" y1="17.6348" x2="91.8138" y2="10.3886" width="0.254" layer="1"/>
 <wire x1="76.2" y1="14.224" x2="76.2" y2="12.4206" width="0.1524" layer="1"/>
 <wire x1="76.2" y1="12.4206" x2="78.232" y2="10.3886" width="0.1524" layer="1"/>
 <wire x1="76.2" y1="14.224" x2="76.2" y2="20.066" width="0.1524" layer="16"/>
-<wire x1="121.3485" y1="67.945" x2="121.3485" y2="67.945" width="0" layer="19" extent="1-16"/>
-<wire x1="118.8085" y1="67.945" x2="121.3485" y2="67.945" width="0" layer="19" extent="1-1"/>
-<wire x1="118.8085" y1="67.945" x2="118.8085" y2="67.945" width="0" layer="19" extent="1-16"/>
-<wire x1="116.2685" y1="67.945" x2="118.8085" y2="67.945" width="0" layer="19" extent="1-1"/>
-<wire x1="116.2685" y1="67.945" x2="116.2685" y2="67.945" width="0" layer="19" extent="1-16"/>
-<wire x1="118.872" y1="64.008" x2="118.8085" y2="67.945" width="0" layer="19" extent="1-1"/>
 </signal>
 <signal name="N$21">
@@
 <wire x1="51.308" y1="13.208" x2="38.354" y2="13.208" width="0.1524" layer="16"/>
 <wire x1="38.354" y1="13.208" x2="25.4" y2="13.208" width="0.1524" layer="16"/>
-<wire x1="30.734" y1="22.86" x2="33.02" y2="22.86" width="0" layer="19" extent="1-16"/>
 <wire x1="87.6552" y1="20.8348" x2="85.5912" y2="20.8348" width="0.1524" layer="1"/>
 <wire x1="85.5912" y1="20.8348" x2="78.359" y2="28.067" width="0.1524" layer="1"/>
@@
 </signal>
 <signal name="N$46">
-<contactref element="RSET_SETS_PEAK_CURRENT" pad="1"/>
+<contactref element="RSET" pad="1"/>
 <contactref element="MAX6955" pad="17"/>
 <wire x1="85.852" y1="18.288" x2="86.106" y2="18.288" width="0.1524" layer="16"/>
@@
 <signal name="N$11">
 <contactref element="MAX6955" pad="3"/>
-<contactref element="SV1" pad="2"/>
+<contactref element="AD0" pad="2"/>
 <wire x1="78.74" y1="20.066" x2="78.74" y2="21.844" width="0.1524" layer="16"/>
 <wire x1="78.74" y1="21.844" x2="86.36" y2="29.464" width="0.1524" layer="16"/>
@@
 </signal>
 <signal name="N$12">
-<contactref element="SV2" pad="2"/>
+<contactref element="AD1" pad="2"/>
 <contactref element="MAX6955" pad="6"/>
 <wire x1="78.74" y1="14.224" x2="80.01" y2="15.494" width="0.1524" layer="16"/>
@@
 </drawing>
 <compatibility>
+<note version="6.3" minversion="6.2.2" severity="warning">
+Since Version 6.2.2 text objects can contain more than one line,
+which will not be processed correctly with this version.
+</note>
 <note version="8.2" severity="warning">
 Since Version 8.2, EAGLE supports online libraries. The ids
