File: Status Board/Status_Board.sch (EAGLE design)
At the start: 47 parts

Commit message: Added Final Bulk Decoupling cap, updated lables, Gerber files are not updated to reflect new cap yet.
Parts:
- added BULK: F, SparkFun-Capacitors:0.1UF-KIT-EZ-50V-20%
Connections:
- net GND: now also BULK.2
- net VCC: now also BULK.1
Changed lines of the file:
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@@
 <part name="P+5" library="supply1" library_urn="urn:adsk.eagle:library:371" deviceset="VCC" device=""/>
 <part name="GND7" library="supply1" library_urn="urn:adsk.eagle:library:371" deviceset="GND" device=""/>
+<part name="BULK" library="SparkFun-Capacitors" deviceset="0.1UF" device="-KIT-EZ-50V-20%" value="F"/>
 </parts>
 <sheets>
@@
 <instance part="P+5" gate="VCC" x="-170.18" y="194.31" rot="R270"/>
 <instance part="GND7" gate="1" x="-171.45" y="233.68" rot="R90"/>
+<instance part="BULK" gate="G$1" x="-223.52" y="95.25" rot="R270"/>
 </instances>
 <busses>
@@
 <wire x1="-218.44" y1="105.41" x2="-210.82" y2="105.41" width="0.1524" layer="91"/>
 <junction x="-210.82" y="105.41"/>
+<pinref part="BULK" gate="G$1" pin="1"/>
+<wire x1="-218.44" y1="95.25" x2="-218.44" y2="105.41" width="0.1524" layer="91"/>
+<junction x="-218.44" y="105.41"/>
 </segment>
 <segment>
@@
 <pinref part="GND6" gate="1" pin="GND"/>
 <wire x1="-226.06" y1="105.41" x2="-226.06" y2="111.76" width="0.1524" layer="91"/>
-</segment>
-<segment>
+<pinref part="BULK" gate="G$1" pin="2"/>
+<wire x1="-226.06" y1="105.41" x2="-226.06" y2="95.25" width="0.1524" layer="91"/>
+<junction x="-226.06" y="105.41"/>
+</segment>
+<segment>
