File: Status Board/Old Revs/Status Board 1.0.sch (EAGLE design)
At the start: 47 parts

Commit message: Updated lables position and content
Connections:
- net 013 renamed N$40
- net AD0 renamed N$11
- net AD1 renamed N$12
- net ISET renamed N$46
- net O0 renamed N$20
- net O1 renamed N$21
- net O10 renamed N$30
- net O11 renamed N$31
- net O12 renamed N$32
- net O14 renamed N$34
- net O15 renamed N$35
- net O16 renamed N$36
- net O17 renamed N$37
- net O18 renamed N$38
- net O2 renamed N$22
- net O3 renamed N$23
- net O4 renamed N$26
- net O5 renamed N$27
- net O6 renamed N$33
- net O7 renamed N$56
- net O8 renamed N$15
- net O9 renamed N$29
- net OSC renamed N$13
- net P0 renamed N$4
- net P1 renamed N$5
- net P2 renamed N$6
- net P3 renamed N$7
- net P4 renamed N$8
- net SCL renamed N$2
- net SDA renamed N$43
Changed lines of the file:
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@@
 </busses>
 <nets>
-<net name="O0" class="0">
+<net name="N$20" class="0">
 <segment>
 <wire x1="-63.5" y1="-1.27" x2="-109.22" y2="-1.27" width="0.1524" layer="91"/>
@@
 </segment>
 </net>
-<net name="O1" class="0">
+<net name="N$21" class="0">
 <segment>
 <wire x1="-205.74" y1="62.23" x2="-205.74" y2="1.27" width="0.1524" layer="91"/>
@@
 </segment>
 </net>
-<net name="O9" class="0">
+<net name="N$29" class="0">
 <segment>
 <wire x1="-182.88" y1="62.23" x2="-182.88" y2="21.59" width="0.1524" layer="91"/>
@@
 </segment>
 </net>
-<net name="O10" class="0">
+<net name="N$30" class="0">
 <segment>
 <wire x1="-180.34" y1="62.23" x2="-180.34" y2="24.13" width="0.1524" layer="91"/>
@@
 </segment>
 </net>
-<net name="O11" class="0">
+<net name="N$31" class="0">
 <segment>
 <wire x1="-177.8" y1="26.67" x2="-83.82" y2="26.67" width="0.1524" layer="91"/>
@@
 </segment>
 </net>
-<net name="O12" class="0">
+<net name="N$32" class="0">
 <segment>
 <wire x1="-175.26" y1="62.23" x2="-175.26" y2="29.21" width="0.1524" layer="91"/>
@@
 </segment>
 </net>
-<net name="O14" class="0">
+<net name="N$34" class="0">
 <segment>
 <wire x1="-170.18" y1="62.23" x2="-170.18" y2="34.29" width="0.1524" layer="91"/>
@@
 </segment>
 </net>
-<net name="O15" class="0">
+<net name="N$35" class="0">
 <segment>
 <wire x1="-167.64" y1="62.23" x2="-167.64" y2="36.83" width="0.1524" layer="91"/>
@@
 </segment>
 </net>
-<net name="O16" class="0">
+<net name="N$36" class="0">
 <segment>
 <wire x1="-165.1" y1="62.23" x2="-165.1" y2="39.37" width="0.1524" layer="91"/>
@@
 </segment>
 </net>
-<net name="O17" class="0">
+<net name="N$37" class="0">
 <segment>
 <wire x1="-162.56" y1="62.23" x2="-162.56" y2="41.91" width="0.1524" layer="91"/>
@@
 </segment>
 </net>
-<net name="O18" class="0">
+<net name="N$38" class="0">
 <segment>
 <wire x1="-160.02" y1="62.23" x2="-160.02" y2="44.45" width="0.1524" layer="91"/>
@@
 </segment>
 </net>
-<net name="013" class="0">
+<net name="N$40" class="0">
 <segment>
 <wire x1="-88.9" y1="31.75" x2="7.62" y2="31.75" width="0.1524" layer="91"/>
@@
 </segment>
 </net>
-<net name="O4" class="0">
+<net name="N$26" class="0">
 <segment>
 <wire x1="257.81" y1="-15.24" x2="255.27" y2="-15.24" width="0.1524" layer="91"/>
@@
 </segment>
 </net>
-<net name="O5" class="0">
+<net name="N$27" class="0">
 <segment>
 <wire x1="257.81" y1="-17.78" x2="252.73" y2="-17.78" width="0.1524" layer="91"/>
@@
 </segment>
 </net>
-<net name="O2" class="0">
+<net name="N$22" class="0">
 <segment>
 <wire x1="533.4" y1="-15.24" x2="530.86" y2="-15.24" width="0.1524" layer="91"/>
@@
 </segment>
 </net>
-<net name="O3" class="0">
+<net name="N$23" class="0">
 <segment>
 <wire x1="533.4" y1="-17.78" x2="528.32" y2="-17.78" width="0.1524" layer="91"/>
@@
 </segment>
 </net>
-<net name="O6" class="0">
+<net name="N$33" class="0">
 <segment>
 <wire x1="525.78" y1="-20.32" x2="533.4" y2="-20.32" width="0.1524" layer="91"/>
@@
 </segment>
 </net>
-<net name="O7" class="0">
+<net name="N$56" class="0">
 <segment>
 <wire x1="553.72" y1="-27.94" x2="556.26" y2="-27.94" width="0.1524" layer="91"/>
@@
 </segment>
 </net>
-<net name="SDA" class="0">
+<net name="N$43" class="0">
 <segment>
 <pinref part="U$2" gate="G$1" pin="SDA_ESC"/>
@@
 </segment>
 </net>
-<net name="ISET" class="0">
+<net name="N$46" class="0">
 <segment>
 <pinref part="RSET" gate="G$1" pin="1"/>
@@
 </segment>
 </net>
-<net name="SCL" class="0">
+<net name="N$2" class="0">
 <segment>
 <pinref part="MAX6955" gate="G$1" pin="SCL"/>
@@
 </segment>
 </net>
-<net name="P0" class="0">
+<net name="N$4" class="0">
 <segment>
 <pinref part="MAX6955" gate="G$1" pin="P0"/>
@@
 </segment>
 </net>
-<net name="P1" class="0">
+<net name="N$5" class="0">
 <segment>
 <pinref part="SW1" gate="A" pin="7"/>
@@
 </segment>
 </net>
-<net name="P2" class="0">
+<net name="N$6" class="0">
 <segment>
 <pinref part="SW1" gate="A" pin="6"/>
@@
 </segment>
 </net>
-<net name="P3" class="0">
+<net name="N$7" class="0">
 <segment>
 <pinref part="SW1" gate="A" pin="5"/>
@@
 </segment>
 </net>
-<net name="P4" class="0">
+<net name="N$8" class="0">
 <segment>
 <pinref part="MAX6955" gate="G$1" pin="P4"/>
@@
 </segment>
 </net>
-<net name="O8" class="0">
+<net name="N$15" class="0">
 <segment>
 <pinref part="DEP4B" gate="G$1" pin="A"/>
@@
 </segment>
 </net>
-<net name="OSC" class="0">
+<net name="N$13" class="0">
 <segment>
 <pinref part="C1" gate="G$1" pin="2"/>
@@
 </segment>
 </net>
-<net name="AD0" class="0">
+<net name="N$11" class="0">
 <segment>
 <pinref part="MAX6955" gate="G$1" pin="AD0"/>
@@
 </segment>
 </net>
-<net name="AD1" class="0">
+<net name="N$12" class="0">
 <segment>
 <pinref part="AD1" gate="G$1" pin="2"/>
