File: BatteryMonitor/Battery_Monitor.brd (EAGLE design)
At the start: 58.1 x 60.8 mm, 40 parts, among them IC1 MAX232

Commit message: Battery monitor board is updated with spi headers
Parts:
- added SPI_PINS: (no value), pinhead:2X03
- moved MEGA_RX 0.68 mm to (24.9, 35.3)
- moved SDA 0.53 mm to (23.0, 19.2)
- moved C1 0.53 mm to (13.9, 34.8)
- moved C2 0.53 mm to (13.9, 29.9)
- moved C6 0.53 mm to (14.4, 7.24)
- moved HUMIDITY 0.53 mm to (13.8, 10.6)
- moved R5 0.53 mm to (13.8, 23.4)
- moved R6 0.53 mm to (15.8, 19.1)
- moved C5 0.53 mm to (17.3, 7.75)
- moved SCL 0.53 mm to (21.2, 24.6)
- moved 16MHZ_CRYSTAL 0.53 mm to (17.3, 33.2)
Connections:
- new net MISO: ATMEGA.11, SPI_PINS.1
- new net MOSI: ATMEGA.10, SPI_PINS.3
- new net RESET: ATMEGA.13, SPI_PINS.4
- new net SCK: ATMEGA.9, SPI_PINS.5
- net 5V: now also SPI_PINS.2
- net GND: now also SPI_PINS.6
Routing:
- net SCK: track 0.00 -> 17.2 mm
- net RESET: track 0.00 -> 15.1 mm
- net MOSI: track 0.00 -> 13.9 mm
- net MISO: track 0.00 -> 11.1 mm
- net VBUS: track 40.9 -> 38.3 mm
- net MEGA_RX: track 26.3 -> 24.6 mm
- net 5V: track 314.0 -> 315.0 mm
- net GND: track 141.8 -> 142.7 mm
- net SDA: track 29.2 -> 29.8 mm
- net SCL: track 24.7 -> 25.2 mm
- net TAL1: track 15.4 -> 16.0 mm
- net TAL2: track 10.7 -> 11.2 mm
Other:
- board text added: "GND SCK RST MOSI 5V MISO"
