File: debugBoard/debugBoard.brd (EAGLE design)
At the start: 73.9 x 55.9 mm, 12 parts

Commit message: open invitation for august to mess with this layout before he yells at me
Parts:
- removed GND: 22-27-2021-02, con-molex:6410-02
- added OSCILLISCOPE_GND: 22-27-2021-02, con-molex:6410-02
Connections:
- net GND: now also OSCILLISCOPE_GND.1, OSCILLISCOPE_GND.2; no longer GND.1, GND.2
Routing:
- net SDA_DEPTH: track 57.0 -> 60.9 mm, vias 1 -> 0
- net GND: track 48.8 -> 52.1 mm
- net EXTRA1: track 24.3 -> 22.0 mm
Other:
- board size 73.9 x 55.9 mm -> 73.8 x 56 mm
Changed lines of the file:
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@@
 <setting verticaltext="up"/>
 </settings>
-<grid distance="0.005" unitdist="inch" unit="inch" style="lines" multiple="1" display="no" altdistance="0.0625" altunitdist="inch" altunit="inch"/>
+<grid distance="0.001" unitdist="inch" unit="inch" style="lines" multiple="1" display="no" altdistance="0.0625" altunitdist="inch" altunit="inch"/>
 <layers>
 <layer number="1" name="Top" color="4" fill="1" visible="yes" active="yes"/>
@@
 <board>
 <plain>
-<wire x1="14" y1="0" x2="87.6" y2="0" width="0.1524" layer="20"/>
-<wire x1="87.6" y1="0" x2="87.6" y2="7.8" width="0.1524" layer="20"/>
-<wire x1="87.6" y1="7.8" x2="87.884" y2="7.8" width="0.1524" layer="20"/>
+<wire x1="14.1016" y1="-0.0508" x2="87.8794" y2="-0.127" width="0.1524" layer="20"/>
+<wire x1="87.8794" y1="-0.127" x2="87.8794" y2="7.673" width="0.1524" layer="20"/>
+<wire x1="87.8794" y1="7.673" x2="87.884" y2="7.8" width="0.1524" layer="20"/>
 <wire x1="87.884" y1="7.8" x2="87.884" y2="55.88" width="0.1524" layer="20"/>
 <wire x1="87.884" y1="55.88" x2="14.097" y2="55.88" width="0.1524" layer="20"/>
 <wire x1="14.097" y1="55.88" x2="14.097" y2="7.8" width="0.1524" layer="20"/>
-<wire x1="14.097" y1="7.8" x2="14" y2="7.8" width="0.1524" layer="20"/>
-<wire x1="14" y1="7.8" x2="14" y2="0" width="0.1524" layer="20"/>
+<wire x1="14.097" y1="7.8" x2="14.1016" y2="7.7492" width="0.1524" layer="20"/>
+<wire x1="14.1016" y1="7.7492" x2="14.1016" y2="-0.0508" width="0.1524" layer="20"/>
 <text x="15.113" y="53.086" size="1.778" layer="21">UNDERWATER ROBOTICS</text>
 <text x="85.217" y="53.848" size="1.778" layer="21" rot="R270">CENTER FOR AUTOMOTIVE RESEARCH</text>
@@
 <attribute name="OC_NEWARK" value="unknown" x="19.431" y="21.209" size="1.778" layer="27" display="off"/>
 </element>
-<element name="GND" library="con-molex" library_urn="urn:adsk.eagle:library:165" package="6410-02" value="22-27-2021-02" x="49.276" y="37.338">
-<attribute name="MF" value="" x="49.276" y="37.338" size="1.778" layer="27" display="off"/>
-<attribute name="MPN" value="" x="49.276" y="37.338" size="1.778" layer="27" display="off"/>
-<attribute name="OC_FARNELL" value="unknown" x="49.276" y="37.338" size="1.778" layer="27" display="off"/>
-<attribute name="OC_NEWARK" value="unknown" x="49.276" y="37.338" size="1.778" layer="27" display="off"/>
+<element name="OSCILLISCOPE_GND" library="con-molex" library_urn="urn:adsk.eagle:library:165" package="6410-02" value="22-27-2021-02" x="52.5272" y="37.465">
+<attribute name="MF" value="" x="52.5272" y="37.465" size="1.778" layer="27" display="off"/>
+<attribute name="MPN" value="" x="52.5272" y="37.465" size="1.778" layer="27" display="off"/>
+<attribute name="OC_FARNELL" value="unknown" x="52.5272" y="37.465" size="1.778" layer="27" display="off"/>
+<attribute name="OC_NEWARK" value="unknown" x="52.5272" y="37.465" size="1.778" layer="27" display="off"/>
 </element>
 <element name="GROUND" library="con-molex" library_urn="urn:adsk.eagle:library:165" package="6410-02" value="22-27-2021-02" x="27.813" y="21.209">
@@
 <contactref element="GROUND" pad="2"/>
 <contactref element="GROUND" pad="1"/>
-<contactref element="GND" pad="2"/>
-<contactref element="GND" pad="1"/>
+<contactref element="OSCILLISCOPE_GND" pad="2"/>
+<contactref element="OSCILLISCOPE_GND" pad="1"/>
 <polygon width="0.1524" layer="16">
 <vertex x="23.495" y="10.16"/>
@@
 </polygon>
 <wire x1="26.543" y1="21.209" x2="29.083" y2="21.209" width="1.27" layer="16"/>
-<wire x1="48.006" y1="37.338" x2="50.546" y2="37.338" width="1.016" layer="16"/>
+<wire x1="51.2572" y1="37.465" x2="53.7972" y2="37.465" width="1.016" layer="16"/>
 <wire x1="26.543" y1="21.209" x2="26.8605" y2="20.8915" width="0.508" layer="16"/>
 <wire x1="26.8605" y1="20.8915" x2="26.8605" y2="3.175" width="0.508" layer="16"/>
 <wire x1="29.083" y1="21.209" x2="45.212" y2="37.338" width="0.508" layer="16"/>
-<wire x1="45.212" y1="37.338" x2="48.006" y2="37.338" width="0.508" layer="16"/>
+<wire x1="45.212" y1="37.338" x2="51.2572" y2="37.465" width="0.508" layer="16"/>
 <wire x1="24.3205" y1="3.175" x2="24.3205" y2="3.175" width="0" layer="19" extent="1-16"/>
 </signal>
@@
 <contactref element="U$1" pad="EXTRA1"/>
 <contactref element="TESTPOINTS" pad="1"/>
-<wire x1="31.877" y1="3.2385" x2="31.877" y2="16.637" width="0.3048" layer="16"/>
-<wire x1="31.877" y1="3.2385" x2="31.9405" y2="3.175" width="0.3048" layer="16"/>
-<wire x1="31.877" y1="16.637" x2="36.83" y2="21.59" width="0.254" layer="16"/>
-<wire x1="36.83" y1="21.59" x2="40.64" y2="21.59" width="0.254" layer="16"/>
+<wire x1="31.9405" y1="3.175" x2="31.9405" y2="11.3919" width="0.254" layer="16"/>
+<wire x1="31.9405" y1="11.3919" x2="40.5892" y2="20.0406" width="0.254" layer="16"/>
+<wire x1="40.5892" y1="20.0406" x2="40.5892" y2="21.5392" width="0.254" layer="16"/>
+<wire x1="40.5892" y1="21.5392" x2="40.64" y2="21.59" width="0.254" layer="16"/>
 </signal>
 <signal name="EXTRA3">
@@
 <contactref element="SDA_DEPTH" pad="1"/>
 <contactref element="U$1" pad="SDA_DEPTH"/>
-<wire x1="52.705" y1="49.403" x2="52.705" y2="41.148" width="0.4064" layer="1"/>
 <wire x1="50.292" y1="49.53" x2="52.832" y2="49.53" width="0.4064" layer="16"/>
-<via x="52.705" y="49.403" extent="1-16" drill="0.35"/>
-<wire x1="52.705" y1="41.148" x2="72.5805" y2="21.2725" width="0.4064" layer="1"/>
-<wire x1="72.5805" y1="21.2725" x2="72.5805" y2="3.175" width="0.4064" layer="1"/>
-<wire x1="52.705" y1="49.403" x2="52.832" y2="49.53" width="0" layer="19" extent="1-1"/>
+<wire x1="52.832" y1="49.53" x2="55.5752" y2="49.53" width="0.4064" layer="1"/>
+<wire x1="65.532" y1="39.5732" x2="65.532" y2="31.3436" width="0.4064" layer="1"/>
+<wire x1="65.532" y1="31.3436" x2="72.6186" y2="24.257" width="0.4064" layer="1"/>
+<wire x1="72.6186" y1="24.257" x2="72.6186" y2="2.159" width="0.4064" layer="1"/>
+<wire x1="72.6186" y1="2.159" x2="72.5424" y2="2.0828" width="0.4064" layer="1"/>
+<wire x1="72.5424" y1="2.0828" x2="72.5424" y2="3.1369" width="0.4064" layer="1"/>
+<wire x1="72.5424" y1="3.1369" x2="72.5805" y2="3.175" width="0.4064" layer="1"/>
+<wire x1="55.5752" y1="49.53" x2="65.532" y2="39.5732" width="0.4064" layer="1"/>
 </signal>
 <signal name="SCL_DEPTH">
@@
 <contactref element="U$1" pad="SCL_DEPTH"/>
 <wire x1="59.055" y1="49.276" x2="61.595" y2="49.276" width="0.508" layer="1"/>
-<wire x1="61.595" y1="49.276" x2="66.294" y2="44.577" width="0.4064" layer="1"/>
-<wire x1="66.294" y1="44.577" x2="66.294" y2="31.877" width="0.4064" layer="1"/>
-<wire x1="66.294" y1="31.877" x2="75.1205" y2="23.0505" width="0.4064" layer="1"/>
-<wire x1="75.1205" y1="23.0505" x2="75.1205" y2="3.175" width="0.4064" layer="1"/>
+<wire x1="61.595" y1="49.276" x2="61.595" y2="45.0342" width="0.4064" layer="1"/>
+<wire x1="61.595" y1="45.0342" x2="66.421" y2="40.2082" width="0.4064" layer="1"/>
+<wire x1="66.421" y1="40.2082" x2="66.421" y2="31.8008" width="0.4064" layer="1"/>
+<wire x1="66.421" y1="31.8008" x2="75.057" y2="23.1648" width="0.4064" layer="1"/>
+<wire x1="75.057" y1="23.1648" x2="75.057" y2="3.2385" width="0.4064" layer="1"/>
+<wire x1="75.057" y1="3.2385" x2="75.1205" y2="3.175" width="0.4064" layer="1"/>
 </signal>
 <signal name="SDA_SENSOR">
