File: acoustics/Nice Acoustics/acoustics.brd (EAGLE design)
At the start: 120 x 80 mm, 176 parts, among them P1 22-23-2021, X1 22-23-2021, X2 22-23-2021, X3 22-23-2021, X4 22-23-2021

Commit message: Labelled Acoustics input connectors.
Parts:
- moved PF_R12 29.4 mm to (70.2, -37.4)
- renumbered H4_PREAMP2 to PA_PREAMP2, H4_PREAMP3 to SF_PREAMP3, X1 to PF_IN, X2 to PA_IN, X3 to SF_IN, X4 to SA_IN

Commit message: Changing Labels and fixing Layout of Acoustic board (#102)
Parts:
- moved ADC_PF 527.0 mm to (104.6, 31.7), turned to 270 degrees
- moved PF_REFGEN 372.1 mm to (85.2, 29.4), turned to 270.9 degrees
- moved PF_PREAMP 274.5 mm to (108.5, 65.7), turned to 178.4 degrees
- moved PF_R8 135.8 mm to (108.6, 54.8), turned to 270 degrees
- moved PF_C8 133.2 mm to (107.8, 48.3), turned to 180 degrees
- moved PF_R9 123.1 mm to (108.7, 51.0), turned to 270 degrees
- moved PF_DA 119.6 mm to (105.4, 58.9), turned to 270 degrees
- moved PF_R13 99.5 mm to (106.8, 51.0), turned to 270 degrees
- moved PF_R12 99.3 mm to (106.7, 54.9), turned to 270 degrees
- moved PF_C5 39.4 mm to (24.3, 31.5)
Routing:
- net N$88: track 0.00 -> 2.23 mm
- net N$109: track 0.00 -> 2.11 mm
- net DIFF_P_PF: track 0.00 -> 1.95 mm
- net DIFF_N_PF: track 0.00 -> 1.90 mm
- net N$102: track 0.00 -> 1.81 mm
- net N$97: track 0.00 -> 1.76 mm
- net +3V3: track 0.00 -> 1.70 mm, vias 0 -> 1
- net GND: track 0.00 -> 1.50 mm, vias 0 -> 1
Other:
- outline, holes or cut-outs redrawn

Commit message: Added more connections (#103)
Parts:
- moved PF_R2 297.2 mm to (106.0, 67.1), turned to 270 degrees
- moved PF_R1 296.6 mm to (107.8, 70.3), turned to 270 degrees
- moved PF_C1 293.4 mm to (108.0, 67.1), turned to 270 degrees
- moved PF_R6 159.1 mm to (109.0, 64.0), turned to 270 degrees
- moved PF_R10 150.5 mm to (106.9, 64.1), turned to 270 degrees
- moved PF_R11 138.7 mm to (105.2, 61.0), turned to 270 degrees
- moved PF_C7 132.7 mm to (107.9, 60.1), turned to 180 degrees
- moved PF_C6 129.5 mm to (107.9, 61.7), turned to 180 degrees
- moved PF_R7 124.4 mm to (110.1, 60.9), turned to 270 degrees
- moved PF_R14 99.0 mm to (103.1, 61.0), turned to 270 degrees
- moved PF_R5 97.0 mm to (112.2, 60.9), turned to 270 degrees
- moved PF_C9 92.9 mm to (103.6, 58.0), turned to 270 degrees
- moved PF_C5 90.7 mm to (111.1, 57.9), turned to 270 degrees
- moved PF_PREAMP 1.91 mm to (109.9, 67.0)
Routing:
- net N$88: track 2.23 -> 10.9 mm
- net N$109: track 2.11 -> 10.2 mm
- net N$101: track 0.00 -> 5.39 mm
- net N$100: track 0.00 -> 5.01 mm
- net N$99: track 0.00 -> 4.92 mm
- net AMPED_PF: track 0.00 -> 4.67 mm
- net N$134: track 0.00 -> 3.30 mm
- net N$98: track 0.00 -> 2.60 mm
- net N$102: track 1.81 -> 3.68 mm
- net GND: track 1.50 -> 3.32 mm, vias 1 -> 2
- net N$97: track 1.76 -> 3.12 mm

Commit message: Finished PA channel (#104)
Parts:
- removed ADC_H5: ADS8322, ti-ads8322:TQFP-32
- removed H4ADC_C1: 1uf, rcl:C0603K
- removed H4RF_C_2, H4_C3, H4_C4, H4_C5, H4_C6, H4_C_POW1, PF_15: 1uf, rcl:C0603
- removed H4RF_C_IN2: 10uf, rcl:C0603
- removed H4RF_C_O5: 0.1uf, rcl:C0603
- removed H4RF_C_O6: 47uf, rcl:C0603
- removed H4RF_R_4: 121k, resistor:R0603
- removed H4RF_R_5: 47m, resistor:R0603
- removed H4_R1: 60.4k, rcl:R0603
- removed H4_R2: 10K, rcl:R0603
- removed H4_REFGEN2: REF6025, REF6025:REF6025
- removed PA_PREAMP2: TLV6741, lio:SC70-5
- removed PF_C20: 270pF, resistor:C0603
- removed PF_C21: 1nF, resistor:C0603
- removed PF_C22: 470 pF, resistor:C0603
- removed PF_C23: 22nF, resistor:C0603
- removed PF_DA1: THS4551, THS4551:VSSOP-8
- removed PF_R19, PF_R22: 330, resistor:R0603
- removed PF_R20: 1.2K, resistor:R0603
- removed PF_R21, PF_R25, PF_R26: 1.2k, resistor:R0603
- removed PF_R23, PF_R24: 5, resistor:R0603
- removed PF_R27, PF_R28: 10, resistor:R0603
- added ADC_PA: ADS8322, ti-ads8322:TQFP-32
- added PA_C10: 10uf, rcl:C0603
- added PA_C11, PA_C14, PA_C15, PA_C17, PA_C18, PA_C19: 1uf, rcl:C0603
- added PA_C12: 47uf, rcl:C0603
- added PA_C13: 0.1uf, rcl:C0603
- added PA_C16: 1uf, rcl:C0603K
- added PA_C5, PA_C9: 270pF, resistor:C0603
- added PA_C6: 470 pF, resistor:C0603
- added PA_C7: 1nF, resistor:C0603
- added PA_C8: 22nF, resistor:C0603
- added PA_DA: THS4551, THS4551:VSSOP-8
- added PA_PREAMP: TLV6741, lio:SC70-5
- added PA_R10, PA_R14, PA_R5: 1.2k, resistor:R0603
- added PA_R11, PA_R7: 330, resistor:R0603
- added PA_R12, PA_R8: 5, resistor:R0603
- added PA_R13, PA_R9: 10, resistor:R0603
- added PA_R15: 121k, resistor:R0603
- added PA_R16: 47m, resistor:R0603
- added PA_R17: 60.4k, rcl:R0603
- added PA_R18: 10K, rcl:R0603
- added PA_R6: 1.2K, resistor:R0603
- added PA_REFGEN: REF6025, REF6025:REF6025
- PF_C15: value 270pF -> 1uf; device resistor:C0603 -> rcl:C0603
- moved PA_R3 326.3 mm to (80.6, 60.0), turned to 90 degrees
- moved PA_C2 325.1 mm to (76.4, 64.7), turned to 270 degrees
- moved PA_R4 322.8 mm to (82.0, 58.3), turned to 270 degrees
- moved PA_C4 314.4 mm to (79.6, 55.8), turned to 90 degrees
- moved PA_R1 314.4 mm to (76.5, 61.4), turned to 270 degrees
- moved PA_R2 312.7 mm to (73.3, 57.6), turned to 270 degrees
- moved PA_C1 308.3 mm to (74.9, 57.6), turned to 270 degrees
- moved PA_C3 306.7 mm to (78.8, 59.9), turned to 90 degrees
- moved PF_C15 103.2 mm to (8.41, -503.2)
- moved PF_REFGEN 27.3 mm to (110.6, 39.3)
- moved SA_IN 23.1 mm to (26.9, 72.6)
- moved SF_IN 15.4 mm to (49.6, 72.8)
- moved PA_IN 4.90 mm to (75.1, 73.0)
Connections:
- net +3V3: now also ADC_PA.27, ADC_PA.28, ADC_PA.29, ADC_PA.32, ADC_PA.6, PA_C10.2, PA_C16.1, PA_C19.1, PA_DA.3, PA_PREAMP.5, PA_REFGEN.1, PA_REFGEN.2; no longer ADC_H5.27, ADC_H5.28, ADC_H5.29, ADC_H5.32, ADC_H5.6, H4ADC_C1.1, H4RF_C_IN2.2, H4_C_POW1.1, H4_REFGEN2.1, H4_REFGEN2.2, PA_PREAMP2.5, PF_DA1.3
- net AMPED_PA: now also PA_PREAMP.4, PA_R6.1; no longer PA_PREAMP2.4, PF_R20.1
- net CLK: now also ADC_PA.24; no longer ADC_H5.24
- net DIFF_N_PA: now also ADC_PA.3, PA_C8.1, PA_R9.2; no longer ADC_H5.3, PF_C23.1, PF_R27.2
- net DIFF_P_PA: now also ADC_PA.4, PA_C8.2, PA_R13.2; no longer ADC_H5.4, PF_C23.2, PF_R28.2
- net DOUT_PA: now also ADC_PA.20; no longer ADC_H5.20
- net DRDY_PA: now also ADC_PA.19; no longer ADC_H5.19
- net GND: now also ADC_PA.10, ADC_PA.12, ADC_PA.13, ADC_PA.14, ADC_PA.15, ADC_PA.16, ADC_PA.18, ADC_PA.21, ADC_PA.23, ADC_PA.26, ADC_PA.30, ADC_PA.31, ADC_PA.5, PA_C10.1, PA_C11.1, PA_C13.1, PA_C14.1, PA_C15.1, PA_C16.2, PA_C17.2, PA_C18.1, PA_C19.2, PA_DA.6, PA_PREAMP.2, PA_R10.1, PA_R15.1, PA_R16.1, PA_R17.2, PA_R18.2, PA_REFGEN.7, PA_REFGEN.8, PF_C15.1; no longer ADC_H5.10, ADC_H5.12, ADC_H5.13, ADC_H5.14, ADC_H5.15, ADC_H5.16, ADC_H5.18, ADC_H5.21, ADC_H5.23, ADC_H5.26, ADC_H5.30, ADC_H5.31, ADC_H5.5, H4ADC_C1.2, H4RF_C_2.1, H4RF_C_IN2.1, H4RF_C_O5.1, H4RF_R_4.1, H4RF_R_5.1, H4_C3.1, H4_C4.1, H4_C5.2, H4_C6.1, H4_C_POW1.2, H4_R1.2, H4_R2.2, H4_REFGEN2.7, H4_REFGEN2.8, PA_PREAMP2.2, PF_15.1, PF_DA1.6, PF_R21.1
- net N$1: now also PA_C5.2, PA_DA.5, PA_R8.1; no longer PF_C15.2, PF_DA1.5, PF_R23.1
- net N$110: now also PA_C11.2, PA_REFGEN.4; no longer H4RF_C_2.2, H4_REFGEN2.4
- net N$116: now also PA_R15.2, PA_REFGEN.3; no longer H4RF_R_4.2, H4_REFGEN2.3
- net N$117: now also PA_C12.1, PA_R16.2; no longer H4RF_C_O6.1, H4RF_R_5.2
- net N$136: now also ADC_PA.1, PA_C15.2; no longer ADC_H5.1, H4_C4.2
- net N$138: now also PA_PREAMP.3; no longer PA_PREAMP2.3
- net N$139: now also PA_PREAMP.1; no longer PA_PREAMP2.1
- net N$140: now also ADC_PA.8, PA_R18.1; no longer ADC_H5.8, H4_R2.1
- net N$144: now also ADC_PA.7, PA_R17.1; no longer ADC_H5.7, H4_R1.1
- net N$148: now also ADC_PA.11, PA_C17.1; no longer ADC_H5.11, H4_C5.1
- net N$149: now also ADC_PA.25, PA_C18.2; no longer ADC_H5.25, H4_C6.2
- net N$150: now also PF_C15.2; no longer PF_15.2
- net N$151: now also ADC_PA.2, PA_C14.2; no longer ADC_H5.2, H4_C3.2
- net N$2: now also PA_C5.1, PA_C7.1, PA_DA.8, PA_R7.2; no longer PF_C15.1, PF_C21.1, PF_DA1.8, PF_R19.2
- net N$3: now also PA_C7.2, PA_C9.1, PA_DA.1, PA_R11.2; no longer PF_C20.1, PF_C21.2, PF_DA1.1, PF_R22.2
- net N$4: now also PA_C6.1, PA_R5.1, PA_R6.2, PA_R7.1; no longer PF_C22.1, PF_R19.1, PF_R20.2, PF_R25.1
- net N$5: now also PA_C6.2, PA_R10.2, PA_R11.1, PA_R14.1; no longer PF_C22.2, PF_R21.2, PF_R22.1, PF_R26.1
- net N$6: now also PA_C9.2, PA_DA.4, PA_R12.1; no longer PF_C20.2, PF_DA1.4, PF_R24.1
- net N$7: now also PA_R5.2, PA_R8.2, PA_R9.1; no longer PF_R23.2, PF_R25.2, PF_R27.1
- net N$8: now also PA_R12.2, PA_R13.1, PA_R14.2; no longer PF_R24.2, PF_R26.2, PF_R28.1
- net REF_PA: now also ADC_PA.9, PA_C12.2, PA_C13.2, PA_REFGEN.5, PA_REFGEN.6; no longer ADC_H5.9, H4RF_C_O5.2, H4RF_C_O6.2, H4_REFGEN2.5, H4_REFGEN2.6
- net SCLK: now also ADC_PA.22; no longer ADC_H5.22
- net START: now also ADC_PA.17; no longer ADC_H5.17
Routing:
- net DRDY_PF: track 0.00 -> 122.4 mm
- net SCLK: track 0.00 -> 111.6 mm, vias 0 -> 2
- net CLK: track 0.00 -> 110.6 mm, vias 0 -> 2
- net DOUT_PF: track 0.00 -> 108.5 mm, vias 0 -> 2
- net START: track 0.00 -> 105.6 mm, vias 0 -> 2
- net DRDY_PA: track 0.00 -> 87.5 mm
- net DOUT_PA: track 0.00 -> 74.6 mm, vias 0 -> 2
- net GND: track 3.32 -> 44.6 mm, vias 2 -> 27
- net +3V3: track 1.70 -> 18.5 mm, vias 1 -> 10
- net N$8: track 0.00 -> 11.3 mm
- net N$7: track 0.00 -> 10.8 mm
- net RAW_PA: track 0.00 -> 7.49 mm
- net AMPED_PA: track 0.00 -> 6.28 mm
- net REF_PA: track 0.00 -> 6.25 mm
- net DIFF_P_PA: track 0.00 -> 6.09 mm
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