File: acoustics/Nice Acoustics/acoustics.sch (EAGLE design)
At the start: 176 parts, among them P1 22-23-2021, X1 22-23-2021, X2 22-23-2021, X3 22-23-2021, X4 22-23-2021

Commit message: Labelled Acoustics input connectors.
Parts:
- renumbered H4_PREAMP2 to PA_PREAMP2, H4_PREAMP3 to SF_PREAMP3, X1 to PF_IN, X2 to PA_IN, X3 to SF_IN, X4 to SA_IN
Changed lines of the file:
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@@
 <part name="AGND48" library="supply1" library_urn="urn:adsk.eagle:library:371" deviceset="AGND" device=""/>
 <part name="AGND49" library="supply1" library_urn="urn:adsk.eagle:library:371" deviceset="AGND" device=""/>
-<part name="H4_PREAMP2" library="lio" deviceset="TLV6741" device=""/>
+<part name="PA_PREAMP2" library="lio" deviceset="TLV6741" device=""/>
 <part name="+3V26" library="supply1" library_urn="urn:adsk.eagle:library:371" deviceset="+3V3" device=""/>
 <part name="AGND50" library="supply1" library_urn="urn:adsk.eagle:library:371" deviceset="AGND" device=""/>
@@
 <part name="AGND52" library="supply1" library_urn="urn:adsk.eagle:library:371" deviceset="AGND" device=""/>
 <part name="AGND53" library="supply1" library_urn="urn:adsk.eagle:library:371" deviceset="AGND" device=""/>
-<part name="H4_PREAMP3" library="lio" deviceset="TLV6741" device=""/>
+<part name="SF_PREAMP3" library="lio" deviceset="TLV6741" device=""/>
 <part name="+3V27" library="supply1" library_urn="urn:adsk.eagle:library:371" deviceset="+3V3" device=""/>
 <part name="AGND54" library="supply1" library_urn="urn:adsk.eagle:library:371" deviceset="AGND" device=""/>
@@
 <part name="AGND2" library="supply1" library_urn="urn:adsk.eagle:library:371" deviceset="AGND" device=""/>
 <part name="AGND3" library="supply1" library_urn="urn:adsk.eagle:library:371" deviceset="AGND" device=""/>
-<part name="X1" library="con-molex" library_urn="urn:adsk.eagle:library:165" deviceset="22-23-2021" device=""/>
-<part name="X2" library="con-molex" library_urn="urn:adsk.eagle:library:165" deviceset="22-23-2021" device=""/>
-<part name="X3" library="con-molex" library_urn="urn:adsk.eagle:library:165" deviceset="22-23-2021" device=""/>
-<part name="X4" library="con-molex" library_urn="urn:adsk.eagle:library:165" deviceset="22-23-2021" device=""/>
+<part name="PF_IN" library="con-molex" library_urn="urn:adsk.eagle:library:165" deviceset="22-23-2021" device=""/>
+<part name="PA_IN" library="con-molex" library_urn="urn:adsk.eagle:library:165" deviceset="22-23-2021" device=""/>
+<part name="SF_IN" library="con-molex" library_urn="urn:adsk.eagle:library:165" deviceset="22-23-2021" device=""/>
+<part name="SA_IN" library="con-molex" library_urn="urn:adsk.eagle:library:165" deviceset="22-23-2021" device=""/>
 <part name="AGND4" library="supply1" library_urn="urn:adsk.eagle:library:371" deviceset="AGND" device=""/>
 <part name="AGND5" library="supply1" library_urn="urn:adsk.eagle:library:371" deviceset="AGND" device=""/>
@@
 <instance part="AGND2" gate="VR1" x="35.56" y="30.48"/>
 <instance part="AGND3" gate="VR1" x="22.86" y="30.48"/>
-<instance part="X1" gate="-1" x="129.54" y="81.28"/>
-<instance part="X1" gate="-2" x="129.54" y="78.74"/>
-<instance part="X2" gate="-1" x="129.54" y="66.04"/>
-<instance part="X2" gate="-2" x="129.54" y="63.5"/>
-<instance part="X3" gate="-1" x="129.54" y="50.8"/>
-<instance part="X3" gate="-2" x="129.54" y="48.26"/>
-<instance part="X4" gate="-1" x="129.54" y="35.56"/>
-<instance part="X4" gate="-2" x="129.54" y="33.02"/>
+<instance part="PF_IN" gate="-1" x="129.54" y="81.28"/>
+<instance part="PF_IN" gate="-2" x="129.54" y="78.74"/>
+<instance part="PA_IN" gate="-1" x="129.54" y="66.04"/>
+<instance part="PA_IN" gate="-2" x="129.54" y="63.5"/>
+<instance part="SF_IN" gate="-1" x="129.54" y="50.8"/>
+<instance part="SF_IN" gate="-2" x="129.54" y="48.26"/>
+<instance part="SA_IN" gate="-1" x="129.54" y="35.56"/>
+<instance part="SA_IN" gate="-2" x="129.54" y="33.02"/>
 <instance part="AGND4" gate="VR1" x="124.46" y="27.94"/>
 <instance part="AGND5" gate="VR1" x="124.46" y="43.18"/>
@@
 <net name="RAW_PF" class="0">
 <segment>
-<pinref part="X1" gate="-1" pin="S"/>
+<pinref part="PF_IN" gate="-1" pin="S"/>
 <wire x1="127" y1="81.28" x2="106.68" y2="81.28" width="0.1524" layer="91"/>
 <label x="96.52" y="81.28" size="1.778" layer="95"/>
@@
 <net name="RAW_PA" class="0">
 <segment>
-<pinref part="X2" gate="-1" pin="S"/>
+<pinref part="PA_IN" gate="-1" pin="S"/>
 <wire x1="127" y1="66.04" x2="106.68" y2="66.04" width="0.1524" layer="91"/>
 <label x="96.52" y="66.04" size="1.778" layer="95"/>
@@
 <net name="RAW_SF" class="0">
 <segment>
-<pinref part="X3" gate="-1" pin="S"/>
+<pinref part="SF_IN" gate="-1" pin="S"/>
 <wire x1="127" y1="50.8" x2="106.68" y2="50.8" width="0.1524" layer="91"/>
 <label x="96.52" y="50.8" size="1.778" layer="95"/>
@@
 <net name="RAW_SA" class="0">
 <segment>
-<pinref part="X4" gate="-1" pin="S"/>
+<pinref part="SA_IN" gate="-1" pin="S"/>
 <wire x1="127" y1="35.56" x2="106.68" y2="35.56" width="0.1524" layer="91"/>
 <label x="96.52" y="35.56" size="1.778" layer="95"/>
@@
 </segment>
 <segment>
-<pinref part="X4" gate="-2" pin="S"/>
+<pinref part="SA_IN" gate="-2" pin="S"/>
 <wire x1="127" y1="33.02" x2="124.46" y2="33.02" width="0.1524" layer="91"/>
 <wire x1="124.46" y1="33.02" x2="124.46" y2="30.48" width="0.1524" layer="91"/>
@@
 </segment>
 <segment>
-<pinref part="X3" gate="-2" pin="S"/>
+<pinref part="SF_IN" gate="-2" pin="S"/>
 <wire x1="127" y1="48.26" x2="124.46" y2="48.26" width="0.1524" layer="91"/>
 <wire x1="124.46" y1="48.26" x2="124.46" y2="45.72" width="0.1524" layer="91"/>
@@
 </segment>
 <segment>
-<pinref part="X2" gate="-2" pin="S"/>
+<pinref part="PA_IN" gate="-2" pin="S"/>
 <wire x1="127" y1="63.5" x2="124.46" y2="63.5" width="0.1524" layer="91"/>
 <wire x1="124.46" y1="63.5" x2="124.46" y2="60.96" width="0.1524" layer="91"/>
@@
 </segment>
 <segment>
-<pinref part="X1" gate="-2" pin="S"/>
+<pinref part="PF_IN" gate="-2" pin="S"/>
 <wire x1="127" y1="78.74" x2="124.46" y2="78.74" width="0.1524" layer="91"/>
 <wire x1="124.46" y1="78.74" x2="124.46" y2="76.2" width="0.1524" layer="91"/>
@@
 <attribute name="VALUE" x="20.32" y="287.02" size="1.778" layer="96" rot="R90"/>
 </instance>
-<instance part="H4_PREAMP2" gate="G$1" x="48.26" y="259.08"/>
+<instance part="PA_PREAMP2" gate="G$1" x="48.26" y="259.08"/>
 <instance part="+3V26" gate="G$1" x="50.8" y="254"/>
 <instance part="AGND50" gate="VR1" x="58.42" y="269.24"/>
@@
 <attribute name="VALUE" x="20.32" y="226.06" size="1.778" layer="96" rot="R90"/>
 </instance>
-<instance part="H4_PREAMP3" gate="G$1" x="48.26" y="198.12"/>
+<instance part="SF_PREAMP3" gate="G$1" x="48.26" y="198.12"/>
 <instance part="+3V27" gate="G$1" x="50.8" y="193.04"/>
 <instance part="AGND54" gate="VR1" x="58.42" y="208.28"/>
@@
 <pinref part="+3V26" gate="G$1" pin="+3V3"/>
 <wire x1="50.8" y1="248.92" x2="50.8" y2="251.46" width="0.1524" layer="91"/>
-<pinref part="H4_PREAMP2" gate="G$1" pin="V+"/>
+<pinref part="PA_PREAMP2" gate="G$1" pin="V+"/>
 <wire x1="45.72" y1="248.92" x2="45.72" y2="251.46" width="0.1524" layer="91"/>
 <wire x1="43.18" y1="248.92" x2="45.72" y2="248.92" width="0.1524" layer="91"/>
@@
 <pinref part="+3V27" gate="G$1" pin="+3V3"/>
 <wire x1="50.8" y1="187.96" x2="50.8" y2="190.5" width="0.1524" layer="91"/>
-<pinref part="H4_PREAMP3" gate="G$1" pin="V+"/>
+<pinref part="SF_PREAMP3" gate="G$1" pin="V+"/>
 <wire x1="45.72" y1="187.96" x2="45.72" y2="190.5" width="0.1524" layer="91"/>
 <wire x1="43.18" y1="187.96" x2="45.72" y2="187.96" width="0.1524" layer="91"/>
@@
 </segment>
 <segment>
-<pinref part="H4_PREAMP2" gate="G$1" pin="V-"/>
+<pinref part="PA_PREAMP2" gate="G$1" pin="V-"/>
 <wire x1="45.72" y1="271.78" x2="45.72" y2="274.32" width="0.1524" layer="91"/>
 <wire x1="45.72" y1="274.32" x2="58.42" y2="274.32" width="0.1524" layer="91"/>
@@
 </segment>
 <segment>
-<pinref part="H4_PREAMP3" gate="G$1" pin="V-"/>
+<pinref part="SF_PREAMP3" gate="G$1" pin="V-"/>
 <wire x1="45.72" y1="210.82" x2="45.72" y2="213.36" width="0.1524" layer="91"/>
 <wire x1="45.72" y1="213.36" x2="58.42" y2="213.36" width="0.1524" layer="91"/>
@@
 <pinref part="PA_C1" gate="G$1" pin="1"/>
 <wire x1="27.94" y1="281.94" x2="38.1" y2="281.94" width="0.1524" layer="91"/>
-<pinref part="H4_PREAMP2" gate="G$1" pin="-IN"/>
+<pinref part="PA_PREAMP2" gate="G$1" pin="-IN"/>
 <pinref part="PA_R1" gate="G$1" pin="2"/>
 <wire x1="25.4" y1="264.16" x2="27.94" y2="264.16" width="0.1524" layer="91"/>
@@
 <segment>
 <wire x1="63.5" y1="276.86" x2="63.5" y2="261.62" width="0.1524" layer="91"/>
-<pinref part="H4_PREAMP2" gate="G$1" pin="OUT"/>
+<pinref part="PA_PREAMP2" gate="G$1" pin="OUT"/>
 <wire x1="63.5" y1="261.62" x2="60.96" y2="261.62" width="0.1524" layer="91"/>
 <pinref part="PA_R2" gate="G$1" pin="2"/>
@@
 <segment>
 <pinref part="PA_R4" gate="G$1" pin="1"/>
-<pinref part="H4_PREAMP2" gate="G$1" pin="+IN"/>
+<pinref part="PA_PREAMP2" gate="G$1" pin="+IN"/>
 <wire x1="30.48" y1="259.08" x2="22.86" y2="259.08" width="0.1524" layer="91"/>
 <wire x1="22.86" y1="259.08" x2="22.86" y2="248.92" width="0.1524" layer="91"/>
@@
 <pinref part="SF_C1" gate="G$1" pin="1"/>
 <wire x1="27.94" y1="220.98" x2="38.1" y2="220.98" width="0.1524" layer="91"/>
-<pinref part="H4_PREAMP3" gate="G$1" pin="-IN"/>
+<pinref part="SF_PREAMP3" gate="G$1" pin="-IN"/>
 <pinref part="SF_R1" gate="G$1" pin="2"/>
 <wire x1="25.4" y1="203.2" x2="27.94" y2="203.2" width="0.1524" layer="91"/>
@@
 <segment>
 <wire x1="63.5" y1="215.9" x2="63.5" y2="200.66" width="0.1524" layer="91"/>
-<pinref part="H4_PREAMP3" gate="G$1" pin="OUT"/>
+<pinref part="SF_PREAMP3" gate="G$1" pin="OUT"/>
 <wire x1="63.5" y1="200.66" x2="60.96" y2="200.66" width="0.1524" layer="91"/>
 <pinref part="SF_R2" gate="G$1" pin="2"/>
@@
 <segment>
 <pinref part="SF_R4" gate="G$1" pin="1"/>
-<pinref part="H4_PREAMP3" gate="G$1" pin="+IN"/>
+<pinref part="SF_PREAMP3" gate="G$1" pin="+IN"/>
 <wire x1="30.48" y1="198.12" x2="22.86" y2="198.12" width="0.1524" layer="91"/>
 <wire x1="22.86" y1="198.12" x2="22.86" y2="187.96" width="0.1524" layer="91"/>

Commit message: Finished PA channel (#104)
Parts:
- removed PF_15: 1uf, rcl:C-EUC0603
- added PA_C5: 270pF, resistor:C-EUC0603
- PF_C15: value 270pF -> 1uf; device resistor:C-EUC0603 -> rcl:C-EUC0603
- renumbered ADC_H5 to ADC_PA, H4ADC_C1 to PA_C16, H4RF_C_2 to PA_C11, H4RF_C_IN2 to PA_C10, H4RF_C_O5 to PA_C13, H4RF_C_O6 to PA_C12, H4RF_R_4 to PA_R15, H4RF_R_5 to PA_R16, H4_C3 to PA_C14, H4_C4 to PA_C15, H4_C5 to PA_C17, H4_C6 to PA_C18, H4_C_POW1 to PA_C19, H4_R1 to PA_R17, H4_R2 to PA_R18, H4_REFGEN2 to PA_REFGEN, PA_PREAMP2 to PA_PREAMP, PF_C20 to PA_C9, PF_C21 to PA_C7, PF_C22 to PA_C6, PF_C23 to PA_C8, PF_DA1 to PA_DA, PF_R19 to PA_R7, PF_R20 to PA_R6, PF_R21 to PA_R10, PF_R22 to PA_R11, PF_R23 to PA_R8, PF_R24 to PA_R12, PF_R25 to PA_R5, PF_R26 to PA_R14, PF_R27 to PA_R9, PF_R28 to PA_R13
Connections:
- net GND: now also PF_C15.1; no longer PF_15.1
- net N$1: now also PA_C5.2; no longer PF_C15.2
- net N$150: now also PF_C15.2; no longer PF_15.2
- net N$2: now also PA_C5.1; no longer PF_C15.1
